File: Noise-SH/PanelMisc.sch (KiCad schematic (older format))
At the start: 28 parts, among them J10 Conn__Back, J11 Eurorack_10, J5 WQP-PJ398SM, J6 WQP-PJ398SM, J7 WQP-PJ398SM, J8 WQP-PJ398SM, J9 Conn_Front, SW5 ON_ON, SW6 SPST, U2 TL072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

Commit message: Noise-SH: change name of project symbol lib
Parts:
- C1, C10, C11, C2: symbol Noise-SH-rescue:CP_10U--lmp-synth -> Noise-SH:CP_10U--lmp-synth
- C3, C4, C5, C6, C7: symbol Noise-SH-rescue:CC_100N--lmp -> Noise-SH:CC_100N--lmp
- D1, D2: symbol Noise-SH-rescue:MBR150--lmp-diode -> Noise-SH:MBR150--lmp-diode
- D3: symbol Noise-SH-rescue:LED_5mm_Blue--lmp-synth -> Noise-SH:LED_5mm_Blue--lmp-synth
- H1: symbol Noise-SH-rescue:PCB_Delptronics_MCS_4HP--lmp-synth -> Noise-SH:PCB_Delptronics_MCS_4HP--lmp-synth
- J10: symbol Noise-SH-rescue:Conn_Delptronics_Back_Left_4HP--lmp-synth -> Noise-SH:Conn_Delptronics_Back_Left_4HP--lmp-synth
- J11: symbol Noise-SH-rescue:Conn_Delptronics_Pwr_Hdr_10--lmp-synth -> Noise-SH:Conn_Delptronics_Pwr_Hdr_10--lmp-synth
- J5, J6, J7, J8: symbol Noise-SH-rescue:Jack_WQP-PJ398--lmp-synth -> Noise-SH:Jack_WQP-PJ398--lmp-synth
- J9: symbol Noise-SH-rescue:Conn_Delptronics_Front_Left_4HP--lmp-synth -> Noise-SH:Conn_Delptronics_Front_Left_4HP--lmp-synth
- R1, R2: symbol Noise-SH-rescue:R--lmp -> Noise-SH:R--lmp
- RV7, RV8: symbol Noise-SH-rescue:R_POT_Panel_PCB_Alpha--lmp-synth -> Noise-SH:R_POT_Panel_PCB_Alpha--lmp-synth
- SW5: symbol Noise-SH-rescue:SW_SPDT_ON_ON--lmp-synth -> Noise-SH:SW_SPDT_ON_ON--lmp-synth
- SW6: symbol Noise-SH-rescue:SW_SPST--lmp-synth -> Noise-SH:SW_SPST--lmp-synth
- U2: symbol Noise-SH-rescue:TL072--lmp-opamp -> Noise-SH:TL072--lmp-opamp
- U4: symbol Noise-SH-rescue:TL074--lmp-opamp -> Noise-SH:TL074--lmp-opamp
Changed lines of the file:
@@
 Front Panel
 $Comp
-L Noise-SH-rescue:Logo_CC_BY_SA--lmp #G1
+L Noise-SH:Logo_CC_BY_SA--lmp #G1
 U 1 1 60E205CA
 P 900 7550
@@
 $EndComp
 $Comp
-L Noise-SH-rescue:Conn_Delptronics_Front_Left_4HP--lmp-synth J9
+L Noise-SH:Conn_Delptronics_Front_Left_4HP--lmp-synth J9
 U 1 1 60E205D9
 P 3550 2200
@@
 $EndComp
 $Comp
-L Noise-SH-rescue:Conn_Delptronics_Back_Left_4HP--lmp-synth J10
+L Noise-SH:Conn_Delptronics_Back_Left_4HP--lmp-synth J10
 U 1 1 60CAA39B
 P 4450 2200
@@
 	3350 3400 3300 3400
 $Comp
-L Noise-SH-rescue:GND--lmp-power #PWR05
+L Noise-SH:GND--lmp-power #PWR05
 U 1 1 60CD7485
 P 3300 3450
@@
 	1550 4900 1550 4850
 $Comp
-L Noise-SH-rescue:GND--lmp-power #PWR04
+L Noise-SH:GND--lmp-power #PWR04
 U 1 1 60E49087
 P 1550 4900
@@
 	1550 6100 1550 6050
 $Comp
-L Noise-SH-rescue:GND--lmp-power #PWR03
+L Noise-SH:GND--lmp-power #PWR03
 U 1 1 60E473D6
 P 1550 6100
@@
 	1550 5500 1550 5450
 $Comp
-L Noise-SH-rescue:GND--lmp-power #PWR02
+L Noise-SH:GND--lmp-power #PWR02
 U 1 1 60E458BF
 P 1550 5500
@@
 	1550 4300 1550 4250
 $Comp
-L Noise-SH-rescue:GND--lmp-power #PWR01
+L Noise-SH:GND--lmp-power #PWR01
 U 1 1 60E205DB
 P 1550 4300
@@
 $EndComp
 $Comp
-L Noise-SH-rescue:Jack_WQP-PJ398--lmp-synth J5
+L Noise-SH:Jack_WQP-PJ398--lmp-synth J5
 U 1 1 60E205DF
 P 1300 4150
@@
 $EndComp
 $Comp
-L Noise-SH-rescue:Jack_WQP-PJ398--lmp-synth J6
+L Noise-SH:Jack_WQP-PJ398--lmp-synth J6
 U 1 1 60E35493
 P 1300 5350
@@
 $EndComp
 $Comp
-L Noise-SH-rescue:Jack_WQP-PJ398--lmp-synth J7
+L Noise-SH:Jack_WQP-PJ398--lmp-synth J7
 U 1 1 60E3736C
 P 1300 5950
@@
 $EndComp
 $Comp
-L Noise-SH-rescue:Jack_WQP-PJ398--lmp-synth J8
+L Noise-SH:Jack_WQP-PJ398--lmp-synth J8
 U 1 1 60E378DF
 P 1300 4750
@@
 NoConn ~ 1500 5250
 $Comp
-L Noise-SH-rescue:LED_5mm_Blue--lmp-synth D3
+L Noise-SH:LED_5mm_Blue--lmp-synth D3
 U 1 1 60E9F439
 P 1350 3650
@@
 	1050 1850 1050 2250
 $Comp
-L Noise-SH-rescue:R_POT_Panel_PCB_Alpha--lmp-synth RV7
+L Noise-SH:R_POT_Panel_PCB_Alpha--lmp-synth RV7
 U 1 1 60E2D734
 P 1350 2650
@@
 	1350 2800 1350 2850
 $Comp
-L Noise-SH-rescue:SW_SPST--lmp-synth SW6
+L Noise-SH:SW_SPST--lmp-synth SW6
 U 1 1 60F35C8E
 P 1300 2250
@@
 	1050 1650 1100 1650
 $Comp
-L Noise-SH-rescue:SW_SPDT_ON_ON--lmp-synth SW5
+L Noise-SH:SW_SPDT_ON_ON--lmp-synth SW5
 U 1 1 60E2ECA7
 P 1300 1550
@@
 	950  1750 1650 1750
 $Comp
-L Noise-SH-rescue:R_POT_Panel_PCB_Alpha--lmp-synth RV8
+L Noise-SH:R_POT_Panel_PCB_Alpha--lmp-synth RV8
 U 1 1 61183B05
 P 1350 3150
@@
 OUT-NOISE-PINK
 $Comp
-L Noise-SH-rescue:GND--lmp-power #PWR06
+L Noise-SH:GND--lmp-power #PWR06
 U 1 1 60E205DD
 P 4700 3450
@@
 	9250 1100 9550 1100
 $Comp
-L Noise-SH-rescue:PWR_FLAG--lmp-power #FLG0102
+L Noise-SH:PWR_FLAG--lmp-power #FLG0102
 U 1 1 60E47861
 P 9550 1700
@@
 $EndComp
 $Comp
-L Noise-SH-rescue:PWR_FLAG--lmp-power #FLG0101
+L Noise-SH:PWR_FLAG--lmp-power #FLG0101
 U 1 1 60E46A75
 P 9550 1100
@@
 	6450 3100 7150 3100
 $Comp
-L Noise-SH-rescue:GND--lmp-power #PWR011
+L Noise-SH:GND--lmp-power #PWR011
 U 1 1 60E6B187
 P 7800 3150
@@
 $EndComp
 $Comp
-L Noise-SH-rescue:TL072--lmp-opamp U2
+L Noise-SH:TL072--lmp-opamp U2
 U 3 1 60E82BE4
 P 8200 3100
@@
 $EndComp
 $Comp
-L Noise-SH-rescue:CC_100N--lmp C6
+L Noise-SH:CC_100N--lmp C6
 U 1 1 60EA094A
 P 8500 2950
@@
 $EndComp
 $Comp
-L Noise-SH-rescue:CC_100N--lmp C7
+L Noise-SH:CC_100N--lmp C7
 U 1 1 60EA0950
 P 8500 3250
@@
 $EndComp
 $Comp
-L Noise-SH-rescue:CC_100N--lmp C5
+L Noise-SH:CC_100N--lmp C5
 U 1 1 60E8BD91
 P 7150 3250
@@
 $EndComp
 $Comp
-L Noise-SH-rescue:CC_100N--lmp C4
+L Noise-SH:CC_100N--lmp C4
 U 1 1 60E8B4DE
 P 7150 2950
@@
 $EndComp
 $Comp
-L Noise-SH-rescue:TL074--lmp-opamp U4
+L Noise-SH:TL074--lmp-opamp U4
 U 5 1 60E8AF46
 P 6850 3100
@@
 $EndComp
 $Comp
-L Noise-SH-rescue:-12V--lmp-power #PWR09
+L Noise-SH:-12V--lmp-power #PWR09
 U 1 1 60E5D3C2
 P 6450 3500
@@
 $EndComp
 $Comp
-L Noise-SH-rescue:GND--lmp-power #PWR08
+L Noise-SH:GND--lmp-power #PWR08
 U 1 1 60E5D3BA
 P 6450 3150
@@
 $EndComp
 $Comp
-L Noise-SH-rescue:+12V--lmp-power #PWR07
+L Noise-SH:+12V--lmp-power #PWR07
 U 1 1 60E5D3B4
 P 6450 2700
@@
 	9250 1100 9250 1000
 $Comp
-L Noise-SH-rescue:PWR_FLAG--lmp-power #FLG04
+L Noise-SH:PWR_FLAG--lmp-power #FLG04
 U 1 1 60C8985D
 P 7650 1100
@@
 	7950 1700 8100 1700
 $Comp
-L Noise-SH-rescue:CP_10U--lmp-synth C11
+L Noise-SH:CP_10U--lmp-synth C11
 U 1 1 60E3F037
 P 8550 1550
@@
 $EndComp
 $Comp
-L Noise-SH-rescue:CP_10U--lmp-synth C10
+L Noise-SH:CP_10U--lmp-synth C10
 U 1 1 60E3E7EC
 P 8550 1250
@@
 $EndComp
 $Comp
-L Noise-SH-rescue:R--lmp R2
+L Noise-SH:R--lmp R2
 U 1 1 60E3E434
 P 8250 1700
@@
 $EndComp
 $Comp
-L Noise-SH-rescue:R--lmp R1
+L Noise-SH:R--lmp R1
 U 1 1 60E3DDAE
 P 8250 1100
@@
 Power
 $Comp
-L Noise-SH-rescue:-12V--lmp-power #PWR015
+L Noise-SH:-12V--lmp-power #PWR015
 U 1 1 60C864E4
 P 7950 1800
@@
 Connection ~ 6950 1400
 $Comp
-L Noise-SH-rescue:PWR_FLAG--lmp-power #FLG01
+L Noise-SH:PWR_FLAG--lmp-power #FLG01
 U 1 1 60E205CC
 P 6450 1100
@@
 $EndComp
 $Comp
-L Noise-SH-rescue:PWR_FLAG--lmp-power #FLG02
+L Noise-SH:PWR_FLAG--lmp-power #FLG02
 U 1 1 60E205CD
 P 6450 1300
@@
 $EndComp
 $Comp
-L Noise-SH-rescue:PWR_FLAG--lmp-power #FLG03
+L Noise-SH:PWR_FLAG--lmp-power #FLG03
 U 1 1 60E205CE
 P 6450 1500
@@
 	7000 1700 7050 1700
 $Comp
-L Noise-SH-rescue:MBR150--lmp-diode D1
+L Noise-SH:MBR150--lmp-diode D1
 U 1 1 60E205CF
 P 7200 1700
@@
 $EndComp
 $Comp
-L Noise-SH-rescue:MBR150--lmp-diode D2
+L Noise-SH:MBR150--lmp-diode D2
 U 1 1 60E205D0
 P 7200 1100
@@
 $EndComp
 $Comp
-L Noise-SH-rescue:CP_10U--lmp-synth C2
+L Noise-SH:CP_10U--lmp-synth C2
 U 1 1 60E205D1
 P 7500 1250
@@
 $EndComp
 $Comp
-L Noise-SH-rescue:CP_10U--lmp-synth C1
+L Noise-SH:CP_10U--lmp-synth C1
 U 1 1 60E205D2
 P 7500 1550
@@
 $EndComp
 $Comp
-L Noise-SH-rescue:GND--lmp-power #PWR014
+L Noise-SH:GND--lmp-power #PWR014
 U 1 1 60C80BF1
 P 7950 1450
@@
 Connection ~ 7500 1700
 $Comp
-L Noise-SH-rescue:+12V--lmp-power #PWR013
+L Noise-SH:+12V--lmp-power #PWR013
 U 1 1 60E205D4
 P 7950 1000
@@
 	7950 1800 7950 1700
 $Comp
-L Noise-SH-rescue:PWR_FLAG--lmp-power #FLG05
+L Noise-SH:PWR_FLAG--lmp-power #FLG05
 U 1 1 60C89F71
 P 7650 1700
@@
 	6750 2800 7150 2800
 $Comp
-L Noise-SH-rescue:CC_100N--lmp C3
+L Noise-SH:CC_100N--lmp C3
 U 1 1 6126B150
 P 9000 1400
@@
 IN-SAMPLE is normalled from OUT-NOISE.
 $Comp
-L Noise-SH-rescue:PCB_Delptronics_MCS_4HP--lmp-synth H1
+L Noise-SH:PCB_Delptronics_MCS_4HP--lmp-synth H1
 U 1 1 61B16299
 P 7300 5200
@@
 	6950 1100 6450 1100
 $Comp
-L Noise-SH-rescue:Conn_Delptronics_Pwr_Hdr_10--lmp-synth J11
+L Noise-SH:Conn_Delptronics_Pwr_Hdr_10--lmp-synth J11
 U 1 1 60E205CB
 P 6650 1300
