File: modules/LFO-DigiVC/LFO-DigiVC.kicad_pcb (KiCad board)
At the start: 6 copper layers, 101.6 x 106.7 mm, 58 parts, among them J1 FTDI USB-TTL, J10 Conn_Front, J11 Conn_Back, J5 WQP-PJ398, J6 WQP-PJ398, J7 WQP-PJ398, J8 WQP-PJ398, J9 Eurorack_10, Q1 2N3904, SW6 ON_OFF_ON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

Commit message: LFO-DigiVC: clean up schematic and layout, add more files
Parts:
- moved C10 102.4 mm to (188.0, 124.5)
- moved C3 102.4 mm to (184.2, 138.4)
- moved C5 102.4 mm to (215.9, 99.1)
- moved C6 102.4 mm to (213.4, 63.5)
- moved C8 102.4 mm to (226.1, 68.6)
- moved C9 102.4 mm to (188.0, 111.8)
- moved D1 102.4 mm to (219.7, 138.4)
- moved D2 102.4 mm to (212.1, 142.0)
- moved D3 102.4 mm to (198.1, 86.4)
- moved J1 102.4 mm to (226.1, 83.8)
- moved J11 102.4 mm to (177.8, 55.9)
- moved J9 102.4 mm to (226.1, 142.2)
- moved JP1 102.4 mm to (213.4, 78.7)
- moved Q1 102.4 mm to (205.7, 38.1)
- moved R1 102.4 mm to (195.6, 83.8)
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Routing:
- net Net-(C11-Pad1): track 34.7 -> 36.7 mm
- net POT-IN-1: track 30.0 -> 30.8 mm
Other:
- net class Default: trace_width 0.25 -> 0.0508
- rule trace_min: 0.2 -> 0.0508
