File: modules/VCA-4/prototype/prototype.kicad_pcb (KiCad board)
At the start: 6 copper layers, 40.6 x 81.3 mm, 15 parts, among them J1 Conn_01x09, U1 TL074, U2 SSI2164

Commit message: VCA4 prototype wip
Other:
- board text added: "1"
- board text added: "13"
- board text added: "19"
- board text added: "25"
- board text added: "8"
Changed lines of the file:
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@@
   (gr_line (start 82.55 102.87) (end 82.55 21.59) (layer "Edge.Cuts") (width 0.1))
   (gr_line (start 82.55 21.59) (end 123.19 21.59) (layer "Edge.Cuts") (width 0.1))
+  (gr_text "19" (at 118.11 71.247) (layer "Cmts.User")
+    (effects (font (size 1 1) (thickness 0.15)))
+  )
+  (gr_text "25" (at 120.65 86.36) (layer "Cmts.User")
+    (effects (font (size 1 1) (thickness 0.15)))
+  )
   (gr_text "CV1" (at 104.14 101.6) (layer "Cmts.User")
     (effects (font (size 1.524 1.524) (thickness 0.254)))
@@
   (gr_text "May connect to \nexternal CV instead" (at 99.822 90.297) (layer "Cmts.User")
     (effects (font (size 1 1) (thickness 0.15)) (justify left))
+  )
+  (gr_text "8" (at 117.983 42.672) (layer "Cmts.User")
+    (effects (font (size 1 1) (thickness 0.15)))
   )
   (gr_text "+5V" (at 97.155 101.6) (layer "Cmts.User")
@@
     (effects (font (size 1.524 1.524) (thickness 0.254)))
   )
+  (gr_text "13" (at 117.983 55.88) (layer "Cmts.User")
+    (effects (font (size 1 1) (thickness 0.15)))
+  )
+  (gr_text "1" (at 118.11 25.4) (layer "Cmts.User")
+    (effects (font (size 1 1) (thickness 0.15)))
+  )
   (segment (start 99.06 73.66) (end 88.9 73.66) (width 0.4064) (layer "F.Cu") (net 0))

Commit message: VCA4 prototype wip
Parts:
- added R11: 11K, -lmp-stripboard:SB_Gen_1, F.Cu at (88.9, 61.0)
Changed lines of the file:
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@@
+    )
+  )
+  (footprint "-lmp-stripboard:SB_Gen_1" (layer "F.Cu")
+    (at 88.9 60.96 180)
+    (descr "Stripboard, span 1 row")
+    (tags "Stripboard")
+    (property "Distributor" "Mouser")
+    (property "DistributorPartLink" "https://www.mouser.ca/c/passive-components/resistors/film-resistors/metal-film-resistors-through-hole/?m=YAGEO&power%20rating=166%20mW%20%281%2F6%20W%29&tolerance=1%20%25&instock=y")
+    (property "DistributorPartNum" "603-MFR-12*")
+    (property "Manufacturer" "YAGEO")
+    (property "ManufacturerPartNum" "MFR-12*")
+    (property "Sheetfile" "prototype.kicad_sch")
+    (property "Sheetname" "")
+    (property "Value2" "1%, 1/6 W")
+    (attr through_hole)
+    (fp_text reference "R11" (at 1.27 -2.37 180) (layer "F.SilkS")
+      (effects (font (size 1 1) (thickness 0.15)))
+    )
+    (fp_text value "11K" (at 1.27 2.37 180) (layer "F.Fab")
+      (effects (font (size 1 1) (thickness 0.15)))
+    )
+    (fp_text user "${REFERENCE}" (at 1.27 -2.37 180) (layer "F.Fab")
+      (effects (font (size 1 1) (thickness 0.15)))
+    )
+    (fp_line (start 1.37 0) (end 1.44 0) (layer "F.SilkS") (width 0.12))
+    (fp_circle (center 0 0) (end 1.37 0) (layer "F.SilkS") (width 0.12) (fill none))
+    (fp_line (start -1.5 -1.5) (end -1.5 1.5) (layer "F.CrtYd") (width 0.05))
+    (fp_line (start 3.59 -1.5) (end -1.5 -1.5) (layer "F.CrtYd") (width 0.05))
+    (fp_line (start 3.59 1.5) (end 3.59 -1.5) (layer "F.CrtYd") (width 0.05))
+    (fp_line (start -1.5 1.5) (end 3.59 1.5) (layer "F.CrtYd") (width 0.05))
+    (fp_line (start 0 0) (end 2.54 0) (layer "F.Fab") (width 0.1))
+    (fp_circle (center 0 0) (end 1.25 0) (layer "F.Fab") (width 0.1) (fill none))
+    (pad "1" thru_hole circle locked (at 0 0 180) (size 1.6 1.6) (drill 0.8) (layers *.Cu *.Mask)
+      (net 12 "Net-(R2-Pad2)") (pintype "passive"))
+    (pad "2" thru_hole oval locked (at 2.54 0 180) (size 1.6 1.6) (drill 0.8) (layers *.Cu *.Mask)
+      (net 23 "GND") (pintype "passive"))
+    (model "${KISYS3DMOD}/Resistor_THT.3dshapes/R_Axial_DIN0207_L6.3mm_D2.5mm_P2.54mm_Vertical.wrl"
+      (offset (xyz 0 0 0))
+      (scale (xyz 1 1 1))
+      (rotate (xyz 0 0 0))
     )
   )
@@
       (net 1 "+12V") (pinfunction "V+") (pintype "power_in"))
   )
+  (gr_circle (center 87.757 60.96) (end 90.68076 60.96) (layer "Dwgs.User") (width 0.508) (fill none))
   (gr_circle (center 100.076 87.884) (end 100.643961 87.884) (layer "Dwgs.User") (width 0.1) (fill solid))
   (gr_line (start 123.19 102.87) (end 82.55 102.87) (layer "Edge.Cuts") (width 0.1))

Commit message: VCA4 prototype wip
Connections:
- RV1 pad 1: +5V -> GND
- RV1 pad 3: GND -> +5V
Routing:
- net +5V: track 87.9 -> 85.8 mm
Changed lines of the file:
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@@
   (net 10 "Net-(R1-Pad1)")
   (net 11 "Net-(R1-Pad2)")
-  (net 12 "Net-(R2-Pad2)")
+  (net 12 "Net-(R11-Pad1)")
   (net 13 "Net-(R3-Pad2)")
   (net 14 "Net-(R5-Pad2)")
@@
     (fp_line (start 4.765 -4.465) (end 4.765 5.065) (layer "F.Fab") (width 0.2))
     (pad "1" thru_hole circle (at 2.54 -1.925 90) (size 1.302857 1.302857) (drill 0.76) (layers *.Cu *.Mask)
-      (net 3 "+5V") (pinfunction "1") (pintype "passive"))
+      (net 23 "GND") (pinfunction "1") (pintype "passive"))
     (pad "2" thru_hole circle (at 0 -1.925 90) (size 1.302857 1.302857) (drill 0.76) (layers *.Cu *.Mask)
       (net 10 "Net-(R1-Pad1)") (pinfunction "2") (pintype "passive"))
     (pad "3" thru_hole circle (at -2.54 -1.925 90) (size 1.302857 1.302857) (drill 0.76) (layers *.Cu *.Mask)
-      (net 23 "GND") (pinfunction "3") (pintype "passive"))
+      (net 3 "+5V") (pinfunction "3") (pintype "passive"))
     (model "C:\\Users\\Len\\OneDrive\\Documents\\Electronics\\KiCad\\download\\SamacSys_Parts.3dshapes\\3310R-101-103L.stp"
       (offset (xyz 0 0 0))
@@
       (net 3 "+5V") (pintype "passive"))
     (pad "2" thru_hole oval locked (at 7.62 0 270) (size 1.6 1.6) (drill 0.8) (layers *.Cu *.Mask)
-      (net 12 "Net-(R2-Pad2)") (pintype "passive"))
+      (net 12 "Net-(R11-Pad1)") (pintype "passive"))
     (model "${KISYS3DMOD}/Resistor_THT.3dshapes/R_Axial_DIN0207_L6.3mm_D2.5mm_P7.62mm_Horizontal.wrl"
       (offset (xyz 0 0 0))
@@
       (net 11 "Net-(R1-Pad2)") (pinfunction "-") (pintype "input"))
     (pad "3" thru_hole oval locked (at 0 5.08) (size 1.6 1.6) (drill 0.8) (layers *.Cu *.Mask)
-      (net 12 "Net-(R2-Pad2)") (pinfunction "+") (pintype "input"))
+      (net 12 "Net-(R11-Pad1)") (pinfunction "+") (pintype "input"))
     (pad "4" thru_hole oval locked (at 0 7.62) (size 1.6 1.6) (drill 0.8) (layers *.Cu *.Mask)
       (net 1 "+12V") (pinfunction "V+") (pintype "power_in"))
@@
     (fp_circle (center 0 0) (end 1.25 0) (layer "F.Fab") (width 0.1) (fill none))
     (pad "1" thru_hole circle locked (at 0 0 180) (size 1.6 1.6) (drill 0.8) (layers *.Cu *.Mask)
-      (net 12 "Net-(R2-Pad2)") (pintype "passive"))
+      (net 12 "Net-(R11-Pad1)") (pintype "passive"))
     (pad "2" thru_hole oval locked (at 2.54 0 180) (size 1.6 1.6) (drill 0.8) (layers *.Cu *.Mask)
       (net 23 "GND") (pintype "passive"))
@@
       (net 1 "+12V") (pinfunction "V+") (pintype "power_in"))
   )
-  (gr_circle (center 87.757 60.96) (end 90.68076 60.96) (layer "Dwgs.User") (width 0.508) (fill none))
-  (gr_circle (center 100.076 87.884) (end 100.643961 87.884) (layer "Dwgs.User") (width 0.1) (fill solid))
+  (gr_circle (center 100.965 88.9) (end 101.532961 88.9) (layer "Dwgs.User") (width 0.1) (fill solid))
   (gr_line (start 123.19 102.87) (end 82.55 102.87) (layer "Edge.Cuts") (width 0.1))
   (gr_line (start 123.19 21.59) (end 123.19 102.87) (layer "Edge.Cuts") (width 0.1))
@@
     (effects (font (size 1.524 1.524) (thickness 0.254)))
   )
-  (gr_text "May connect to \nexternal CV instead" (at 99.822 90.297) (layer "Cmts.User")
+  (gr_text "May connect to \nexternal CV instead" (at 99.822 91.44) (layer "Cmts.User")
     (effects (font (size 1 1) (thickness 0.15)) (justify left))
   )
@@
   (segment (start 99.06 53.34) (end 88.9 53.34) (width 0.4064) (layer "F.Cu") (net 3))
   (segment (start 99.06 88.9) (end 88.9 88.9) (width 0.4064) (layer "F.Cu") (net 3))
-  (segment (start 116.84 81.28) (end 106.68 81.28) (width 0.4064) (layer "F.Cu") (net 3))
-  (via (at 106.68 81.28) (size 0.8) (drill 0.4) (layers "F.Cu" "B.Cu") (net 3))
+  (segment (start 116.84 86.36) (end 106.68 86.36) (width 0.4064) (layer "F.Cu") (net 3))
+  (via (at 106.68 86.36) (size 0.8) (drill 0.4) (layers "F.Cu" "B.Cu") (net 3))
   (via (at 88.9 88.9) (size 0.8) (drill 0.4) (layers "F.Cu" "B.Cu") (net 3))
   (via (at 88.9 53.34) (size 0.8) (drill 0.4) (layers "F.Cu" "B.Cu") (net 3))
@@
   (segment (start 90.17 54.61) (end 90.17 87.63) (width 0.4064) (layer "In2.Cu") (net 3))
   (segment (start 90.17 87.63) (end 88.9 88.9) (width 0.4064) (layer "In2.Cu") (net 3))
-  (segment (start 99.06 88.9) (end 106.68 81.28) (width 0.4064) (layer "In4.Cu") (net 3))
+  (segment (start 104.14 86.36) (end 106.68 86.36) (width 0.4064) (layer "In4.Cu") (net 3))
+  (segment (start 101.6 88.9) (end 104.14 86.36) (width 0.4064) (layer "In4.Cu") (net 3))
+  (segment (start 99.06 88.9) (end 101.6 88.9) (width 0.4064) (layer "In4.Cu") (net 3))
   (segment (start 99.06 86.36) (end 88.9 86.36) (width 0.4064) (layer "F.Cu") (net 7))
   (via (at 99.06 86.36) (size 0.8) (drill 0.4) (layers "F.Cu" "B.Cu") (net 7))
@@
   (segment (start 116.84 60.96) (end 106.68 60.96) (width 0.4064) (layer "F.Cu") (net 23))
   (segment (start 119.38 25.36) (end 119.38 60.96) (width 0.4064) (layer "F.Cu") (net 23))
+  (segment (start 116.84 81.28) (end 106.68 81.28) (width 0.4064) (layer "F.Cu") (net 23))
   (segment (start 116.84 66.04) (end 106.68 66.04) (width 0.4064) (layer "F.Cu") (net 23))
-  (segment (start 116.84 86.36) (end 106.68 86.36) (width 0.4064) (layer "F.Cu") (net 23))
   (segment (start 119.38 95.25) (end 119.38 95.25) (width 0.4064) (layer "F.Cu") (net 23))
   (segment (start 86.36 95.25) (end 86.36 95.25) (width 0.4064) (layer "F.Cu") (net 23))
@@
   (via (at 119.38 95.25) (size 0.8) (drill 0.4) (layers "F.Cu" "B.Cu") (net 23))
   (via (at 88.9 43.18) (size 0.8) (drill 0.4) (layers "F.Cu" "B.Cu") (net 23))
-  (via (at 116.84 86.36) (size 0.8) (drill 0.4) (layers "F.Cu" "B.Cu") (net 23))
+  (via (at 116.84 81.28) (size 0.8) (drill 0.4) (layers "F.Cu" "B.Cu") (net 23))
   (via (at 86.36 43.18) (size 0.8) (drill 0.4) (layers "F.Cu" "B.Cu") (net 23))
-  (via (at 119.38 86.36) (size 0.8) (drill 0.4) (layers "F.Cu" "B.Cu") (net 23))
+  (via (at 119.38 81.28) (size 0.8) (drill 0.4) (layers "F.Cu" "B.Cu") (net 23))
   (via (at 86.36 95.25) (size 0.8) (drill 0.4) (layers "F.Cu" "B.Cu") (net 23))
   (via (at 119.38 60.96) (size 0.8) (drill 0.4) (layers "F.Cu" "B.Cu") (net 23))
@@
   (segment (start 119.38 66.04) (end 116.84 66.04) (width 0.4064) (layer "In1.Cu") (net 23))
   (segment (start 88.9 43.18) (end 86.36 43.18) (width 0.4064) (layer "In1.Cu") (net 23))
-  (segment (start 119.38 86.36) (end 116.84 86.36) (width 0.4064) (layer "In1.Cu") (net 23))
+  (segment (start 119.38 81.28) (end 116.84 81.28) (width 0.4064) (layer "In1.Cu") (net 23))
   (segment (start 116.84 60.96) (end 119.38 60.96) (width 0.4064) (layer "In1.Cu") (net 23))
   (segment (start 86.36 95.25) (end 86.995 95.885) (width 0.25) (layer "B.Cu") (net 23))
