File: modules/VCA-4/VCA-4.kicad_sch (KiCad schematic)
At the start: 58 parts, among them U2 SSI2164, U3 TL074, U4 TL074, U5 TL074, U6 TL074

Commit message: VCA-4: wip
Other:
- note added: "TODO: Fix this! CV is all wrong. See VCA-CV-2164-2.cjs TODO: Check if voltage clamping is needed."
- note removed: "TODO: Fix this! CV is all wrong. See datasheet. TODO: Check if voltage clamping is needed."
Changed lines of the file:
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@@
     (effects (font (size 1.27 1.27) (thickness 0.254) bold) (justify left bottom))
   )
-  (text "TODO: Fix this! \nCV is all wrong. See datasheet.\n\nTODO: Check if voltage clamping is needed."
+  (text "TODO: Fix this! \nCV is all wrong. See VCA-CV-2164-2.cjs\n\nTODO: Check if voltage clamping is needed."
     (at 66.04 82.55 0)
     (effects (font (size 1.27 1.27)) (justify left bottom))

Commit message: VCA-4: wip
Parts:
- added R2, R3, R52, R53: 25K5, -lmp-misc:R_Axial_DIN0207_L6.3mm_D2.5mm_P7.62mm_Horizontal, symbol -lmp:R_1%_0W166
- added R50, R51, R54, R55: 11K, -lmp-misc:R_Axial_DIN0207_L6.3mm_D2.5mm_P7.62mm_Horizontal, symbol -lmp:R_1%_0W166
- R10, R12, R30, R33: value 100K -> 150K
- R11, R29, R32, R9: value 100K -> 75K
- R13, R14, R34, R35: value 66K5 -> 60K1; DistributorPartLink https://www.mouser.ca/ProductDetail/YAGEO/MFR-25FRF52-66K5?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 -> https://www.mouser.ca/ProductDetail/71-RN55D-F-60.1K; DistributorPartNum 603-MFR-25FRF52-66K5 -> 71-RN55D-F-60.1K; Manufacturer YAGEO -> Vishay / Dale; ManufacturerPartNum MFR-25FRF52-66K5 -> RN55D6012FB14; Value2 (none) -> 1%
Connections:
- net GND: now also R50.2, R51.2, R54.2, R55.2
- removed net +2VREF: U3.10 (+), U3.12 (+), U3.3 (+), U3.5 (+)
- new net: R2.2, R50.1, U3.3 (+)
- new net: R3.2, R51.1, U3.5 (+)
- new net: R52.2, R54.1, U3.12 (+)
- new net: R53.2, R55.1, U3.10 (+)
- new net +5VREF: R2.1, R3.1, R52.1, R53.1
Other:
- note removed: "TODO: Fix this! CV is all wrong. See VCA-CV-2164-2.cjs TODO: Check if voltage clamping is needed."

Commit message: VCA-4: wip
Parts:
- U3, U4, U5, U6: footprint -lmp-misc:DIP-14_W7.62mm_LongPads -> Package_DIP:DIP-14_W7.62mm

Commit message: VCA-4: wip
Parts:
- U2: footprint -lmp-breakout:Breakout_DIP-16_W15.24mm -> -lmp-breakout:Breakout_DIP-SOIC-16_W15.24mm
Changed lines of the file:
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@@
     (property "Reference" "U2" (id 0) (at 50.8 37.6682 0))
     (property "Value" "SSI2164" (id 1) (at 50.8 39.9796 0))
-    (property "Footprint" "-lmp-breakout:Breakout_DIP-16_W15.24mm" (id 2) (at 50.8 50.8 0)
+    (property "Footprint" "-lmp-breakout:Breakout_DIP-SOIC-16_W15.24mm" (id 2) (at 50.8 50.8 0)
       (effects (font (size 1.27 1.27)) hide)
     )
@@
     (property "Reference" "U2" (id 0) (at 50.8 120.2182 0))
     (property "Value" "SSI2164" (id 1) (at 50.8 122.5296 0))
-    (property "Footprint" "-lmp-breakout:Breakout_DIP-16_W15.24mm" (id 2) (at 50.8 133.35 0)
+    (property "Footprint" "-lmp-breakout:Breakout_DIP-SOIC-16_W15.24mm" (id 2) (at 50.8 133.35 0)
       (effects (font (size 1.27 1.27)) hide)
     )
@@
     (property "Reference" "U2" (id 0) (at 181.61 37.6682 0))
     (property "Value" "SSI2164" (id 1) (at 181.61 39.9796 0))
-    (property "Footprint" "-lmp-breakout:Breakout_DIP-16_W15.24mm" (id 2) (at 181.61 50.8 0)
+    (property "Footprint" "-lmp-breakout:Breakout_DIP-SOIC-16_W15.24mm" (id 2) (at 181.61 50.8 0)
       (effects (font (size 1.27 1.27)) hide)
     )
@@
     (property "Reference" "U2" (id 0) (at 181.61 104.9782 0))
     (property "Value" "SSI2164" (id 1) (at 181.61 107.2896 0))
-    (property "Footprint" "-lmp-breakout:Breakout_DIP-16_W15.24mm" (id 2) (at 181.61 118.11 0)
+    (property "Footprint" "-lmp-breakout:Breakout_DIP-SOIC-16_W15.24mm" (id 2) (at 181.61 118.11 0)
       (effects (font (size 1.27 1.27)) hide)
     )
@@
     )
     (path "/00000000-0000-0000-0000-000061c4369e"
-      (reference "U2") (unit 1) (value "SSI2164") (footprint "-lmp-breakout:Breakout_DIP-16_W15.24mm")
+      (reference "U2") (unit 1) (value "SSI2164") (footprint "-lmp-breakout:Breakout_DIP-SOIC-16_W15.24mm")
     )
     (path "/00000000-0000-0000-0000-000061d2ef99"
-      (reference "U2") (unit 2) (value "SSI2164") (footprint "-lmp-breakout:Breakout_DIP-16_W15.24mm")
+      (reference "U2") (unit 2) (value "SSI2164") (footprint "-lmp-breakout:Breakout_DIP-SOIC-16_W15.24mm")
     )
     (path "/00000000-0000-0000-0000-000061d67dc0"
-      (reference "U2") (unit 3) (value "SSI2164") (footprint "-lmp-breakout:Breakout_DIP-16_W15.24mm")
+      (reference "U2") (unit 3) (value "SSI2164") (footprint "-lmp-breakout:Breakout_DIP-SOIC-16_W15.24mm")
     )
     (path "/00000000-0000-0000-0000-000061f3ffd3"
-      (reference "U2") (unit 4) (value "SSI2164") (footprint "-lmp-breakout:Breakout_DIP-16_W15.24mm")
+      (reference "U2") (unit 4) (value "SSI2164") (footprint "-lmp-breakout:Breakout_DIP-SOIC-16_W15.24mm")
     )
     (path "/00000000-0000-0000-0000-000061c69b4e/00000000-0000-0000-0000-000061c656ef"
-      (reference "U2") (unit 5) (value "SSI2164") (footprint "-lmp-breakout:Breakout_DIP-16_W15.24mm")
+      (reference "U2") (unit 5) (value "SSI2164") (footprint "-lmp-breakout:Breakout_DIP-SOIC-16_W15.24mm")
     )
     (path "/00000000-0000-0000-0000-000061cdcc6f"

Commit message: VCA-4: Better explamation of normallling
Other:
- note added: "If a channel's output is not patched, it is normalled to mix with the next channel's output."
- note added: "When channel 1's output is normalled to channel 2, it must be inverted before mixing into the last inverting stage."
- note removed: "If a channel's output is not patched, it is normalled to mix with the next channel."
Changed lines of the file:
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@@
     (stroke (width 0) (type default) (color 0 0 0 0))
+  )
+  (text "When channel 1's output is normalled to channel 2, \nit must be inverted before mixing into the last \ninverting stage."
+    (at 68.58 182.88 0)
+    (effects (font (size 1.27 1.27)) (justify left bottom))
   )
   (text "Power & Stuff" (at 304.8 72.39 0)
@@
     (effects (font (size 1.27 1.27) (thickness 0.254) bold) (justify left bottom))
   )
-  (text "If a channel's output is not patched, \nit is normalled to mix with the next channel."
-    (at 85.09 67.31 0)
+  (text "If a channel's output is not patched, it is \nnormalled to mix with the next channel's output."
+    (at 83.82 67.31 0)
     (effects (font (size 1.27 1.27)) (justify left bottom))
   )

Commit message: VCA-4: BOM cleanup
Parts:
- R10, R12, R30, R33: DistributorPartLink https://www.mouser.ca/c/?m=YAGEO&power+rating=166+mW+(1%2f6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 -> https://www.mouser.ca/ProductDetail/YAGEO/MFR-12FTF52-150K?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; DistributorPartNum 603-MFR-12* -> 603-MFR-12FTF52-150K; ManufacturerPartNum MFR-12* -> MFR-12FTF52-150K
- R11, R29, R32, R9: DistributorPartLink https://www.mouser.ca/c/?m=YAGEO&power+rating=166+mW+(1%2f6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 -> https://www.mouser.ca/ProductDetail/YAGEO/MFR-12FTF52-75K?q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; DistributorPartNum 603-MFR-12* -> 603-MFR-12FTF52-75K; ManufacturerPartNum MFR-12* -> MFR-12FTF52-75K
- R15, R16, R36, R37: DistributorPartLink https://www.mouser.ca/c/?m=YAGEO&power+rating=166+mW+(1%2f6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 -> https://www.mouser.ca/ProductDetail/YAGEO/MFR-12FTF52-20K?q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; DistributorPartNum 603-MFR-12* -> 603-MFR-12FTF52-20K; ManufacturerPartNum MFR-12* -> MFR-12FTF52-20K
- R2, R3, R52, R53: DistributorPartLink https://www.mouser.ca/c/?m=YAGEO&power+rating=166+mW+(1%2f6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 -> https://www.mouser.ca/ProductDetail/603-MFR-25FRF52-25K5; DistributorPartNum 603-MFR-12* -> 603-MFR-25FRF52-25K5; ManufacturerPartNum MFR-12* -> MFR-25FRF52-25K5
- R50, R51, R54, R55: DistributorPartLink https://www.mouser.ca/c/?m=YAGEO&power+rating=166+mW+(1%2f6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 -> https://www.mouser.ca/ProductDetail/YAGEO/MFR-12FTF52-11K?q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; DistributorPartNum 603-MFR-12* -> 603-MFR-12FTF52-11K; ManufacturerPartNum MFR-12* -> MFR-12FTF52-11K
