File: modules/VCA-4/Controls.kicad_sch (KiCad schematic)
At the start: 26 parts, among them J1 WQP-PJ398, J10 WQP-PJ398, J11 WQP-PJ398, J12 WQP-PJ398, J13 Conn_Socket_24, J14 Conn_Header_24, J15 Conn_Socket_24, J16 Conn_Header_24, J18 Conn_Socket_4, J19 Conn_Header_4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

Commit message: VCA-4: wip
Connections:
- net +5VREF: no longer J1.TN
- net GND: now also J1.TN
Other:
- note removed: "TODO: IN-CV-1 normal GND"
- note removed: "TODO: change CV pots to Song Huei"

Commit message: VCA-4: Better explamation of normallling
Other:
- note added: "Each CV input is normalled to the next one. Each output is normalled to mix with the next one."
- moved on the sheet: J1, J10, J11, J12, J2, J3, J4, J5, J6, J7, J8, J9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

Commit message: VCA-4: BOM cleanup
Parts:
- RV1, RV3, RV5, RV7: DistributorPartLink2 https://www.mouser.ca/c/passive-components/potentiometers-t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 -> https://www.mouser.ca/ProductDetail/Alpha-Taiwan/RD901F-40-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; DistributorPartNum2 311-1940F-* -> 311-1940F-15R1-B100K; ManufacturerPartNum RD901F-* -> RD901F-40-15R1-B100K-00DL1
- RV2, RV4, RV6, RV8: Distributor2 Mouser -> Thonk; Distributor3 SynthCube -> (none); DistributorPartLink2 https://www.mouser.ca/c/passive-components/potentiometers-t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 -> https://www.thonk.co.uk/shop/ttpots/; DistributorPartLink3 https://synthcube.com/cart/alpha-9mm-potentiometer-right-an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 -> (none); DistributorPartNum2 311-1940F-* -> Group_SongHuei_TTP; DistributorPartNum3 9MMALPHAPOTMSTR -> (none)

Commit message: VCA-4: Fix pot footprints
Parts:
- RV2: footprint -lmp-synth:Potentiometer_Alpha_RD901F-40-00D_Single_Vertical -> -lmp-synth:Potentiometer_SongHuei_Single_Vertical; Label CV-ATTEN-1 -> CV-AMT-1
- RV4: footprint -lmp-synth:Potentiometer_Alpha_RD901F-40-00D_Single_Vertical -> -lmp-synth:Potentiometer_SongHuei_Single_Vertical; Label CV-ATTEN-2 -> CV-AMT-2
- RV6: footprint -lmp-synth:Potentiometer_Alpha_RD901F-40-00D_Single_Vertical -> -lmp-synth:Potentiometer_SongHuei_Single_Vertical; Label CV-ATTEN-3 -> CV-AMT-3
- RV8: footprint -lmp-synth:Potentiometer_Alpha_RD901F-40-00D_Single_Vertical -> -lmp-synth:Potentiometer_SongHuei_Single_Vertical; Label CV-ATTEN-4 -> CV-AMT-4

Commit message: VCA-4: schematic tweaks
Parts:
- RV2: Label CV-AMT-1 -> [label]; Value2 LIN -> [LIN/LOG]
- RV4: Label CV-AMT-2 -> [label]; Value2 LIN -> [LIN/LOG]
- RV6: Label CV-AMT-3 -> [label]; Value2 LIN -> [LIN/LOG]
- RV8: Label CV-AMT-4 -> [label]; Value2 LIN -> [LIN/LOG]
Other:
- title: Controls & Connectors - Eurorack 4XVCA Module -> Power & Hardware - Eurorack 4XVCA Module
- moved on the sheet: J1, J10, J11, J12, J14, J15, J18, J19, J2, J3, J4, J5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
Changed lines of the file:
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@@
   (paper "A4")
   (title_block
-    (title "Controls & Connectors - Eurorack 4XVCA Module")
+    (title "Power & Hardware - Eurorack 4XVCA Module")
     (date "2021-12-24")
     (rev "1.0")

Commit message: VCA-4: schematic tweaks
Parts:
- RV2: Label [label] -> CV-AMT-1; Value2 [LIN/LOG] -> LIN
- RV4: Label [label] -> CV-AMT-2; Value2 [LIN/LOG] -> LIN
- RV6: Label [label] -> CV-AMT-3; Value2 [LIN/LOG] -> LIN
- RV8: Label [label] -> CV-AMT-4; Value2 [LIN/LOG] -> LIN

Commit message: VCA-4: BOM update
Parts:
- J13, J15, J18: Distributor (none) -> Adafruit; Distributor2 (none) -> Mouser; DistributorPartLink (none) -> https://www.adafruit.com/product/598; DistributorPartLink2 (none) -> https://www.mouser.ca/ProductDetail/Wurth-Elektronik/613032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; DistributorPartNum (none) -> 598; DistributorPartNum2 (none) -> 710-61303211821
- J14, J16, J19: Distributor (none) -> Adafruit; Distributor2 (none) -> Mouser; DistributorPartLink (none) -> https://www.adafruit.com/product/392; DistributorPartLink2 (none) -> https://www.mouser.ca/ProductDetail/649-1012937893601BLF; DistributorPartNum (none) -> 392; DistributorPartNum2 (none) -> 649-1012937893601BLF
