File: modules/Audiout/PanelPower.kicad_sch (KiCad schematic)
At the start: 21 parts, among them J1 WQP-PJ398, J2 WQP-PJ398, J3 WQP419GR, J4 WQP419GR, J5 WQP419GR, J6 Conn_Front, J7 Conn_Rear, J8 Conn_Eurorack_16, U2 TL072, U3 TL074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

Commit message: Audiout: Correct footprints in schematic
Parts:
- U2: footprint -lmp-misc:DIP-8_W7.62mm_LongPads -> Package_DIP:DIP-8_W7.62mm
- U3: footprint -lmp-misc:DIP-14_W7.62mm_LongPads -> Package_DIP:DIP-14_W7.62mm
- U4: footprint -lmp-breakout:Breakout_DIP-8_W7.62mm -> -lmp-breakout:Breakout_DIP-SOIC-8_W7.62mm
Changed lines of the file:
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@@
       (effects (font (size 1.27 1.27)) (justify left))
     )
-    (property "Footprint" "-lmp-misc:DIP-14_W7.62mm_LongPads" (id 2) (at 250.19 48.26 0)
+    (property "Footprint" "Package_DIP:DIP-14_W7.62mm" (id 2) (at 250.19 48.26 0)
       (effects (font (size 1.27 1.27)) hide)
     )
@@
       (effects (font (size 1.27 1.27)) (justify left))
     )
-    (property "Footprint" "-lmp-breakout:Breakout_DIP-8_W7.62mm" (id 2) (at 205.74 85.09 0)
+    (property "Footprint" "-lmp-breakout:Breakout_DIP-SOIC-8_W7.62mm" (id 2) (at 205.74 85.09 0)
       (effects (font (size 1.27 1.27)) hide)
     )
@@
       (effects (font (size 1.27 1.27)) (justify left))
     )
-    (property "Footprint" "-lmp-misc:DIP-8_W7.62mm_LongPads" (id 2) (at 226.06 50.8 0)
-      (effects (font (size 1.27 1.27)) hide)
-    )
+    (property "Footprint" "Package_DIP:DIP-8_W7.62mm" (id 2) (at 226.06 50.8 0)
+      (effects (font (size 1.27 1.27)) hide)
+    )

Commit message: Audiout: BOM stuff
Other:
- note added: "TODO: connector properties for BOM"
Changed lines of the file:
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@@
     (effects (font (size 1.27 1.27) (thickness 0.254) bold) (justify left bottom))
+  )
+  (text "TODO: connector properties for BOM" (at 100.33 33.02 0)
+    (effects (font (size 1.27 1.27)) (justify left bottom))
   )
   (text "+" (at 43.18 137.16 0)

Commit message: Audiout: Improvements to input stage
Other:
- title: Controls, Connectors & Power - Eurorack Audiout Module -> Main - Eurorack Audiout Module
Changed lines of the file:
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@@
   (paper "A4")
   (title_block
-    (title "Controls, Connectors & Power - Eurorack Audiout Module")
+    (title "Main - Eurorack Audiout Module")
     (date "2021-11-30")
     (rev "1.2")
