File: modules/Audiout/Audiout.kicad_sch (KiCad schematic)
At the start: 36 parts, among them U2 TL072, U3 TL074, U4 LM4808

Commit message: Audiout: note for future self
Other:
- note added: "TODO: Verify all footprints & part nums"
Changed lines of the file:
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@@
+    (effects (font (size 1.27 1.27)) (justify left bottom))
+  )
+  (text "TODO: Verify all footprints & part nums" (at 208.28 45.72 0)
     (effects (font (size 1.27 1.27)) (justify left bottom))
   )

Commit message: Audiout: change input coupling caps
Parts:
- C10, C9: value 470N -> 1U; footprint -lmp-misc:C_Rect_Kemet_L7.2mm_W2.5mm_P5mm -> -lmp-misc:C_Rect_L7.2mm_W4.5mm_P5.00mm; DistributorPartLink https://www.mouser.ca/ProductDetail/?qs=Jv4FAWB%252B0HZ72wF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 -> https://www.mouser.ca/ProductDetail/KEMET/R82DC4100AA60K?qs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; DistributorPartNum 80-R82DC3470SH60J -> 80-R82DC4100AA60K; ManufacturerPartNum R82DC3470SH60J -> R82DC4100AA60K
Changed lines of the file:
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@@
     (in_bom yes) (on_board yes)
     (property "Reference" "C9" (id 0) (at 35.56 31.6992 90))
-    (property "Value" "470N" (id 1) (at 35.56 34.0106 90))
-    (property "Footprint" "-lmp-misc:C_Rect_Kemet_L7.2mm_W2.5mm_P5mm" (id 2) (at 31.75 39.0652 0)
+    (property "Value" "1U" (id 1) (at 35.56 34.0106 90))
+    (property "Footprint" "-lmp-misc:C_Rect_L7.2mm_W4.5mm_P5.00mm" (id 2) (at 31.75 39.0652 0)
       (effects (font (size 1.27 1.27)) hide)
     )
@@
       (effects (font (size 1.27 1.27)) hide)
     )
-    (property "Value2" "" (id 4) (at 35.56 34.036 90))
+    (property "Value2" "" (id 4) (at 35.56 34.036 90)
+      (effects (font (size 1.27 1.27)) hide)
+    )
     (property "Distributor" "Mouser" (id 5) (at 35.56 38.1 0)
       (effects (font (size 1.27 1.27)) hide)
@@
       (effects (font (size 1.27 1.27)) hide)
     )
-    (property "ManufacturerPartNum" "R82DC3470SH60J" (id 7) (at 35.56 38.1 0)
-      (effects (font (size 1.27 1.27)) hide)
-    )
-    (property "DistributorPartNum" "80-R82DC3470SH60J" (id 8) (at 35.56 38.1 0)
-      (effects (font (size 1.27 1.27)) hide)
-    )
-    (property "DistributorPartLink" "https://www.mouser.ca/ProductDetail/?qs=Jv4FAWB%252B0HZ72wFOzKdj%2Fw%3D%3D" (id 9) (at 35.56 38.1 0)
+    (property "ManufacturerPartNum" "R82DC4100AA60K" (id 7) (at 35.56 38.1 0)
+      (effects (font (size 1.27 1.27)) hide)
+    )
+    (property "DistributorPartNum" "80-R82DC4100AA60K" (id 8) (at 35.56 38.1 0)
+      (effects (font (size 1.27 1.27)) hide)
+    )
+    (property "DistributorPartLink" "https://www.mouser.ca/ProductDetail/KEMET/R82DC4100AA60K?qs=Jv4FAWB%252B0HY7sWoVYON7mg%3D%3D" (id 9) (at 35.56 38.1 0)
       (effects (font (size 1.27 1.27)) hide)
     )
@@
     (in_bom yes) (on_board yes)
     (property "Reference" "C10" (id 0) (at 35.56 116.7892 90))
-    (property "Value" "470N" (id 1) (at 35.56 119.1006 90))
-    (property "Footprint" "-lmp-misc:C_Rect_Kemet_L7.2mm_W2.5mm_P5mm" (id 2) (at 31.75 124.1552 0)
+    (property "Value" "1U" (id 1) (at 35.56 119.1006 90))
+    (property "Footprint" "-lmp-misc:C_Rect_L7.2mm_W4.5mm_P5.00mm" (id 2) (at 31.75 124.1552 0)
       (effects (font (size 1.27 1.27)) hide)
     )
@@
       (effects (font (size 1.27 1.27)) hide)
     )
-    (property "ManufacturerPartNum" "R82DC3470SH60J" (id 6) (at 35.56 123.19 0)
+    (property "ManufacturerPartNum" "R82DC4100AA60K" (id 6) (at 35.56 123.19 0)
       (effects (font (size 1.27 1.27)) hide)
     )
@@
       (effects (font (size 1.27 1.27)) hide)
     )
-    (property "DistributorPartNum" "80-R82DC3470SH60J" (id 8) (at 35.56 123.19 0)
-      (effects (font (size 1.27 1.27)) hide)
-    )
-    (property "DistributorPartLink" "https://www.mouser.ca/ProductDetail/?qs=Jv4FAWB%252B0HZ72wFOzKdj%2Fw%3D%3D" (id 9) (at 35.56 123.19 0)
+    (property "DistributorPartNum" "80-R82DC4100AA60K" (id 8) (at 35.56 123.19 0)
+      (effects (font (size 1.27 1.27)) hide)
+    )
+    (property "DistributorPartLink" "https://www.mouser.ca/ProductDetail/KEMET/R82DC4100AA60K?qs=Jv4FAWB%252B0HY7sWoVYON7mg%3D%3D" (id 9) (at 35.56 123.19 0)
       (effects (font (size 1.27 1.27)) hide)
     )
@@
     )
     (path "/00000000-0000-0000-0000-000060e495f8"
-      (reference "C9") (unit 1) (value "470N") (footprint "-lmp-misc:C_Rect_Kemet_L7.2mm_W2.5mm_P5mm")
+      (reference "C9") (unit 1) (value "1U") (footprint "-lmp-misc:C_Rect_L7.2mm_W4.5mm_P5.00mm")
     )
     (path "/00000000-0000-0000-0000-000060f459b0"
-      (reference "C10") (unit 1) (value "470N") (footprint "-lmp-misc:C_Rect_Kemet_L7.2mm_W2.5mm_P5mm")
+      (reference "C10") (unit 1) (value "1U") (footprint "-lmp-misc:C_Rect_L7.2mm_W4.5mm_P5.00mm")
     )
     (path "/00000000-0000-0000-0000-000060e6d9a4"

Commit message: Audiout: add a note
Other:
- note added: "TODO: 10U input caps??"
Changed lines of the file:
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@@
+    (effects (font (size 1.27 1.27)) (justify left bottom))
+  )
+  (text "TODO: 10U input caps??" (at 20.32 67.31 0)
     (effects (font (size 1.27 1.27)) (justify left bottom))
   )

Commit message: Audiout: add a note
Other:
- note added: "TODO: 10U input caps?? and put after op-amp? See Befaco Outv3"
- note removed: "TODO: 10U input caps??"
Changed lines of the file:
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@@
     (effects (font (size 1.27 1.27)) (justify left bottom))
   )
-  (text "TODO: 10U input caps??" (at 20.32 67.31 0)
+  (text "TODO: 10U input caps??\nand put after op-amp?\nSee Befaco Outv3"
+    (at 20.32 69.85 0)
     (effects (font (size 1.27 1.27)) (justify left bottom))
   )

Commit message: Audiout: Improvements to input stage
Parts:
- added C11, C12: 47P, -lmp-misc:C_Disc_D5.0mm_W2.5mm_P2.50mm, symbol -lmp:CC
- added R11, R12: 100K, -lmp-misc:R_Axial_DIN0207_L6.3mm_D2.5mm_P7.62mm_Horizontal, symbol -lmp:R
- C10, C9: value 1U -> 10U; footprint -lmp-misc:C_Rect_L7.2mm_W4.5mm_P5.00mm -> -lmp-misc:C_Radial_D5.0mm_H5.0mm_P2.50mm; symbol -lmp:CF -> -lmp-synth:CNP_10U; DistributorPartLink https://www.mouser.ca/ProductDetail/KEMET/R82DC4100AA60K?qs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 -> https://www.mouser.ca/ProductDetail/Panasonic/ECE-A1EN100UI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; DistributorPartNum 80-R82DC4100AA60K -> 667-ECE-A1EN100UI; Manufacturer KEMET -> Panasonic; ManufacturerPartNum R82DC4100AA60K -> ECE-A1EN100UI; Value2 (none) -> NPE
- C15: Distributor (none) -> Mouser; DistributorPartLink (none) -> https://www.mouser.ca/ProductDetail/Rubycon/50YXJ1M5X11?qs=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; DistributorPartNum (none) -> 232-50YXJ1M5X11; Manufacturer (none) -> Rubycon; ManufacturerPartNum (none) -> 50YXJ1M5X11
- R1, R2: value 100K -> 150K; Distributor (none) -> Mouser; DistributorPartLink (none) -> https://www.mouser.ca/ProductDetail/YAGEO/MFR-12FTF52-150K?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; DistributorPartNum (none) -> 603-MFR-12FTF52-150K; Manufacturer (none) -> YAGEO; ManufacturerPartNum (none) -> MFR-12FTF52-150K
- R19, R20: Distributor (none) -> Mouser; DistributorPartLink (none) -> https://www.mouser.ca/ProductDetail/603-MFR-12FTF52-100K; DistributorPartNum (none) -> 603-MFR-12FTF52-100K; Manufacturer (none) -> YAGEO; ManufacturerPartNum (none) -> MFR-12FTF52-100K
- R29, R30, R31, R32, R5, R6, R7, R8: Distributor (none) -> Mouser; DistributorPartLink (none) -> https://www.mouser.ca/ProductDetail/YAGEO/MFR-12FRF52-10K?q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; DistributorPartNum (none) -> 603-MFR-12FRF5210K; Manufacturer (none) -> YAGEO; ManufacturerPartNum (none) -> MFR-12FRF52-10K
- R3, R4: value 100K -> 47K; Distributor (none) -> Mouser; DistributorPartLink (none) -> https://www.mouser.ca/ProductDetail/YAGEO/MFR-12FTF52-47K?q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; DistributorPartNum (none) -> 603-MFR-12FTF52-47K; Manufacturer (none) -> YAGEO; ManufacturerPartNum (none) -> MFR-12FTF52-47K
Connections:
- net GND: now also R11.2, R12.2
- net IN-LEFT: now also R11.1
- net IN-RIGHT: now also R12.1
- net PHONES-LEFT: now also C11.1
- net PHONES-RIGHT: now also C12.1
- net at R1.1, R3.2, U2.2 (-): now also C11.2
- net at R2.1, R4.2, U2.6 (-): now also C12.2
Other:
- note added: "Change input & feedback resistors to adjust max gain"
- note removed: "TODO: 10U input caps?? and put after op-amp? See Befaco Outv3"
- moved on the sheet: C10, C15, C16, C17, C18, C19, C9, R1, R10, R15, R16, R17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

Commit message: Audiout: Update the PCB
Parts:
- C15: footprint -lmp-misc:CP_Radial_D4.0mm_P2.50mm -> Capacitor_THT:CP_Radial_D5.0mm_P2.00mm
- C18, C19: footprint Capacitor_THT:CP_Radial_D8.0mm_P5.00mm -> Capacitor_THT:CP_Radial_D8.0mm_P3.50mm
Other:
- note removed: "TODO: Verify all footprints & part nums"
Changed lines of the file:
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@@
-    (effects (font (size 1.27 1.27)) (justify left bottom))
-  )
-  (text "TODO: Verify all footprints & part nums" (at 208.28 48.26 0)
     (effects (font (size 1.27 1.27)) (justify left bottom))
   )
@@
       (effects (font (size 1.27 1.27)) (justify left))
     )
-    (property "Footprint" "-lmp-misc:CP_Radial_D4.0mm_P2.50mm" (id 2) (at 187.6552 115.57 0)
+    (property "Footprint" "Capacitor_THT:CP_Radial_D5.0mm_P2.00mm" (id 2) (at 187.6552 115.57 0)
       (effects (font (size 1.27 1.27)) hide)
     )
@@
     (property "Reference" "C18" (id 0) (at 224.79 83.693 90))
     (property "Value" "220U" (id 1) (at 224.79 86.0044 90))
-    (property "Footprint" "Capacitor_THT:CP_Radial_D8.0mm_P5.00mm" (id 2) (at 228.6 89.2048 0)
+    (property "Footprint" "Capacitor_THT:CP_Radial_D8.0mm_P3.50mm" (id 2) (at 228.6 89.2048 0)
       (effects (font (size 1.27 1.27)) hide)
     )
@@
     (property "Reference" "C19" (id 0) (at 224.79 116.713 90))
     (property "Value" "220U" (id 1) (at 224.79 119.0244 90))
-    (property "Footprint" "Capacitor_THT:CP_Radial_D8.0mm_P5.00mm" (id 2) (at 228.6 122.2248 0)
+    (property "Footprint" "Capacitor_THT:CP_Radial_D8.0mm_P3.50mm" (id 2) (at 228.6 122.2248 0)
       (effects (font (size 1.27 1.27)) hide)
     )
@@
     )
     (path "/00000000-0000-0000-0000-000060e6d9a4"
-      (reference "C15") (unit 1) (value "1U") (footprint "-lmp-misc:CP_Radial_D4.0mm_P2.50mm")
+      (reference "C15") (unit 1) (value "1U") (footprint "Capacitor_THT:CP_Radial_D5.0mm_P2.00mm")
     )
     (path "/00000000-0000-0000-0000-000060e7790f"
@@
     )
     (path "/00000000-0000-0000-0000-000060e73a2b"
-      (reference "C18") (unit 1) (value "220U") (footprint "Capacitor_THT:CP_Radial_D8.0mm_P5.00mm")
+      (reference "C18") (unit 1) (value "220U") (footprint "Capacitor_THT:CP_Radial_D8.0mm_P3.50mm")
     )
     (path "/00000000-0000-0000-0000-000060e931cd"
-      (reference "C19") (unit 1) (value "220U") (footprint "Capacitor_THT:CP_Radial_D8.0mm_P5.00mm")
+      (reference "C19") (unit 1) (value "220U") (footprint "Capacitor_THT:CP_Radial_D8.0mm_P3.50mm")
     )
     (path "/00000000-0000-0000-0000-000060cbfb6a/00000000-0000-0000-0000-000060cb8a0c"
