File: modules/Audiout/prototype/prototype.kicad_pcb (KiCad board)
At the start: 6 copper layers, 40.6 x 78.7 mm, 14 parts, among them J1 Conn_01x09, U1 TL074

Commit message: Audiout: Prototype tweaking
Parts:
- C1: value 470N -> 1U
- R10, R9: value 1K -> 100R; footprint -lmp-misc:R_Axial_DIN0207_L6.3mm_D2.5mm_P7.62mm_Horizontal -> -lmp-misc:R_Axial_DIN0207_L6.3mm_D2.5mm_P10.16mm_Horizontal

Commit message: Audiout: Prototype updated after testing
Parts:
- added C2: 47P, -lmp-misc:C_Disc_D5.0mm_W2.5mm_P2.50mm, F.Cu at (94.0, 61.0)
- added R11: 100K, -lmp-stripboard:SB_Gen_1, F.Cu at (86.4, 50.8)
- C1: value 1U -> 10U; footprint -lmp-misc:C_Rect_Kemet_L7.2mm_W2.5mm_P5mm -> -lmp-misc:C_Radial_D5.0mm_H5.0mm_P2.50mm
- R1: value 100K -> 150K
- R2: value 100K -> 47K
- moved R2 2.54 mm to (96.5, 63.5)
- moved C1 1.27 mm to (99.1, 52.1)
Routing:
- net IN-OUT-1: track 63.3 -> 64.6 mm
- net Net-(C1-Pad2): track 10.2 -> 11.4 mm, vias 0 -> 1
