File: modules/Mixer2/prototype1/prototype.kicad_pcb (KiCad board)
At the start: 6 copper layers, 40.6 x 78.7 mm, 25 parts, among them J1 Conn_01x09, U1 TL074, U2 TL071

Commit message: Mixer2 - prototype - wip
Parts:
- D3: footprint Diode_THT:D_DO-35_SOD27_P7.62mm_Horizontal -> -lmp-stripboard:SB_Gen_1
- R1: footprint -lmp-misc:R_Axial_DIN0207_L6.3mm_D2.5mm_P7.62mm_Horizontal -> -lmp-stripboard:SB_Gen_2
- R10, R4, R8: footprint -lmp-misc:R_Axial_DIN0207_L6.3mm_D2.5mm_P7.62mm_Horizontal -> -lmp-stripboard:SB_Gen_1
- R9: footprint -lmp-misc:R_Axial_DIN0207_L6.3mm_D2.5mm_P10.16mm_Horizontal -> -lmp-stripboard:SB_Gen_1
- moved R13 60.5 mm to (96.5, 43.2), turned to -90 degrees
- moved C3 57.1 mm to (88.9, 66.0), turned to 180 degrees
- moved D2 53.9 mm to (91.4, 66.0), turned to 90 degrees
- moved R1 53.7 mm to (83.8, 68.6)
- moved R2 50.4 mm to (94.0, 68.6), turned to 90 degrees
- moved D4 48.1 mm to (91.4, 55.9), turned to 90 degrees
- moved R11 43.6 mm to (96.5, 63.5), turned to 90 degrees
- moved D3 42.3 mm to (99.1, 51.0), turned to -90 degrees
- moved C2 36.1 mm to (109.2, 76.2), turned to -90 degrees
- moved R12 35.9 mm to (111.1, 63.5), turned to 90 degrees
- moved R10 33.0 mm to (119.4, 68.6), turned to 180 degrees
- moved R8 28.3 mm to (111.8, 76.2), turned to -90 degrees
- moved R3 27.2 mm to (109.2, 58.4), turned to -90 degrees
- moved D1 23.6 mm to (113.7, 68.6), turned to 90 degrees
- moved R9 22.5 mm to (114.3, 78.7), turned to -90 degrees
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Routing:
- net (no net): track 284.5 -> 193.0 mm
- net Net-(D2-Pad2): track 10.2 -> 57.8 mm, vias 0 -> 2
- net Net-(C3-Pad1): track 30.5 -> 73.9 mm, vias 0 -> 4
- net VREF-4: track 10.2 -> 51.6 mm, vias 0 -> 4
- net Net-(C2-Pad2): track 10.2 -> 39.1 mm, vias 0 -> 2
- net Net-(D4-Pad1): track 0.00 -> 27.9 mm, vias 0 -> 2
- net OUTPUT: track 3.17 -> 29.2 mm, vias 0 -> 1
- net GND: track 216.0 -> 238.9 mm, vias 8 -> 12
- net Net-(C1-Pad2): track 20.3 -> 37.8 mm, vias 0 -> 2
- net INPUT: track 13.3 -> 28.7 mm, vias 0 -> 1
- net +12V: track 110.5 -> 120.7 mm, vias 3 -> 5
- net Net-(D3-Pad1): track 0.00 -> 10.2 mm
- net -12V: track 101.1 -> 111.3 mm, vias 3 -> 5
Other:
- board text added: "1"
- board text added: "10"
- board text added: "15"
- board text added: "20"
- board text added: "25"
- board text added: "5"

Commit message: Mixer2 - change prototype1
Parts:
- U2: value TL071 -> TL072
- moved R13 12.7 mm to (106.7, 50.8), turned to 180 degrees
- moved D3 2.54 mm to (96.5, 51.0)
Connections:
- U2 pad 1: unconnected-(U2-Pad1) -> Net-(R13-Pad1)
- U2 pad 6: Net-(R13-Pad1) -> unconnected-(U2-Pad6)
- U2 pad 7: +12V -> unconnected-(U2-Pad7)
- U2 pad 8: unconnected-(U2-Pad8) -> +12V
Routing:
- net Net-(R13-Pad1): track 10.2 -> 22.9 mm, vias 0 -> 2
- net unconnected-(U2-Pad8): track 10.2 -> 0.00 mm
- net unconnected-(U2-Pad7): track 0.00 -> 10.2 mm
- net unconnected-(U2-Pad6): track 0.00 -> 10.2 mm
- net unconnected-(U2-Pad1): track 10.2 -> 0.00 mm
- net (no net): track 193.0 -> 182.9 mm

Commit message: Mixer2 - prototype1
Parts:
- moved RV1 5.08 mm to (96.5, 86.4), turned to -90 degrees
Routing:
- net INPUT: track 28.7 -> 34.8 mm
- net Net-(D2-Pad2): track 57.8 -> 60.4 mm
Changed lines of the file:
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@@
   )
   (footprint "-lmp-misc:Potentiometer_Bourns_3386P_Top" (layer "F.Cu")
-    (at 96.52 91.44 90)
+    (at 96.52 86.36 -90)
     (descr "3386P-EY5-202LF-1")
     (tags "Variable Resistor")
@@
     (fp_line (start -2.225 -4.78) (end 7.305 -4.78) (layer "F.Fab") (width 0.2))
     (fp_line (start -2.225 4.75) (end -2.225 -4.78) (layer "F.Fab") (width 0.2))
-    (pad "1" thru_hole circle locked (at 0 0 90) (size 1.303 1.303) (drill 0.76) (layers *.Cu *.Mask)
+    (pad "1" thru_hole circle locked (at 0 0 270) (size 1.303 1.303) (drill 0.76) (layers *.Cu *.Mask)
       (net 15 "INPUT") (pinfunction "1") (pintype "passive"))
-    (pad "2" thru_hole circle locked (at 2.54 2.54 90) (size 1.303 1.303) (drill 0.76) (layers *.Cu *.Mask)
+    (pad "2" thru_hole circle locked (at 2.54 2.54 270) (size 1.303 1.303) (drill 0.76) (layers *.Cu *.Mask)
       (net 21 "Net-(R5-Pad1)") (pinfunction "2") (pintype "passive"))
-    (pad "3" thru_hole circle locked (at 5.08 0 90) (size 1.303 1.303) (drill 0.76) (layers *.Cu *.Mask)
+    (pad "3" thru_hole circle locked (at 5.08 0 270) (size 1.303 1.303) (drill 0.76) (layers *.Cu *.Mask)
       (net 2 "GND") (pinfunction "3") (pintype "passive"))
     (model "C:\\Users\\Len\\OneDrive\\Documents\\Electronics\\KiCad\\download\\SamacSys_Parts.3dshapes\\3386P-EY5-202LF.stp"
@@
   (segment (start 84.219999 95.649999) (end 83.82 95.25) (width 0.25) (layer "B.Cu") (net 1))
   (segment (start 86.36 25.4) (end 86.36 53.34) (width 0.4064) (layer "F.Cu") (net 2))
-  (segment (start 99.06 86.36) (end 88.9 86.36) (width 0.4064) (layer "F.Cu") (net 2))
   (segment (start 116.84 73.66) (end 106.68 73.66) (width 0.4064) (layer "F.Cu") (net 2))
+  (segment (start 99.06 91.44) (end 88.9 91.44) (width 0.4064) (layer "F.Cu") (net 2))
   (segment (start 99.06 73.66) (end 88.9 73.66) (width 0.4064) (layer "F.Cu") (net 2))
   (segment (start 99.06 53.34) (end 88.9 53.34) (width 0.4064) (layer "F.Cu") (net 2))
@@
   (via (at 86.36 73.66) (size 0.8) (drill 0.4) (layers "F.Cu" "B.Cu") (net 2))
   (via (at 86.36 95.25) (size 0.8) (drill 0.4) (layers "F.Cu" "B.Cu") (net 2))
+  (via (at 88.9 91.44) (size 0.8) (drill 0.4) (layers "F.Cu" "B.Cu") (net 2))
   (via (at 119.38 91.44) (size 0.8) (drill 0.4) (layers "F.Cu" "B.Cu") (net 2))
-  (via (at 88.9 86.36) (size 0.8) (drill 0.4) (layers "F.Cu" "B.Cu") (net 2))
   (via (at 88.9 53.34) (size 0.8) (drill 0.4) (layers "F.Cu" "B.Cu") (net 2))
-  (via (at 86.36 86.36) (size 0.8) (drill 0.4) (layers "F.Cu" "B.Cu") (net 2))
+  (via (at 86.36 91.44) (size 0.8) (drill 0.4) (layers "F.Cu" "B.Cu") (net 2))
   (segment (start 116.84 73.66) (end 119.38 73.66) (width 0.4064) (layer "In1.Cu") (net 2))
-  (segment (start 88.9 86.36) (end 86.36 86.36) (width 0.4064) (layer "In1.Cu") (net 2))
   (segment (start 88.9 73.66) (end 86.36 73.66) (width 0.4064) (layer "In1.Cu") (net 2))
   (segment (start 86.36 53.34) (end 88.9 53.34) (width 0.4064) (layer "In1.Cu") (net 2))
   (segment (start 116.84 91.44) (end 119.38 91.44) (width 0.4064) (layer "In1.Cu") (net 2))
+  (segment (start 88.9 91.44) (end 86.36 91.44) (width 0.4064) (layer "In1.Cu") (net 2))
   (segment (start 86.36 95.25) (end 86.995 95.885) (width 0.25) (layer "B.Cu") (net 2))
   (segment (start 107.95 95.885) (end 110.49 98.425) (width 0.25) (layer "B.Cu") (net 2))
@@
   (via (at 114.3 88.9) (size 0.8) (drill 0.4) (layers "F.Cu" "B.Cu") (net 11))
   (via (at 99.06 58.42) (size 0.8) (drill 0.4) (layers "F.Cu" "B.Cu") (net 11))
+  (segment (start 114.3 88.9) (end 114.3 85.353025) (width 0.4064) (layer "In2.Cu") (net 11))
+  (segment (start 104.630493 82.405493) (end 104.14 81.915) (width 0.4064) (layer "In2.Cu") (net 11))
+  (segment (start 112.131975 83.185) (end 106.512389 83.185) (width 0.4064) (layer "In2.Cu") (net 11))
   (segment (start 102.87 78.848949) (end 102.87 67.618153) (width 0.4064) (layer "In2.Cu") (net 11))
-  (segment (start 104.630493 82.405493) (end 104.14 81.915) (width 0.4064) (layer "In2.Cu") (net 11))
-  (segment (start 114.3 88.9) (end 110.050577 84.650577) (width 0.4064) (layer "In2.Cu") (net 11))
+  (arc (start 113.665 83.82) (mid 112.961642 83.350031) (end 112.131975 83.185) (width 0.4064) (layer "In2.Cu") (net 11))
+  (arc (start 102.87 67.618153) (mid 101.879813 62.640148) (end 99.06 58.42) (width 0.4064) (layer "In2.Cu") (net 11))
+  (arc (start 106.512389 83.185) (mid 105.493914 82.982413) (end 104.630493 82.405493) (width 0.4064) (layer "In2.Cu") (net 11))
+  (arc (start 114.3 85.353025) (mid 114.134969 84.523358) (end 113.665 83.82) (width 0.4064) (layer "In2.Cu") (net 11))
   (arc (start 104.14 81.915) (mid 103.200062 80.508284) (end 102.87 78.848949) (width 0.4064) (layer "In2.Cu") (net 11))
-  (arc (start 108.045417 83.82) (mid 106.197274 83.452381) (end 104.630493 82.405493) (width 0.4064) (layer "In2.Cu") (net 11))
-  (arc (start 110.050577 84.650577) (mid 109.130587 84.035859) (end 108.045417 83.82) (width 0.4064) (layer "In2.Cu") (net 11))
-  (arc (start 102.87 67.618153) (mid 101.879813 62.640148) (end 99.06 58.42) (width 0.4064) (layer "In2.Cu") (net 11))
   (segment (start 99.06 50.8) (end 88.9 50.8) (width 0.4064) (layer "F.Cu") (net 12))
   (segment (start 99.06 55.88) (end 88.9 55.88) (width 0.4064) (layer "F.Cu") (net 13))
@@
   (arc (start 106.045 93.345) (mid 107.454906 95.455074) (end 107.95 97.944076) (width 0.4064) (layer "In4.Cu") (net 14))
   (arc (start 104.14 88.745924) (mid 104.635094 91.234926) (end 106.045 93.345) (width 0.4064) (layer "In4.Cu") (net 14))
-  (segment (start 99.06 91.44) (end 88.9 91.44) (width 0.4064) (layer "F.Cu") (net 15))
-  (via (at 88.9 91.44) (size 0.8) (drill 0.4) (layers "F.Cu" "B.Cu") (net 15))
-  (segment (start 95.589723 95.25) (end 97.744872 95.25) (width 0.4064) (layer "In4.Cu") (net 15))
-  (segment (start 88.9 91.44) (end 90.673727 93.213727) (width 0.4064) (layer "In4.Cu") (net 15))
+  (segment (start 99.06 86.36) (end 88.9 86.36) (width 0.4064) (layer "F.Cu") (net 15))
+  (via (at 91.44 86.36) (size 0.8) (drill 0.4) (layers "F.Cu" "B.Cu") (net 15))
+  (segment (start 93.606445 95.25) (end 94.878025 95.25) (width 0.4064) (layer "In4.Cu") (net 15))
+  (segment (start 91.44 90.805) (end 91.44 93.085788) (width 0.4064) (layer "In4.Cu") (net 15))
+  (segment (start 91.44 86.36) (end 91.44 91.814208) (width 0.4064) (layer "In4.Cu") (net 15))
+  (segment (start 96.52 95.25) (end 97.744872 95.25) (width 0.4064) (layer "In4.Cu") (net 15))
+  (segment (start 95.589723 95.25) (end 96.52 95.25) (width 0.4064) (layer "In4.Cu") (net 15))
+  (segment (start 94.878025 95.25) (end 96.52 95.25) (width 0.4064) (layer "In4.Cu") (net 15))
   (arc (start 97.744872 95.25) (mid 101.893209 96.075156) (end 105.41 98.425) (width 0.4064) (layer "In4.Cu") (net 15))
-  (arc (start 90.673727 93.213727) (mid 92.929205 94.720789) (end 95.589723 95.25) (width 0.4064) (layer "In4.Cu") (net 15))
+  (arc (start 91.44 93.085788) (mid 91.60462 93.913391) (end 92.07342 94.615) (width 0.4064) (layer "In4.Cu") (net 15))
+  (arc (start 92.07342 94.615) (mid 92.776778 95.084969) (end 93.606445 95.25) (width 0.4064) (layer "In4.Cu") (net 15))
   (segment (start 99.06 68.58) (end 88.9 68.58) (width 0.4064) (layer "F.Cu") (net 18))
   (segment (start 99.06 60.96) (end 88.9 60.96) (width 0.4064) (layer "F.Cu") (net 19))

Commit message: Mixer2 - prototype1
Parts:
- R5, R7: footprint -lmp-stripboard:SB_Gen_5 -> -lmp-misc:R_Axial_DIN0207_L6.3mm_D2.5mm_P7.62mm_Horizontal
- R9: footprint -lmp-stripboard:SB_Gen_1 -> -lmp-misc:R_Axial_DIN0207_L6.3mm_D2.5mm_P7.62mm_Horizontal
- moved R5 17.8 mm to (88.9, 71.1)
- moved R7 17.8 mm to (116.8, 71.1)
- moved C1 12.7 mm to (96.5, 63.5)
- moved C2 12.7 mm to (109.2, 63.5)
- moved C3 12.7 mm to (88.9, 53.3)
- moved D2 12.7 mm to (91.4, 53.3)
- moved D4 12.7 mm to (91.4, 43.2)
- moved R11 12.7 mm to (96.5, 50.8)
- moved R12 12.7 mm to (111.1, 50.8)
- moved R3 12.7 mm to (109.2, 45.7)
- moved R4 12.7 mm to (116.8, 53.3)
- moved R6 12.7 mm to (94.0, 63.5)
- moved R8 12.7 mm to (111.8, 63.5)
- moved U1 12.7 mm to (99.1, 50.8)
- moved D1 12.7 mm to (113.7, 55.9)
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Routing:
- net Net-(R5-Pad1): track 10.2 -> 38.7 mm, vias 0 -> 2
- net (no net): track 182.9 -> 162.6 mm
- net Net-(D2-Pad2): track 60.4 -> 78.2 mm, vias 2 -> 4
- net Net-(C1-Pad2): track 37.8 -> 53.5 mm
- net OUTPUT: track 29.2 -> 38.4 mm

Commit message: Mixer2 - prototype1
Routing:
- net Net-(C1-Pad2): track 53.5 -> 56.0 mm
- net INPUT: track 34.8 -> 35.7 mm
- net Net-(R5-Pad1): track 38.7 -> 39.6 mm
- net Net-(D2-Pad2): track 78.2 -> 79.0 mm
Changed lines of the file:
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@@
   (segment (start 93.98 66.04) (end 88.9 66.04) (width 0.4064) (layer "F.Cu") (net 5))
   (segment (start 114.3 86.36) (end 106.68 86.36) (width 0.4064) (layer "F.Cu") (net 5))
-  (via (at 114.3 86.36) (size 0.8) (drill 0.4) (layers "F.Cu" "B.Cu") (net 5))
+  (via (at 116.84 86.36) (size 0.8) (drill 0.4) (layers "F.Cu" "B.Cu") (net 5))
   (via (at 91.44 66.04) (size 0.8) (drill 0.4) (layers "F.Cu" "B.Cu") (net 5))
-  (segment (start 112.503949 82.023949) (end 109.002103 78.522103) (width 0.4064) (layer "In4.Cu") (net 5))
-  (segment (start 100.33 74.93) (end 98.951051 74.93) (width 0.4064) (layer "In4.Cu") (net 5))
-  (segment (start 95.885 73.66) (end 93.685064 71.460064) (width 0.4064) (layer "In4.Cu") (net 5))
-  (arc (start 98.951051 74.93) (mid 97.291716 74.599938) (end 95.885 73.66) (width 0.4064) (layer "In4.Cu") (net 5))
-  (arc (start 93.685064 71.460064) (mid 92.023473 68.973317) (end 91.44 66.04) (width 0.4064) (layer "In4.Cu") (net 5))
-  (arc (start 109.002103 78.522103) (mid 105.023309 75.863557) (end 100.33 74.93) (width 0.4064) (layer "In4.Cu") (net 5))
-  (arc (start 114.3 86.36) (mid 113.833222 84.013346) (end 112.503949 82.023949) (width 0.4064) (layer "In4.Cu") (net 5))
+  (segment (start 93.685064 71.460064) (end 95.885 73.66) (width 0.4064) (layer "In4.Cu") (net 5))
+  (segment (start 98.951051 74.93) (end 102.561847 74.93) (width 0.4064) (layer "In4.Cu") (net 5))
+  (segment (start 111.76 78.74) (end 115.043948 82.023948) (width 0.4064) (layer "In4.Cu") (net 5))
+  (arc (start 115.043948 82.023948) (mid 116.373221 84.013346) (end 116.84 86.36) (width 0.4064) (layer "In4.Cu") (net 5))
+  (arc (start 95.885 73.66) (mid 97.291716 74.599938) (end 98.951051 74.93) (width 0.4064) (layer "In4.Cu") (net 5))
+  (arc (start 91.44 66.04) (mid 92.023473 68.973317) (end 93.685064 71.460064) (width 0.4064) (layer "In4.Cu") (net 5))
+  (arc (start 102.561847 74.93) (mid 107.539851 75.920187) (end 111.76 78.74) (width 0.4064) (layer "In4.Cu") (net 5))
   (segment (start 99.06 63.5) (end 88.9 63.5) (width 0.4064) (layer "F.Cu") (net 6))
   (segment (start 116.84 66.04) (end 106.68 66.04) (width 0.4064) (layer "F.Cu") (net 8))
@@
   (via (at 116.84 88.9) (size 0.8) (drill 0.4) (layers "F.Cu" "B.Cu") (net 11))
   (via (at 111.76 71.12) (size 0.8) (drill 0.4) (layers "F.Cu" "B.Cu") (net 11))
-  (segment (start 116.84 84.237102) (end 116.84 88.9) (width 0.4064) (layer "In1.Cu") (net 11))
+  (segment (start 116.84 88.9) (end 117.211974 88.528026) (width 0.4064) (layer "In1.Cu") (net 11))
   (segment (start 111.76 73.025) (end 111.76 71.12) (width 0.4064) (layer "In1.Cu") (net 11))
+  (segment (start 114.96691 78.771911) (end 114.3 78.105) (width 0.4064) (layer "In1.Cu") (net 11))
   (segment (start 113.556051 77.361051) (end 114.3 78.105) (width 0.4064) (layer "In1.Cu") (net 11))
   (arc (start 111.76 73.025) (mid 112.226778 75.371654) (end 113.556051 77.361051) (width 0.4064) (layer "In1.Cu") (net 11))
-  (arc (start 114.3 78.105) (mid 116.179875 80.918432) (end 116.84 84.237102) (width 0.4064) (layer "In1.Cu") (net 11))
+  (arc (start 118.11 86.36) (mid 117.293138 82.253356) (end 114.96691 78.771911) (width 0.4064) (layer "In1.Cu") (net 11))
+  (arc (start 117.211974 88.528026) (mid 117.876611 87.533327) (end 118.11 86.36) (width 0.4064) (layer "In1.Cu") (net 11))
   (segment (start 102.87 54.918153) (end 102.87 60.86754) (width 0.4064) (layer "In2.Cu") (net 11))
   (segment (start 105.629456 67.529456) (end 109.22 71.12) (width 0.4064) (layer "In2.Cu") (net 11))
@@
   (arc (start 105.301052 95.776052) (mid 103.971779 93.786655) (end 103.505 91.44) (width 0.4064) (layer "In1.Cu") (net 14))
   (segment (start 99.06 86.36) (end 88.9 86.36) (width 0.4064) (layer "F.Cu") (net 15))
-  (via (at 91.44 86.36) (size 0.8) (drill 0.4) (layers "F.Cu" "B.Cu") (net 15))
+  (via (at 88.9 86.36) (size 0.8) (drill 0.4) (layers "F.Cu" "B.Cu") (net 15))
   (segment (start 93.606445 95.25) (end 94.878025 95.25) (width 0.4064) (layer "In4.Cu") (net 15))
   (segment (start 91.44 90.805) (end 91.44 93.085788) (width 0.4064) (layer "In4.Cu") (net 15))
-  (segment (start 91.44 86.36) (end 91.44 91.814208) (width 0.4064) (layer "In4.Cu") (net 15))
   (segment (start 96.52 95.25) (end 97.744872 95.25) (width 0.4064) (layer "In4.Cu") (net 15))
+  (segment (start 91.44 90.17) (end 91.44 91.814208) (width 0.4064) (layer "In4.Cu") (net 15))
   (segment (start 95.589723 95.25) (end 96.52 95.25) (width 0.4064) (layer "In4.Cu") (net 15))
+  (segment (start 88.9 86.36) (end 90.541974 88.001974) (width 0.4064) (layer "In4.Cu") (net 15))
   (segment (start 94.878025 95.25) (end 96.52 95.25) (width 0.4064) (layer "In4.Cu") (net 15))
+  (arc (start 90.541974 88.001974) (mid 91.20661 88.996673) (end 91.44 90.17) (width 0.4064) (layer "In4.Cu") (net 15))
   (arc (start 97.744872 95.25) (mid 101.893209 96.075156) (end 105.41 98.425) (width 0.4064) (layer "In4.Cu") (net 15))
   (arc (start 91.44 93.085788) (mid 91.60462 93.913391) (end 92.07342 94.615) (width 0.4064) (layer "In4.Cu") (net 15))
@@
   (via (at 88.9 88.9) (size 0.8) (drill 0.4) (layers "F.Cu" "B.Cu") (net 21))
   (via (at 91.44 71.12) (size 0.8) (drill 0.4) (layers "F.Cu" "B.Cu") (net 21))
+  (segment (start 88.9 88.9) (end 88.528026 88.528026) (width 0.4064) (layer "In1.Cu") (net 21))
+  (segment (start 87.63 86.36) (end 87.63 84.346051) (width 0.4064) (layer "In1.Cu") (net 21))
   (segment (start 91.44 76.852409) (end 91.44 71.12) (width 0.4064) (layer "In1.Cu") (net 21))
-  (segment (start 88.9 88.9) (end 88.9 82.9845) (width 0.4064) (layer "In1.Cu") (net 21))
-  (arc (start 88.9 82.9845) (mid 89.213238 81.409747) (end 90.105271 80.074729) (width 0.4064) (layer "In1.Cu") (net 21))
+  (segment (start 88.9 81.28) (end 90.105271 80.074729) (width 0.4064) (layer "In1.Cu") (net 21))
+  (arc (start 88.528026 88.528026) (mid 87.863389 87.533328) (end 87.63 86.36) (width 0.4064) (layer "In1.Cu") (net 21))
+  (arc (start 87.63 84.346051) (mid 87.960062 82.686717) (end 88.9 81.28) (width 0.4064) (layer "In1.Cu") (net 21))
   (arc (start 90.105271 80.074729) (mid 91.093115 78.596316) (end 91.44 76.852409) (width 0.4064) (layer "In1.Cu") (net 21))
   (segment (start 99.06 50.8) (end 88.9 50.8) (width 0.4064) (layer "F.Cu") (net 22))

Commit message: Mixer2 - update prototype1
Parts:
- R5: footprint -lmp-misc:R_Axial_DIN0207_L6.3mm_D2.5mm_P7.62mm_Horizontal -> -lmp-stripboard:SB_Gen_10
- R9: footprint -lmp-misc:R_Axial_DIN0207_L6.3mm_D2.5mm_P7.62mm_Horizontal -> -lmp-stripboard:SB_Gen_4
- moved R5 17.8 mm to (88.9, 88.9)
- moved D4 5.10 mm to (91.4, 38.1), turned to -90 degrees
Connections:
- D4 pad 1: Net-(D4-Pad1) -> Net-(D3-Pad1)
- D4 pad 3: Net-(D3-Pad1) -> Net-(D4-Pad3)
- R11 pad 2: Net-(D4-Pad1) -> Net-(D4-Pad3)
- R12 pad 2: Net-(D4-Pad1) -> Net-(D4-Pad3)
Routing:
- net Net-(R5-Pad1): track 39.6 -> 10.2 mm, vias 2 -> 0
- net Net-(D4-Pad3): track 0.00 -> 27.9 mm, vias 0 -> 2
- net Net-(D4-Pad1): track 27.9 -> 0.00 mm, vias 2 -> 0
- net (no net): track 162.6 -> 172.7 mm
- net OUTPUT: track 38.4 -> 36.1 mm
- net INPUT: track 35.7 -> 33.8 mm
Other:
- board text added: "X"

Commit message: Mixer2: fix level indicators - wip
Parts:
- removed the D2 at (91.4, 53.3)
- moved R1 38.2 mm to (121.9, 53.3), turned to 180 degrees
- moved R10 33.1 mm to (86.4, 53.3), turned to 0 degrees
- moved C3 28.1 mm to (116.8, 55.9), turned to 0 degrees
- moved R4 28.1 mm to (88.9, 55.9), turned to 180 degrees
- moved R2 18.0 mm to (111.8, 53.3)
- moved R3 18.0 mm to (91.4, 48.3)
- moved R12 14.6 mm to (96.5, 50.8)
- moved R11 12.7 mm to (109.2, 50.8)
- moved D1 0.63 mm to (114.3, 55.9)
- renumbered D3 to D2, D4 to D3
Connections:
- D1 pad 2: Net-(C2-Pad2) -> Net-(C1-Pad2)
- R1 pad 1: +12V -> -12V
- U1 pad 1: Net-(R11-Pad1) -> Net-(R12-Pad1)
- U1 pad 13: VREF-LO -> VREF-5
- U1 pad 14: Net-(R12-Pad1) -> Net-(R11-Pad1)
- U1 pad 3: VREF-5 -> VREF-LO
- U2 pad 2: VREF-4 -> Net-(C3-Pad1)
- U2 pad 3: Net-(C3-Pad1) -> VREF-4
Routing:
- net Net-(R7-Pad1): track 79.0 -> 40.3 mm, vias 4 -> 2
- net Net-(C1-Pad2): track 55.9 -> 93.7 mm, vias 2 -> 4
- net Net-(C2-Pad2): track 39.1 -> 10.2 mm, vias 2 -> 0
- net (no net): track 172.7 -> 182.9 mm
- net Net-(C3-Pad1): track 73.9 -> 67.3 mm
- net VREF-4: track 51.6 -> 54.0 mm
Other:
- board text removed: "X"

Commit message: Mixer2: fix level indicators - wip
Parts:
- D1: value 1N4148 -> 1N5711
- moved D1 7.62 mm to (114.3, 48.3), turned to -90 degrees
Connections:
- D1 pad 1: Net-(C3-Pad1) -> Net-(C1-Pad2)
- D1 pad 2: Net-(C1-Pad2) -> Net-(C3-Pad1)
