File: modules/VCF-4P/prototype3/prototype.kicad_pcb (KiCad board)
At the start: 6 copper layers, 40.6 x 130.8 mm, 38 parts, among them J1 Conn_01x09, U1 TL074, U2 SSI2140

Commit message: VCF-4P: prototype3 - more tweaking
Parts:
- RV1: value 10K -> 25K
Changed lines of the file:
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@@
   (net 34 "Net-(R23-Pad2)")
   (net 35 "Net-(R26-Pad2)")
-  (net 36 "Net-(U2-Pad12)")
+  (net 36 "Net-(R11-Pad2)")
   (net 37 "Net-(RV2-Pad2)")
   (net 38 "Net-(RV5-Pad3)")
@@
     (property "Sheetfile" "prototype.kicad_sch")
     (property "Sheetname" "")
-    (property "Value2" "15K")
+    (property "Value2" "30K used!")
     (attr through_hole)
     (fp_text reference "R9" (at 3.81 0) (layer "F.SilkS")
@@
       (net 19 "Net-(R11-Pad1)") (pintype "passive"))
     (pad "2" thru_hole oval locked (at 2.54 0 270) (size 1.6 1.6) (drill 0.8) (layers *.Cu *.Mask)
-      (net 36 "Net-(U2-Pad12)") (pintype "passive"))
+      (net 36 "Net-(R11-Pad2)") (pintype "passive"))
     (model "${KISYS3DMOD}/Resistor_THT.3dshapes/R_Axial_DIN0207_L6.3mm_D2.5mm_P2.54mm_Vertical.wrl"
       (offset (xyz 0 0 0))
@@
       (net 3 "-12V") (pinfunction "V-") (pintype "power_in"))
     (pad "12" thru_hole circle (at 15.24 20.32) (size 1.7 1.7) (drill 1) (layers *.Cu *.Mask)
-      (net 36 "Net-(U2-Pad12)") (pinfunction "Q-CTRL") (pintype "input"))
+      (net 36 "Net-(R11-Pad2)") (pinfunction "Q-CTRL") (pintype "input"))
     (pad "13" thru_hole circle (at 15.24 17.78) (size 1.7 1.7) (drill 1) (layers *.Cu *.Mask)
       (net 24 "Net-(R10-Pad1)") (pinfunction "IN+") (pintype "input"))
@@
       (effects (font (size 1 1) (thickness 0.15)))
     )
-    (fp_text value "10K" (at 0 0 90) (layer "F.Fab") hide
+    (fp_text value "25K" (at 0 0 90) (layer "F.Fab") hide
       (effects (font (size 1 1) (thickness 0.15)))
     )
@@
     (property "Sheetfile" "prototype.kicad_sch")
     (property "Sheetname" "")
-    (property "Value2" "47K")
     (attr through_hole)
     (fp_text reference "R7" (at 3.81 0 90) (layer "F.SilkS")
@@
     )
   )
-  (gr_circle (center 88.9 116.84) (end 90.696051 116.84) (layer "Dwgs.User") (width 0.254) (fill none))
-  (gr_circle (center 91.44 110.49) (end 93.236051 110.49) (layer "Dwgs.User") (width 0.254) (fill none))
-  (gr_circle (center 96.52 64.77) (end 98.316051 64.77) (layer "Dwgs.User") (width 0.254) (fill none))
-  (gr_circle (center 100.86898 111.711085) (end 102.665031 111.711085) (layer "Dwgs.User") (width 0.254) (fill none))
-  (gr_circle (center 87.63 107.95) (end 89.426051 107.95) (layer "Dwgs.User") (width 0.254) (fill none))
-  (gr_circle (center 92.71 104.14) (end 94.506051 104.14) (layer "Dwgs.User") (width 0.254) (fill none))
   (gr_line (start 123.19 168.91) (end 82.55 168.91) (layer "Edge.Cuts") (width 0.1))
   (gr_line (start 123.19 38.1) (end 123.19 168.91) (layer "Edge.Cuts") (width 0.1))
