File: modules/FX/prototype/prototype.kicad_pcb (KiCad board)
At the start: 6 copper layers, 40.6 x 78.7 mm, 21 parts, among them J1 Conn_01x09, SW1 SW_LED, U1 TL072, U2 L7808

Commit message: FX prototype wip
Parts:
- moved U2 71.9 mm to (111.8, 66.0), turned to -90 degrees
- moved C2 62.0 mm to (129.6, 79.1)
- moved C3 62.0 mm to (129.6, 83.2)
- moved R7 62.0 mm to (127.2, 75.1)
- moved RV2 53.3 mm to (109.2, 38.1), turned to -90 degrees
- moved C1 53.1 mm to (127.7, 33.7)
- moved R2 53.1 mm to (128.0, 26.4)
- moved RV3 46.6 mm to (109.2, 58.4), turned to -90 degrees
- moved U1 44.2 mm to (106.7, 83.8), turned to 180 degrees
- moved RV1 31.6 mm to (109.2, 48.3), turned to -90 degrees
- moved R6 28.2 mm to (132.5, 39.4)
- moved R8 28.2 mm to (132.5, 47.5)
- moved R9 28.2 mm to (128.9, 52.7)
- moved R3 25.1 mm to (127.0, 66.4)
- moved R4 25.1 mm to (127.0, 70.5)
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Connections:
- RV1 pad 1: Net-(A1-Pad1) -> GND
- RV1 pad 3: GND -> Net-(A1-Pad1)
- RV2 pad 1: Net-(A1-Pad1) -> GND
- RV2 pad 3: GND -> Net-(A1-Pad1)
- RV3 pad 1: Net-(A1-Pad1) -> GND
- RV3 pad 3: GND -> Net-(A1-Pad1)
Routing:
- net (no net): track 375.9 -> 162.6 mm
- net GND: track 216.0 -> 282.1 mm, vias 2 -> 18
- net +12V: track 90.2 -> 139.2 mm, vias 1 -> 5
- net Net-(R1-Pad2): track 30.5 -> 56.6 mm, vias 0 -> 6
- net Net-(R3-Pad1): track 0.00 -> 20.3 mm
- net Net-(A1-Pad1): track 10.2 -> 30.5 mm
- net +8V: track 10.2 -> 27.9 mm, vias 0 -> 2
- net -12V: track 80.8 -> 96.0 mm, vias 1 -> 3
- net Net-(A1-Pad2): track 10.2 -> 22.9 mm, vias 0 -> 2
- net Net-(C3-Pad1): track 0.00 -> 10.2 mm
- net Net-(C2-Pad1): track 0.00 -> 10.2 mm
- net Net-(A1-Pad5): track 10.2 -> 20.3 mm
- net Net-(A1-Pad4): track 10.2 -> 20.3 mm, vias 0 -> 1
- net Net-(A1-Pad3): track 10.2 -> 20.3 mm
- net IN-OUT-2: track 3.17 -> 10.2 mm
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
Commit message: FX prototype wip
Parts:
- R1, R9: footprint -lmp-misc:R_Axial_DIN0207_L6.3mm_D2.5mm_P7.62mm_Horizontal -> -lmp-stripboard:SB_Gen_4
- R2, R4, R6: footprint -lmp-misc:R_Axial_DIN0207_L6.3mm_D2.5mm_P7.62mm_Horizontal -> -lmp-stripboard:SB_Gen_1
- R5: footprint -lmp-misc:R_Axial_DIN0207_L6.3mm_D2.5mm_P7.62mm_Horizontal -> -lmp-stripboard:SB_Gen_5
- moved R2 69.4 mm to (88.9, 83.8), turned to 180 degrees
- moved C1 54.8 mm to (96.5, 78.7), turned to -90 degrees
- moved R5 52.1 mm to (91.4, 40.6), turned to -90 degrees
- moved R6 45.8 mm to (88.9, 53.3), turned to 180 degrees
- moved R3 40.8 mm to (91.4, 86.4), turned to 90 degrees
- moved R4 39.0 mm to (88.9, 78.7), turned to 180 degrees
- moved R8 39.0 mm to (109.2, 78.7), turned to -90 degrees
- moved R9 32.1 mm to (114.3, 81.3), turned to -90 degrees
- moved R10 23.4 mm to (111.8, 78.7)
- moved C2 22.6 mm to (109.2, 88.9), turned to -90 degrees
- moved R7 16.7 mm to (111.8, 81.3), turned to -90 degrees
- moved C3 13.1 mm to (116.8, 86.4)
- moved U1 7.62 mm to (106.7, 91.4)
- moved R1 3.59 mm to (88.9, 43.2)
- moved RV3 0.64 mm to (109.9, 58.4)
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Connections:
- U1 pad 1: Net-(R3-Pad1) -> IN-OUT-2
- U1 pad 2: Net-(R3-Pad1) -> Net-(C2-Pad1)
- U1 pad 3: IN-OUT-1 -> Net-(C3-Pad1)
- U1 pad 5: Net-(C3-Pad1) -> IN-OUT-1
- U1 pad 6: Net-(C2-Pad1) -> Net-(R3-Pad1)
- U1 pad 7: IN-OUT-2 -> Net-(R3-Pad1)
Routing:
- net (no net): track 162.6 -> 121.9 mm
- net Net-(A1-Pad1): track 30.5 -> 70.4 mm, vias 0 -> 6
- net Net-(A1-Pad9): track 10.2 -> 42.9 mm, vias 0 -> 2
- net Net-(A1-Pad10): track 10.2 -> 37.8 mm, vias 0 -> 2
- net Net-(A1-Pad11): track 10.2 -> 36.2 mm, vias 0 -> 2
- net IN-OUT-1: track 10.2 -> 30.6 mm, vias 0 -> 1
- net Net-(A1-Pad4): track 20.3 -> 33.3 mm, vias 1 -> 2
- net Net-(A1-Pad2): track 22.9 -> 10.2 mm, vias 2 -> 0
- net Net-(A1-Pad3): track 20.3 -> 31.1 mm, vias 0 -> 2
- net Net-(A1-Pad5): track 20.3 -> 31.1 mm, vias 0 -> 2
- net Net-(C1-Pad1): track 0.00 -> 10.2 mm
- net IN-OUT-2: track 10.2 -> 18.4 mm, vias 0 -> 1
- net GND: track 282.1 -> 277.0 mm
- net Net-(R3-Pad1): track 20.3 -> 22.9 mm, vias 0 -> 2
