File: modules/FX/prototype/prototype.kicad_sch (KiCad schematic)
At the start: 21 parts, among them J1 Conn_01x09, SW1 SW_LED, U1 TL072, U2 L7808

Commit message: FX prototype wip
Connections:
- net GND: now also RV1.1, RV2.1, RV3.1; no longer RV1.3, RV2.3, RV3.3
- new net: A1.1 (VPOT), R5.1, RV1.3, RV2.3, RV3.3
Changed lines of the file:
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@@
     (pin "1")
   )
-  (symbol (lib_id "-lmp:R_POT_TRIM") (at 52.07 77.47 0) (unit 1)
+  (symbol (lib_id "-lmp:R_POT_TRIM") (at 52.07 77.47 0) (mirror x) (unit 1)
     (in_bom yes) (on_board yes) (fields_autoplaced)
     (property "Reference" "RV2" (id 0) (at 50.292 75.3669 0)
@@
     (pin "1")
   )
-  (symbol (lib_id "-lmp:R_POT_TRIM") (at 43.18 72.39 0) (unit 1)
+  (symbol (lib_id "-lmp:R_POT_TRIM") (at 43.18 72.39 0) (mirror x) (unit 1)
     (in_bom yes) (on_board yes) (fields_autoplaced)
     (property "Reference" "RV1" (id 0) (at 41.402 70.2869 0)
@@
     (pin "1")
   )
-  (symbol (lib_id "-lmp:R_POT_TRIM") (at 60.96 82.55 0) (unit 1)
+  (symbol (lib_id "-lmp:R_POT_TRIM") (at 60.96 82.55 0) (mirror x) (unit 1)
     (in_bom yes) (on_board yes) (fields_autoplaced)
     (property "Reference" "RV3" (id 0) (at 59.182 80.4469 0)

Commit message: FX prototype wip
Parts:
- R1, R9: footprint -lmp-misc:R_Axial_DIN0207_L6.3mm_D2.5mm_P7.62mm_Horizontal -> -lmp-stripboard:SB_Gen_4
- R2, R4, R6: footprint -lmp-misc:R_Axial_DIN0207_L6.3mm_D2.5mm_P7.62mm_Horizontal -> -lmp-stripboard:SB_Gen_1
- R5: footprint -lmp-misc:R_Axial_DIN0207_L6.3mm_D2.5mm_P7.62mm_Horizontal -> -lmp-stripboard:SB_Gen_5
Connections:
- net IN-OUT-1: now also U1.5 (+); no longer U1.3 (+)
- net IN-OUT-2: now also U1.1; no longer U1.7
- net at C2.1, R7.2: now also U1.2 (-); no longer U1.6 (-)
- net at C3.1, R8.2: now also U1.3 (+); no longer U1.5 (+)
- new net: R3.1, U1.6 (-), U1.7
Other:
- moved on the sheet: A1, C1, C2, C3, J1, R1, R10, R2, R3, R4, R5, R6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
