File: modules/FX/FX-proto/FX-proto.kicad_sch (KiCad schematic)
At the start: 32 parts, among them J1 WQP-PJ398, J2 WQP-PJ398, J3 Conn_Eurorack_16, SW1 SW_LED, U1 TL074, U2 L7808

Commit message: FX module - prototype wip
Parts:
- added R8: 50K, -lmp-misc:R_Axial_DIN0207_L6.3mm_D2.5mm_P10.16mm_Horizontal, symbol -lmp:R_1%_0W166
- R10: value 47K -> 120K
Connections:
- net at R10.1, U1.9 (-): now also R8.2; no longer RV5.2
- new net: R8.1, RV5.2
Other:
- note added: "The output must be AC-coupled because the wet & dry signals have different DC offsets"
- note removed: "PROBLEM: Voltage offset: dry is 0-2V, wet is -1-+1V"
- note removed: "TODO: 100K instead?"
- moved on the sheet: RV5
Changed lines of the file:
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@@
     (stroke (width 0) (type default) (color 0 0 0 0))
   )
-  (wire (pts (xy 172.72 50.8) (xy 172.72 29.21))
+  (wire (pts (xy 163.83 50.8) (xy 163.83 29.21))
     (stroke (width 0) (type default) (color 0 0 0 0))
   )
@@
     (stroke (width 0) (type default) (color 0 0 0 0))
   )
-  (wire (pts (xy 172.72 59.69) (xy 172.72 58.42))
+  (wire (pts (xy 163.83 59.69) (xy 163.83 58.42))
     (stroke (width 0) (type default) (color 0 0 0 0))
   )
@@
     (stroke (width 0) (type default) (color 0 0 0 0))
   )
-  (wire (pts (xy 91.44 29.21) (xy 172.72 29.21))
+  (wire (pts (xy 91.44 29.21) (xy 163.83 29.21))
     (stroke (width 0) (type default) (color 0 0 0 0))
   )
@@
     (stroke (width 0) (type default) (color 0 0 0 0))
   )
-  (wire (pts (xy 176.53 54.61) (xy 180.34 54.61))
+  (wire (pts (xy 167.64 54.61) (xy 170.18 54.61))
     (stroke (width 0) (type default) (color 0 0 0 0))
   )
@@
     (stroke (width 0) (type default) (color 0 0 0 0))
   )
+  (wire (pts (xy 177.8 54.61) (xy 180.34 54.61))
+    (stroke (width 0) (type default) (color 0 0 0 0))
+  )
   (wire (pts (xy 48.26 48.26) (xy 48.26 53.34))
     (stroke (width 0) (type default) (color 0 0 0 0))
@@
     (stroke (width 0) (type default) (color 0 0 0 0))
   )
-  (wire (pts (xy 154.94 59.69) (xy 172.72 59.69))
+  (wire (pts (xy 154.94 59.69) (xy 163.83 59.69))
     (stroke (width 0) (type default) (color 0 0 0 0))
   )
@@
     (effects (font (size 1.27 1.27)) (justify left bottom))
   )
-  (text "PROBLEM: Voltage offset: \ndry is 0-2V, wet is -1-+1V"
-    (at 157.48 72.39 0)
+  (text "The output must be AC-coupled \nbecause the wet & dry signals \nhave different DC offsets"
+    (at 175.26 76.2 0)
     (effects (font (size 1.27 1.27)) (justify left bottom))
   )
@@
   (text "using 18K" (at 64.77 46.99 0)
     (effects (font (size 1.27 1.27)) (justify left bottom))
-  )
-  (text "TODO: 100K instead?" (at 198.12 40.64 180)
-    (effects (font (size 1.27 1.27)) (justify right bottom))
   )
   (label "DRY" (at 124.46 29.21 0)
@@
     (pin "1")
   )
-  (symbol (lib_id "-lmp-synth:R_POT_TRIM_Panel_SongHuei") (at 172.72 54.61 0) (unit 1)
-    (in_bom yes) (on_board yes) (fields_autoplaced)
-    (property "Reference" "RV5" (id 0) (at 170.942 52.5069 0)
-      (effects (font (size 1.27 1.27)) (justify right))
-    )
-    (property "Value" "50K" (id 1) (at 170.942 55.0438 0)
-      (effects (font (size 1.27 1.27)) (justify right))
-    )
-    (property "Footprint" "-lmp-synth:Potentiometer_SongHuei_Single_Vertical" (id 2) (at 172.72 54.61 0)
-      (effects (font (size 1.27 1.27)) hide)
-    )
-    (property "Datasheet" "http://www.song-huei.com/proimages//eng/pdfimages/R0904N.pdf" (id 3) (at 172.72 54.61 0)
-      (effects (font (size 1.27 1.27)) hide)
-    )
-    (property "Label" "MIX" (id 4) (at 170.942 57.5807 0)
-      (effects (font (size 1.27 1.27)) (justify right))
-    )
-    (property "Manufacturer" "Song Huei" (id 5) (at 172.72 54.61 0)
-      (effects (font (size 1.27 1.27)) hide)
-    )
-    (property "ManufacturerPartNum" "R0904N*" (id 6) (at 172.72 54.61 0)
-      (effects (font (size 1.27 1.27)) hide)
-    )
-    (property "Distributor" "SynthCube" (id 7) (at 172.72 54.61 0)
-      (effects (font (size 1.27 1.27)) hide)
-    )
-    (property "DistributorPartNum" "SH9MMTPOTMSTR" (id 8) (at 172.72 54.61 0)
-      (effects (font (size 1.27 1.27)) hide)
-    )
-    (property "DistributorPartLink" "https://synthcube.com/cart/9mm-trimmer-pots" (id 9) (at 172.72 54.61 0)
-      (effects (font (size 1.27 1.27)) hide)
-    )
-    (property "Distributor2" "Thonk" (id 10) (at 172.72 54.61 0)
-      (effects (font (size 1.27 1.27)) hide)
-    )
-    (property "DistributorPartNum2" "Group_SongHuei_TTP" (id 11) (at 172.72 54.61 0)
-      (effects (font (size 1.27 1.27)) hide)
-    )
-    (property "DistributorPartLink2" "https://www.thonk.co.uk/shop/ttpots/" (id 12) (at 172.72 54.61 0)
+  (symbol (lib_id "-lmp-synth:R_POT_TRIM_Panel_SongHuei") (at 163.83 54.61 0) (unit 1)
+    (in_bom yes) (on_board yes) (fields_autoplaced)
+    (property "Reference" "RV5" (id 0) (at 162.052 52.5069 0)
+      (effects (font (size 1.27 1.27)) (justify right))
+    )
+    (property "Value" "50K" (id 1) (at 162.052 55.0438 0)
+      (effects (font (size 1.27 1.27)) (justify right))
+    )
+    (property "Footprint" "-lmp-synth:Potentiometer_SongHuei_Single_Vertical" (id 2) (at 163.83 54.61 0)
+      (effects (font (size 1.27 1.27)) hide)
+    )
+    (property "Datasheet" "http://www.song-huei.com/proimages//eng/pdfimages/R0904N.pdf" (id 3) (at 163.83 54.61 0)
+      (effects (font (size 1.27 1.27)) hide)
+    )
+    (property "Label" "MIX" (id 4) (at 162.052 57.5807 0)
+      (effects (font (size 1.27 1.27)) (justify right))
+    )
+    (property "Manufacturer" "Song Huei" (id 5) (at 163.83 54.61 0)
+      (effects (font (size 1.27 1.27)) hide)
+    )
+    (property "ManufacturerPartNum" "R0904N*" (id 6) (at 163.83 54.61 0)
+      (effects (font (size 1.27 1.27)) hide)
+    )
+    (property "Distributor" "SynthCube" (id 7) (at 163.83 54.61 0)
+      (effects (font (size 1.27 1.27)) hide)
+    )
+    (property "DistributorPartNum" "SH9MMTPOTMSTR" (id 8) (at 163.83 54.61 0)
+      (effects (font (size 1.27 1.27)) hide)
+    )
+    (property "DistributorPartLink" "https://synthcube.com/cart/9mm-trimmer-pots" (id 9) (at 163.83 54.61 0)
+      (effects (font (size 1.27 1.27)) hide)
+    )
+    (property "Distributor2" "Thonk" (id 10) (at 163.83 54.61 0)
+      (effects (font (size 1.27 1.27)) hide)
+    )
+    (property "DistributorPartNum2" "Group_SongHuei_TTP" (id 11) (at 163.83 54.61 0)
+      (effects (font (size 1.27 1.27)) hide)
+    )
+    (property "DistributorPartLink2" "https://www.thonk.co.uk/shop/ttpots/" (id 12) (at 163.83 54.61 0)
       (effects (font (size 1.27 1.27)) hide)
     )
@@
     (in_bom yes) (on_board yes) (fields_autoplaced)
     (property "Reference" "R10" (id 0) (at 189.23 42.2742 90))
-    (property "Value" "47K" (id 1) (at 189.23 44.8111 90))
+    (property "Value" "120K" (id 1) (at 189.23 44.8111 90))
     (property "Footprint" "-lmp-misc:R_Axial_DIN0207_L6.3mm_D2.5mm_P7.62mm_Horizontal" (id 2) (at 189.23 48.768 90)
       (effects (font (size 1.27 1.27)) hide)
@@
     (pin "1")
   )
+  (symbol (lib_id "-lmp:R_1%_0W166") (at 173.99 54.61 90) (unit 1)
+    (in_bom yes) (on_board yes) (fields_autoplaced)
+    (property "Reference" "R8" (id 0) (at 173.99 49.8942 90))
+    (property "Value" "50K" (id 1) (at 173.99 52.4311 90))
+    (property "Footprint" "-lmp-misc:R_Axial_DIN0207_L6.3mm_D2.5mm_P10.16mm_Horizontal" (id 2) (at 173.99 56.388 90)
+      (effects (font (size 1.27 1.27)) hide)
+    )
+    (property "Datasheet" "https://www.mouser.ca/datasheet/2/447/Yageo_LR_MFR_1-1714151.pdf" (id 3) (at 173.99 54.61 0)
+      (effects (font (size 1.27 1.27)) hide)
+    )
+    (property "Manufacturer" "YAGEO" (id 4) (at 173.99 54.61 0)
+      (effects (font (size 1.27 1.27)) hide)
+    )
+    (property "ManufacturerPartNum" "MFR-12*" (id 5) (at 173.99 54.61 0)
+      (effects (font (size 1.27 1.27)) hide)
+    )
+    (property "Distributor" "Mouser" (id 6) (at 173.99 54.61 0)
+      (effects (font (size 1.27 1.27)) hide)
+    )
+    (property "DistributorPartNum" "603-MFR-12*" (id 7) (at 173.99 54.61 0)
+      (effects (font (size 1.27 1.27)) hide)
+    )
+    (property "DistributorPartLink" "https://www.mouser.ca/c/?m=YAGEO&power+rating=166+mW+(1%2f6+W)&tolerance=1+%25&instock=y" (id 8) (at 173.99 54.61 0)
+      (effects (font (size 1.27 1.27)) hide)
+    )
+    (property "Value2" "1%, 1/6 W" (id 9) (at 173.99 49.657 90)
+      (effects (font (size 1.27 1.27)) hide)
+    )
+    (pin "1")
+    (pin "2")
+  )
   (sheet_instances
     (path "/" (page "1"))
@@
       (reference "R7") (unit 1) (value "2K2") (footprint "-lmp-misc:R_Axial_DIN0207_L6.3mm_D2.5mm_P7.62mm_Horizontal")
     )
+    (path "/fd4b1314-1824-4744-88d4-df069314039f"
+      (reference "R8") (unit 1) (value "50K") (footprint "-lmp-misc:R_Axial_DIN0207_L6.3mm_D2.5mm_P10.16mm_Horizontal")
+    )
     (path "/70b9914f-0138-470a-a07d-e1a88a53471e"
-      (reference "R10") (unit 1) (value "47K") (footprint "-lmp-misc:R_Axial_DIN0207_L6.3mm_D2.5mm_P7.62mm_Horizontal")
+      (reference "R10") (unit 1) (value "120K") (footprint "-lmp-misc:R_Axial_DIN0207_L6.3mm_D2.5mm_P7.62mm_Horizontal")
     )
     (path "/03216e0c-228a-4522-87f3-4f630b94ac88"

Commit message: FX module - prototype wip
Parts:
- RV5: value 50K -> 100K
Changed lines of the file:
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@@
   (title_block
     (title "FX Module Prototype")
-    (date "2022-08-24")
+    (date "2022-08-26")
     (rev "1.0")
     (company "Len Popp")
@@
       (effects (font (size 1.27 1.27)) (justify right))
     )
-    (property "Value" "50K" (id 1) (at 162.052 55.0438 0)
+    (property "Value" "100K" (id 1) (at 162.052 55.0438 0)
       (effects (font (size 1.27 1.27)) (justify right))
     )
@@
     )
     (path "/2caafe1c-fbc4-4c4c-b87d-819f24ff7b21"
-      (reference "RV5") (unit 1) (value "50K") (footprint "-lmp-synth:Potentiometer_SongHuei_Single_Vertical")
+      (reference "RV5") (unit 1) (value "100K") (footprint "-lmp-synth:Potentiometer_SongHuei_Single_Vertical")
     )
     (path "/15358bc9-b991-48c5-b15f-fb3b0c574570"
