File: modules/Adder/Adder.kicad_pcb (KiCad board)
At the start: 2 copper layers, 101.3 x 108.2 mm, 20 parts, among them J1 WQP-PJ398, J10 Conn_Front, J11 Conn_Back, J2 WQP-PJ398, J3 WQP-PJ398, J4 WQP-PJ398, J9 Conn_Eurorack_16

Commit message: Adder - wip
Parts:
- removed JP1: GATE-BUS, -lmp-misc:PinHeader_1x03_P2.54mm_Vertical
- removed RV1, RV2, RV3, RV4: 100K, -lmp-synth:Potentiometer_Alpha_RD901F-40-00D_Single_Vertical
- added C1: 5P6, -lmp-misc:C_Disc_D5.0mm_W2.5mm_P2.50mm, F.Cu at (186.7, 100.2)
- added C10: 100N, -lmp-misc:C_Disc_D5.0mm_W2.5mm_P2.50mm, F.Cu at (186.7, 108.6)
- added C11: 100N, -lmp-misc:C_Disc_D5.0mm_W2.5mm_P2.50mm, F.Cu at (168.9, 76.2)
- added C12: 100N, -lmp-misc:C_Disc_D5.0mm_W2.5mm_P2.50mm, F.Cu at (186.7, 76.2)
- added C2: 5P6, -lmp-misc:C_Disc_D5.0mm_W2.5mm_P2.50mm, F.Cu at (168.9, 95.1)
- added C6: 100N, -lmp-misc:C_Disc_D5.0mm_W2.5mm_P2.50mm, F.Cu at (186.7, 52.2)
- added C7: 100N, -lmp-misc:C_Disc_D5.0mm_W2.5mm_P2.50mm, F.Cu at (168.9, 100.2)
- added C8: 100N, -lmp-misc:C_Disc_D5.0mm_W2.5mm_P2.50mm, F.Cu at (186.7, 92.6)
- added C9: 100N, -lmp-misc:C_Disc_D5.0mm_W2.5mm_P2.50mm, F.Cu at (168.9, 116.3)
- added D2: LED_Bidi, LED_THT:LED_D3.0mm, F.Cu at (109.2, 130.0)
- added J5: WQP-PJ398, -lmp-synth:Jack_3.5mm_QingPu_WQP-PJ398SM_Vertical, F.Cu at (116.8, 99.1)
- added J6: WQP-PJ398, -lmp-synth:Jack_3.5mm_QingPu_WQP-PJ398SM_Vertical, F.Cu at (116.8, 109.9)
- added J7: WQP-PJ398, -lmp-synth:Jack_3.5mm_QingPu_WQP-PJ398SM_Vertical, F.Cu at (116.8, 120.7)
- added J8: WQP-PJ398, -lmp-synth:Jack_3.5mm_QingPu_WQP-PJ398SM_Vertical, F.Cu at (116.8, 139.7)
- added R1: 1M, -lmp-misc:R_Axial_DIN0207_L6.3mm_D2.5mm_P7.62mm_Horizontal, F.Cu at (184.2, 49.7)
- added R10: 270R, -lmp-misc:R_Axial_DIN0207_L6.3mm_D2.5mm_P10.16mm_Horizontal, F.Cu at (184.2, 103.5)
- added R11: 1M, -lmp-misc:R_Axial_DIN0207_L6.3mm_D2.5mm_P7.62mm_Horizontal, F.Cu at (126.4, 109.2)
- added R12: 1M, -lmp-misc:R_Axial_DIN0207_L6.3mm_D2.5mm_P7.62mm_Horizontal, F.Cu at (128.8, 113.3)
- added R13: 1M, -lmp-misc:R_Axial_DIN0207_L6.3mm_D2.5mm_P7.62mm_Horizontal, F.Cu at (128.5, 117.6)
- added R14: 10K, -lmp-misc:R_Axial_DIN0207_L6.3mm_D2.5mm_P10.16mm_Horizontal, F.Cu at (126.5, 72.4)
- added R15: 10K, -lmp-misc:R_Axial_DIN0207_L6.3mm_D2.5mm_P10.16mm_Horizontal, F.Cu at (126.5, 85.4)
- added R16: 10K, -lmp-misc:R_Axial_DIN0207_L6.3mm_D2.5mm_P10.16mm_Horizontal, F.Cu at (126.4, 97.1)
- added R17: 10K, -lmp-misc:R_Axial_DIN0207_L6.3mm_D2.5mm_P10.16mm_Horizontal, F.Cu at (126.7, 55.0)
- added R18: 10K, -lmp-misc:R_Axial_DIN0207_L6.3mm_D2.5mm_P10.16mm_Horizontal, F.Cu at (126.7, 46.9)
- added R19: 10K, -lmp-misc:R_Axial_DIN0207_L6.3mm_D2.5mm_P10.16mm_Horizontal, F.Cu at (126.5, 76.5)
- added R2: 1M, -lmp-misc:R_Axial_DIN0207_L6.3mm_D2.5mm_P7.62mm_Horizontal, F.Cu at (168.9, 49.7)
- added R20: 270R, -lmp-misc:R_Axial_DIN0207_L6.3mm_D2.5mm_P10.16mm_Horizontal, F.Cu at (126.5, 64.3)
- added R21: 1K, -lmp-misc:R_Axial_DIN0207_L6.3mm_D2.5mm_P10.16mm_Horizontal, F.Cu at (184.2, 113.7)
- added R22: 1K, -lmp-misc:R_Axial_DIN0207_L6.3mm_D2.5mm_P10.16mm_Horizontal, F.Cu at (168.9, 111.1)
- added R3: 1M, -lmp-misc:R_Axial_DIN0207_L6.3mm_D2.5mm_P7.62mm_Horizontal, F.Cu at (168.9, 54.7)
- added R4: 10K, -lmp-misc:R_Axial_DIN0207_L6.3mm_D2.5mm_P10.16mm_Horizontal, F.Cu at (184.2, 44.6)
- added R5: 10K, -lmp-misc:R_Axial_DIN0207_L6.3mm_D2.5mm_P10.16mm_Horizontal, F.Cu at (168.9, 44.5)
- added R6: 10K, -lmp-misc:R_Axial_DIN0207_L6.3mm_D2.5mm_P10.16mm_Horizontal, F.Cu at (171.3, 64.1)
- added R7: 10K, -lmp-misc:R_Axial_DIN0207_L6.3mm_D2.5mm_P10.16mm_Horizontal, F.Cu at (184.2, 57.3)
- added R8: 10K, -lmp-misc:R_Axial_DIN0207_L6.3mm_D2.5mm_P10.16mm_Horizontal, F.Cu at (184.2, 59.8)
- added R9: 10K, -lmp-misc:R_Axial_DIN0207_L6.3mm_D2.5mm_P10.16mm_Horizontal, F.Cu at (184.2, 97.7)
- added U1: LT1014, Package_DIP:DIP-14_W7.62mm, F.Cu at (172.7, 44.6)
- added U2: LT1013, Package_DIP:DIP-8_W7.62mm, F.Cu at (180.3, 100.2)
- added U3: TL072, Package_DIP:DIP-8_W7.62mm, F.Cu at (180.3, 116.2)
- added U4: LT1014, Package_DIP:DIP-14_W7.62mm, F.Cu at (172.7, 68.6)
- C5: value 10U -> 100N; footprint -lmp-misc:CP_Radial_D5.0mm_P2.50mm -> -lmp-misc:C_Disc_D5.0mm_W2.5mm_P2.50mm
- D1: value LED_5mm_Blue -> LED_Bidi; footprint LED_THT:LED_D5.0mm -> LED_THT:LED_D3.0mm
- J10: footprint Connector_PinSocket_2.54mm:PinSocket_1x18_P2.54mm_Vertical -> Connector_PinSocket_2.54mm:PinSocket_1x13_P2.54mm_Vertical
- J11: footprint Connector_PinHeader_2.54mm:PinHeader_1x18_P2.54mm_Horizontal -> Connector_PinHeader_2.54mm:PinHeader_1x13_P2.54mm_Horizontal
- J9: value Conn_Eurorack_16 -> Conn_Eurorack_10; footprint -lmp-synth:IDC-Header-Eurorack-16-TH -> -lmp-synth:IDC-Header-Eurorack-10-TH
- moved J2 80.5 mm to (116.8, 52.7), turned to -90 degrees
- moved J1 77.2 mm to (116.8, 41.9), turned to -90 degrees
- moved C5 66.6 mm to (168.8, 52.2), turned to 180 degrees
- moved J3 54.8 mm to (116.8, 63.5), turned to -90 degrees
- moved J4 49.8 mm to (116.8, 82.5), turned to -90 degrees
- moved D1 39.4 mm to (111.8, 72.9), turned to 180 degrees
- moved J10 15.2 mm to (101.6, 76.2)
- moved J11 15.2 mm to (152.4, 76.2)
- moved C3 3.05 mm to (187.6, 129.5)
- moved C4 2.10 mm to (187.6, 139.4)
- renumbered C2 to C3, C1 to C4
Connections:
- net Net-(J10-Pad10) renamed LED-2-1
- net Net-(J10-Pad11) renamed LED-2-2
- net Net-(J10-Pad12) renamed OUT-2
- net Net-(J10-Pad7) renamed IN-2-1
- net Net-(J10-Pad8) renamed IN-2-2
- net Net-(J10-Pad9) renamed IN-2-3
- C5 pad 1: +5V -> +12V
- D1 pad 1: GND -> LED-1-2
- D1 pad 2: LED-1 -> LED-1-1
- J1 pad T: IN-GATE-1 -> IN-1-1
- J1 pad TN: IN-GATE-BUS -> GND
- J10 pad 1: IN-GATE-1 -> IN-1-1
- J10 pad 13: Net-(J10-Pad13) -> GND
- J10 pad 2: Net-(J10-Pad2) -> IN-1-2
- J10 pad 3: Net-(J10-Pad3) -> IN-1-3
- J10 pad 4: Net-(J10-Pad4) -> LED-1-1
- J10 pad 5: Net-(J10-Pad5) -> LED-1-2
- J10 pad 6: Net-(J10-Pad6) -> OUT-1
- J11 pad 1: IN-GATE-1 -> IN-1-1
- J11 pad 13: Net-(J10-Pad13) -> GND
- J11 pad 2: Net-(J10-Pad2) -> IN-1-2
- J11 pad 3: Net-(J10-Pad3) -> IN-1-3
- J11 pad 4: Net-(J10-Pad4) -> LED-1-1
- J11 pad 5: Net-(J10-Pad5) -> LED-1-2
- J11 pad 6: Net-(J10-Pad6) -> OUT-1
- J2 pad T: OUT-1 -> IN-1-2
- J2 pad TN: unconnected-(J2-PadTN) -> IN-1-1
- J3 pad T: unconnected-(J3-PadT) -> IN-1-3
- J3 pad TN: unconnected-(J3-PadTN) -> IN-1-1
- J4 pad T: unconnected-(J4-PadT) -> OUT-1
Routing:
- net -12V: track 10.1 -> 103.6 mm, vias 0 -> 1
- net +12V: track 11.0 -> 95.7 mm, vias 0 -> 1
- net IN-1-1: track 0.00 -> 35.9 mm
- net Net-(J9-Pad15): track 20.0 -> 0.00 mm
- net +5V: track 18.9 -> 0.00 mm
Other:
- board text added: "Adder"
- board text added: "https://len42.github.io/Synth/"
- board text removed: "GATE BUS"

Commit message: Adder - wip
Parts:
- moved R18 73.1 mm to (181.6, 95.3), turned to 180 degrees
- moved R11 67.8 mm to (184.2, 73.7)
- moved R17 63.1 mm to (184.2, 81.3)
- moved R20 58.5 mm to (168.9, 104.7), turned to 180 degrees
- moved R14 57.7 mm to (184.2, 68.6)
- moved R12 56.3 mm to (168.9, 73.7), turned to 180 degrees
- moved R13 56.0 mm to (168.9, 78.7), turned to 180 degrees
- moved R19 47.8 mm to (168.9, 98.6), turned to 180 degrees
- moved R16 46.0 mm to (171.4, 88.0)
- moved R15 45.4 mm to (171.4, 91.6)
- moved R8 30.3 mm to (191.1, 89.3), turned to -90 degrees
- moved R10 7.12 mm to (184.2, 110.6)
- moved C10 7.00 mm to (186.7, 115.6)
- moved C8 7.00 mm to (186.7, 99.6)
- moved C9 7.00 mm to (168.9, 123.3)
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Connections:
- U4 pad 1: Net-(R14-Pad1) -> Net-(R15-Pad1)
- U4 pad 10: IN-2-3 -> GND
- U4 pad 12: GND -> IN-2-1
- U4 pad 13: Net-(R14-Pad2) -> Net-(R14-Pad1)
- U4 pad 14: Net-(R17-Pad2) -> Net-(R14-Pad1)
- U4 pad 2: Net-(R14-Pad1) -> Net-(R15-Pad1)
- U4 pad 3: IN-2-1 -> IN-2-2
- U4 pad 5: IN-2-2 -> IN-2-3
- U4 pad 6: Net-(R15-Pad1) -> Net-(R16-Pad1)
- U4 pad 7: Net-(R15-Pad1) -> Net-(R16-Pad1)
- U4 pad 8: Net-(R16-Pad1) -> Net-(R17-Pad2)
- U4 pad 9: Net-(R16-Pad1) -> Net-(R14-Pad2)
Routing:
- net IN-1-1: track 35.9 -> 124.0 mm
- net Net-(R4-Pad2): track 0.00 -> 67.6 mm
- net IN-2-1: track 0.00 -> 53.5 mm
- net Net-(R7-Pad2): track 0.00 -> 48.7 mm
- net IN-1-2: track 0.00 -> 44.6 mm
- net IN-1-3: track 0.00 -> 39.3 mm
- net Net-(R14-Pad2): track 0.00 -> 36.9 mm
- net IN-2-2: track 0.00 -> 33.9 mm
- net OUT-2: track 0.00 -> 31.2 mm
- net Net-(R17-Pad2): track 0.00 -> 31.1 mm
- net IN-2-3: track 0.00 -> 29.5 mm
- net +12V: track 95.7 -> 122.8 mm
- net Net-(R15-Pad1): track 0.00 -> 26.5 mm
- net OUT-1: track 0.00 -> 24.9 mm
- net -12V: track 103.6 -> 125.0 mm
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Other:
- board text added: "TODO - shuffle LED connections - adjust resistor positions - make it narrower"

Commit message: Adder - wip
Parts:
- moved R19 3.55 mm to (167.6, 95.2)
- moved D2 2.54 mm to (111.8, 130.0), turned to 180 degrees
Connections:
- J10 pad 10: LED-2-1 -> LED-1-1
- J10 pad 12: OUT-2 -> LED-2-1
- J10 pad 4: LED-1-1 -> OUT-1
- J10 pad 5: LED-1-2 -> IN-2-1
- J10 pad 6: OUT-1 -> IN-2-2
- J10 pad 7: IN-2-1 -> IN-2-3
- J10 pad 8: IN-2-2 -> OUT-2
- J10 pad 9: IN-2-3 -> LED-1-2
- J11 pad 10: LED-2-1 -> LED-1-1
- J11 pad 12: OUT-2 -> LED-2-1
- J11 pad 4: LED-1-1 -> OUT-1
- J11 pad 5: LED-1-2 -> IN-2-1
- J11 pad 6: OUT-1 -> IN-2-2
- J11 pad 7: IN-2-1 -> IN-2-3
- J11 pad 8: IN-2-2 -> OUT-2
- J11 pad 9: IN-2-3 -> LED-1-2
Routing:
- net OUT-2: track 31.2 -> 101.6 mm
- net LED-2-1: track 0.00 -> 60.8 mm
- net LED-2-2: track 3.81 -> 63.9 mm
- net LED-1-1: track 0.00 -> 53.7 mm, vias 0 -> 2
- net LED-1-2: track 3.81 -> 57.2 mm, vias 0 -> 2
- net OUT-1: track 24.9 -> 77.5 mm, vias 0 -> 1
- net IN-2-3: track 29.5 -> 59.9 mm
- net IN-2-1: track 53.5 -> 83.2 mm, vias 0 -> 1
- net IN-2-2: track 33.9 -> 48.6 mm
- net Net-(C2-Pad1): track 13.5 -> 17.3 mm

Commit message: Adder - wip
Parts:
- moved D1 2.54 mm to (109.2, 72.9), turned to 0 degrees
- renumbered R13 to R11, R11 to R13, R16 to R14, R14 to R16
Connections:
- J10 pad 5: IN-2-1 -> IN-2-3
- J10 pad 7: IN-2-3 -> IN-2-1
- J11 pad 5: IN-2-1 -> IN-2-3
- J11 pad 7: IN-2-3 -> IN-2-1
- R11 pad 1: IN-2-3 -> IN-2-1
- R13 pad 1: IN-2-1 -> IN-2-3
- U4 pad 12: IN-2-1 -> IN-2-3
- U4 pad 5: IN-2-3 -> IN-2-1
Routing:
- net IN-2-3: track 59.9 -> 92.8 mm
- net LED-1-1: track 53.7 -> 85.4 mm
- net IN-1-2: track 44.6 -> 72.6 mm
- net IN-1-1: track 124.0 -> 149.0 mm
- net IN-2-1: track 83.2 -> 62.1 mm
- net IN-1-3: track 39.3 -> 59.1 mm
- net LED-1-2: track 57.2 -> 75.2 mm
- net IN-2-2: track 48.6 -> 59.4 mm, vias 0 -> 1
- net OUT-1: track 77.5 -> 81.9 mm
- net OUT-2: track 101.6 -> 98.0 mm
- net LED-2-2: track 63.9 -> 65.7 mm
- net LED-2-1: track 60.8 -> 62.0 mm
Other:
- board text added: "TODO - adjust resistor positions - make it narrower"
- board text removed: "TODO - shuffle LED connections - adjust resistor positions - make it narrower"

Commit message: Adder - wip
Parts:
- moved G1 104.2 mm to (163.4, 140.7)
- moved G3 103.5 mm to (154.9, 140.6)
- moved J9 6.35 mm to (191.9, 139.7)
- moved C3 6.35 mm to (181.2, 129.5)
- moved C4 6.35 mm to (181.2, 139.4)
- moved R12 4.10 mm to (165.1, 72.1), turned to 90 degrees
- moved R11 4.06 mm to (165.1, 80.1), turned to -90 degrees
- moved C2 3.60 mm to (166.4, 99.6)
- moved R20 2.84 mm to (166.4, 103.4)
- moved R9 2.84 mm to (181.6, 103.4)
- moved R1 2.84 mm to (181.6, 48.4)
- moved R13 2.84 mm to (181.6, 72.4)
- moved R2 2.84 mm to (166.4, 48.4)
- moved R3 2.79 mm to (166.4, 55.9)
- moved R10 2.57 mm to (181.6, 111.0)
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Routing:
- net IN-1-1: track 149.0 -> 127.6 mm
- net IN-2-3: track 92.8 -> 87.0 mm
- net +12V: track 122.8 -> 117.4 mm
- net OUT-2: track 98.0 -> 92.6 mm
- net Net-(C2-Pad1): track 17.3 -> 12.5 mm
- net Net-(R17-Pad2): track 31.1 -> 27.1 mm
- net IN-2-2: track 59.4 -> 55.6 mm
- net IN-1-3: track 59.1 -> 55.3 mm
- net IN-2-1: track 62.1 -> 58.4 mm
- net Net-(R4-Pad2): track 67.6 -> 64.1 mm
- net LED-2-1: track 62.0 -> 58.6 mm
- net LED-1-2: track 75.2 -> 71.9 mm
- net OUT-1: track 81.9 -> 78.6 mm
- net LED-1-1: track 85.4 -> 82.4 mm
- net -12V: track 125.0 -> 121.9 mm
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Other:
- board size 101.3 x 108.2 mm -> 95 x 108.2 mm
- board text added: "TODO: clean up this PCB"
- board text removed: "TODO - adjust resistor positions - make it narrower"
- board text removed: "[title]"

Commit message: Adder - wip
Parts:
- moved R18 0.89 mm to (180.8, 95.2)
Connections:
- J10 pad 10: LED-1-1 -> OUT-2
- J10 pad 5: IN-2-3 -> LED-1-2
- J10 pad 6: IN-2-2 -> LED-1-1
- J10 pad 7: IN-2-1 -> IN-2-3
- J10 pad 8: OUT-2 -> IN-2-2
- J10 pad 9: LED-1-2 -> IN-2-1
- J11 pad 10: LED-1-1 -> OUT-2
- J11 pad 5: IN-2-3 -> LED-1-2
- J11 pad 6: IN-2-2 -> LED-1-1
- J11 pad 7: IN-2-1 -> IN-2-3
- J11 pad 8: OUT-2 -> IN-2-2
- J11 pad 9: LED-1-2 -> IN-2-1
Routing:
- net OUT-2: track 92.6 -> 86.8 mm
- net LED-1-1: track 82.4 -> 86.1 mm, vias 2 -> 1
- net LED-1-2: track 71.9 -> 70.5 mm, vias 2 -> 1
- net IN-2-1: track 58.4 -> 57.3 mm
- net Net-(C2-Pad1): track 12.5 -> 13.4 mm
- net OUT-1: track 78.6 -> 79.3 mm
- net IN-2-2: track 55.6 -> 55.1 mm

Commit message: Adder - wip
Routing:
- net LED-1-1: track 86.1 -> 81.7 mm
- net IN-2-1: track 57.3 -> 58.1 mm
Other:
- board text added: "TODO: move refdes"
- board text removed: "TODO: clean up this PCB"

Commit message: Adder - PCB finished
Parts:
- moved R18 0.89 mm to (180.0, 95.2)
Routing:
- net Net-(C2-Pad1): track 13.4 -> 12.5 mm
- net IN-2-3: track 86.6 -> 85.9 mm
- net OUT-1: track 79.3 -> 78.8 mm
Other:
- board text removed: "TODO: move refdes"
