File: modules/Adder/Adder.kicad_sch (KiCad schematic)
At the start: 28 parts, among them U1 LT1014, U2 LT1013, U3 TL072, U4 LT1014

Commit message: Adder - wip
Connections:
- net GND: now also U4.10 (+); no longer U4.12 (+)
- net IN-2-1: now also U4.12 (+); no longer U4.3 (+)
- net IN-2-2: now also U4.3 (+); no longer U4.5 (+)
- net IN-2-3: now also U4.5 (+); no longer U4.10 (+)
- net at R17.2, R18.1: now also U4.8; no longer U4.14
- net at R14.2, R15.2, R16.2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: now also U4.9 (-); no longer U4.13 (-)
- new net: R14.1, U4.13 (-), U4.14
- new net: R16.1, U4.6 (-), U4.7
- new net: R15.1, U4.1, U4.2 (-)
Changed lines of the file:
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@@
     (pin "4")
   )
-  (symbol (lib_id "-lmp-opamp:LT1014") (at 54.61 123.19 0) (unit 1)
+  (symbol (lib_id "-lmp-opamp:LT1014") (at 54.61 123.19 0) (unit 4)
     (in_bom yes) (on_board yes) (fields_autoplaced)
     (property "Reference" "U4" (id 0) (at 54.61 114.4102 0))
@@
     (pin "2")
   )
-  (symbol (lib_id "-lmp-opamp:LT1014") (at 54.61 166.37 0) (unit 3)
+  (symbol (lib_id "-lmp-opamp:LT1014") (at 54.61 166.37 0) (unit 2)
     (in_bom yes) (on_board yes) (fields_autoplaced)
     (property "Reference" "U4" (id 0) (at 54.61 157.5902 0))
@@
     (pin "2")
   )
-  (symbol (lib_id "-lmp-opamp:LT1014") (at 88.9 142.24 0) (mirror x) (unit 4)
+  (symbol (lib_id "-lmp-opamp:LT1014") (at 88.9 142.24 0) (mirror x) (unit 3)
     (in_bom yes) (on_board yes) (fields_autoplaced)
     (property "Reference" "U4" (id 0) (at 88.9 149.3504 0))
@@
     (pin "2")
   )
-  (symbol (lib_id "-lmp-opamp:LT1014") (at 54.61 144.78 0) (unit 2)
+  (symbol (lib_id "-lmp-opamp:LT1014") (at 54.61 144.78 0) (unit 1)
     (in_bom yes) (on_board yes) (fields_autoplaced)
     (property "Reference" "U4" (id 0) (at 54.61 136.0002 0))
@@
       (reference "U3") (unit 3) (value "TL072") (footprint "Package_DIP:DIP-8_W7.62mm")
     )
+    (path "/a4b43659-3bef-4f69-95d6-490780e9a28f"
+      (reference "U4") (unit 1) (value "LT1014") (footprint "Package_DIP:DIP-14_W7.62mm")
+    )
+    (path "/60c4ab7c-49dd-4160-b0aa-96a587a21680"
+      (reference "U4") (unit 2) (value "LT1014") (footprint "Package_DIP:DIP-14_W7.62mm")
+    )
+    (path "/6f3559d9-777f-4e6e-849f-4be419ce2125"
+      (reference "U4") (unit 3) (value "LT1014") (footprint "Package_DIP:DIP-14_W7.62mm")
+    )
     (path "/1b58f4b1-edd2-4fa2-957e-11921d049a8d"
-      (reference "U4") (unit 1) (value "LT1014") (footprint "Package_DIP:DIP-14_W7.62mm")
-    )
-    (path "/a4b43659-3bef-4f69-95d6-490780e9a28f"
-      (reference "U4") (unit 2) (value "LT1014") (footprint "Package_DIP:DIP-14_W7.62mm")
-    )
-    (path "/60c4ab7c-49dd-4160-b0aa-96a587a21680"
-      (reference "U4") (unit 3) (value "LT1014") (footprint "Package_DIP:DIP-14_W7.62mm")
-    )
-    (path "/6f3559d9-777f-4e6e-849f-4be419ce2125"
       (reference "U4") (unit 4) (value "LT1014") (footprint "Package_DIP:DIP-14_W7.62mm")
     )

Commit message: Adder - wip
Parts:
- renumbered R13 to R11, R11 to R13, R16 to R14, R14 to R16
Connections:
- net IN-2-1: now also R11.1, U4.5 (+); no longer R13.1, U4.12 (+)
- net IN-2-3: now also R13.1, U4.12 (+); no longer R11.1, U4.5 (+)
Other:
- moved on the sheet: R11, R13, R14, R16, U4B, U4D

Commit message: Adder - BOM and schematic pdf
Parts:
- R1, R11, R12, R13, R2, R3: DistributorPartLink https://www.mouser.ca/c/?m=YAGEO&power+rating=166+mW+(1%2f6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 -> https://www.mouser.ca/ProductDetail/YAGEO/MFR-12FTF52-1M?qs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; DistributorPartNum 603-MFR-12* -> 603-MFR-12FTF52-1M; ManufacturerPartNum MFR-12* -> MFR-12FTF52-1M; Value2 1%, 1/6 W -> 1% 1/6W
- R10, R20: Value2 1%, 1/4 W -> 1% 1/4W
- R21, R22: Note Output limiting -> (none); Value2 5%, 1/4 W -> 5% 1/4W
Changed lines of the file:
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@@
       (effects (font (size 1.27 1.27)) hide)
     )
-    (property "ManufacturerPartNum" "MFR-12*" (id 5) (at 38.1 125.73 0)
+    (property "ManufacturerPartNum" "MFR-12FTF52-1M" (id 5) (at 38.1 125.73 0)
       (effects (font (size 1.27 1.27)) hide)
     )
@@
       (effects (font (size 1.27 1.27)) hide)
     )
-    (property "DistributorPartNum" "603-MFR-12*" (id 7) (at 38.1 125.73 0)
-      (effects (font (size 1.27 1.27)) hide)
-    )
-    (property "DistributorPartLink" "https://www.mouser.ca/c/?m=YAGEO&power+rating=166+mW+(1%2f6+W)&tolerance=1+%25&instock=y" (id 8) (at 38.1 125.73 0)
-      (effects (font (size 1.27 1.27)) hide)
-    )
-    (property "Value2" "1%, 1/6 W" (id 9) (at 43.053 125.73 90)
+    (property "DistributorPartNum" "603-MFR-12FTF52-1M" (id 7) (at 38.1 125.73 0)
+      (effects (font (size 1.27 1.27)) hide)
+    )
+    (property "DistributorPartLink" "https://www.mouser.ca/ProductDetail/YAGEO/MFR-12FTF52-1M?qs=oAGoVhmvjhw%2F%2F4epxEjLtQ%3D%3D" (id 8) (at 38.1 125.73 0)
+      (effects (font (size 1.27 1.27)) hide)
+    )
+    (property "Value2" "1% 1/6W" (id 9) (at 43.053 125.73 90)
       (effects (font (size 1.27 1.27)) hide)
     )
@@
       (effects (font (size 1.27 1.27)) hide)
     )
-    (property "Value2" "1%, 1/4 W" (id 4) (at 137.16 142.6012 90))
+    (property "Value2" "1% 1/4W" (id 4) (at 137.16 142.6012 90))
     (property "Note" "Output limiting" (id 5) (at 139.065 146.685 90)
       (effects (font (size 1.27 1.27)) hide)
@@
       (effects (font (size 1.27 1.27)) hide)
     )
-    (property "ManufacturerPartNum" "MFR-12*" (id 5) (at 38.1 168.91 0)
+    (property "ManufacturerPartNum" "MFR-12FTF52-1M" (id 5) (at 38.1 168.91 0)
       (effects (font (size 1.27 1.27)) hide)
     )
@@
       (effects (font (size 1.27 1.27)) hide)
     )
-    (property "DistributorPartNum" "603-MFR-12*" (id 7) (at 38.1 168.91 0)
-      (effects (font (size 1.27 1.27)) hide)
-    )
-    (property "DistributorPartLink" "https://www.mouser.ca/c/?m=YAGEO&power+rating=166+mW+(1%2f6+W)&tolerance=1+%25&instock=y" (id 8) (at 38.1 168.91 0)
-      (effects (font (size 1.27 1.27)) hide)
-    )
-    (property "Value2" "1%, 1/6 W" (id 9) (at 43.053 168.91 90)
+    (property "DistributorPartNum" "603-MFR-12FTF52-1M" (id 7) (at 38.1 168.91 0)
+      (effects (font (size 1.27 1.27)) hide)
+    )
+    (property "DistributorPartLink" "https://www.mouser.ca/ProductDetail/YAGEO/MFR-12FTF52-1M?qs=oAGoVhmvjhw%2F%2F4epxEjLtQ%3D%3D" (id 8) (at 38.1 168.91 0)
+      (effects (font (size 1.27 1.27)) hide)
+    )
+    (property "Value2" "1% 1/6W" (id 9) (at 43.053 168.91 90)
       (effects (font (size 1.27 1.27)) hide)
     )
@@
       (effects (font (size 1.27 1.27)) hide)
     )
-    (property "ManufacturerPartNum" "MFR-12*" (id 5) (at 38.1 147.32 0)
+    (property "ManufacturerPartNum" "MFR-12FTF52-1M" (id 5) (at 38.1 147.32 0)
       (effects (font (size 1.27 1.27)) hide)
     )
@@
       (effects (font (size 1.27 1.27)) hide)
     )
-    (property "DistributorPartNum" "603-MFR-12*" (id 7) (at 38.1 147.32 0)
-      (effects (font (size 1.27 1.27)) hide)
-    )
-    (property "DistributorPartLink" "https://www.mouser.ca/c/?m=YAGEO&power+rating=166+mW+(1%2f6+W)&tolerance=1+%25&instock=y" (id 8) (at 38.1 147.32 0)
-      (effects (font (size 1.27 1.27)) hide)
-    )
-    (property "Value2" "1%, 1/6 W" (id 9) (at 43.053 147.32 90)
+    (property "DistributorPartNum" "603-MFR-12FTF52-1M" (id 7) (at 38.1 147.32 0)
+      (effects (font (size 1.27 1.27)) hide)
+    )
+    (property "DistributorPartLink" "https://www.mouser.ca/ProductDetail/YAGEO/MFR-12FTF52-1M?qs=oAGoVhmvjhw%2F%2F4epxEjLtQ%3D%3D" (id 8) (at 38.1 147.32 0)
+      (effects (font (size 1.27 1.27)) hide)
+    )
+    (property "Value2" "1% 1/6W" (id 9) (at 43.053 147.32 90)
       (effects (font (size 1.27 1.27)) hide)
     )
@@
       (effects (font (size 1.27 1.27)) hide)
     )
-    (property "ManufacturerPartNum" "MFR-12*" (id 5) (at 38.1 60.96 0)
+    (property "ManufacturerPartNum" "MFR-12FTF52-1M" (id 5) (at 38.1 60.96 0)
       (effects (font (size 1.27 1.27)) hide)
     )
@@
       (effects (font (size 1.27 1.27)) hide)
     )
-    (property "DistributorPartNum" "603-MFR-12*" (id 7) (at 38.1 60.96 0)
-      (effects (font (size 1.27 1.27)) hide)
-    )
-    (property "DistributorPartLink" "https://www.mouser.ca/c/?m=YAGEO&power+rating=166+mW+(1%2f6+W)&tolerance=1+%25&instock=y" (id 8) (at 38.1 60.96 0)
-      (effects (font (size 1.27 1.27)) hide)
-    )
-    (property "Value2" "1%, 1/6 W" (id 9) (at 43.053 60.96 90)
+    (property "DistributorPartNum" "603-MFR-12FTF52-1M" (id 7) (at 38.1 60.96 0)
+      (effects (font (size 1.27 1.27)) hide)
+    )
+    (property "DistributorPartLink" "https://www.mouser.ca/ProductDetail/YAGEO/MFR-12FTF52-1M?qs=oAGoVhmvjhw%2F%2F4epxEjLtQ%3D%3D" (id 8) (at 38.1 60.96 0)
+      (effects (font (size 1.27 1.27)) hide)
+    )
+    (property "Value2" "1% 1/6W" (id 9) (at 43.053 60.96 90)
       (effects (font (size 1.27 1.27)) hide)
     )
@@
       (effects (font (size 1.27 1.27)) hide)
     )
-    (property "ManufacturerPartNum" "MFR-12*" (id 5) (at 38.1 39.37 0)
+    (property "ManufacturerPartNum" "MFR-12FTF52-1M" (id 5) (at 38.1 39.37 0)
       (effects (font (size 1.27 1.27)) hide)
     )
@@
       (effects (font (size 1.27 1.27)) hide)
     )
-    (property "DistributorPartNum" "603-MFR-12*" (id 7) (at 38.1 39.37 0)
-      (effects (font (size 1.27 1.27)) hide)
-    )
-    (property "DistributorPartLink" "https://www.mouser.ca/c/?m=YAGEO&power+rating=166+mW+(1%2f6+W)&tolerance=1+%25&instock=y" (id 8) (at 38.1 39.37 0)
-      (effects (font (size 1.27 1.27)) hide)
-    )
-    (property "Value2" "1%, 1/6 W" (id 9) (at 43.053 39.37 90)
+    (property "DistributorPartNum" "603-MFR-12FTF52-1M" (id 7) (at 38.1 39.37 0)
+      (effects (font (size 1.27 1.27)) hide)
+    )
+    (property "DistributorPartLink" "https://www.mouser.ca/ProductDetail/YAGEO/MFR-12FTF52-1M?qs=oAGoVhmvjhw%2F%2F4epxEjLtQ%3D%3D" (id 8) (at 38.1 39.37 0)
+      (effects (font (size 1.27 1.27)) hide)
+    )
+    (property "Value2" "1% 1/6W" (id 9) (at 43.053 39.37 90)
       (effects (font (size 1.27 1.27)) hide)
     )
@@
       (effects (font (size 1.27 1.27)) hide)
     )
-    (property "Value2" "1%, 1/4 W" (id 4) (at 137.16 56.2412 90))
+    (property "Value2" "1% 1/4W" (id 4) (at 137.16 56.2412 90))
     (property "Note" "Output limiting" (id 5) (at 139.065 60.325 90)
       (effects (font (size 1.27 1.27)) hide)
@@
       (effects (font (size 1.27 1.27)) hide)
     )
-    (property "Value2" "5%, 1/4 W" (id 4) (at 139.1921 169.3407 0)
+    (property "Value2" "5% 1/4W" (id 4) (at 139.1921 169.3407 0)
       (effects (font (size 1.27 1.27)) (justify right))
     )
-    (property "Note" "Output limiting" (id 5) (at 139.065 168.275 90)
+    (property "Note" "" (id 5) (at 139.065 168.275 90)
       (effects (font (size 1.27 1.27)) hide)
     )
@@
       (effects (font (size 1.27 1.27)) hide)
     )
-    (property "Value2" "5%, 1/4 W" (id 4) (at 139.1921 82.9807 0)
+    (property "Value2" "5% 1/4W" (id 4) (at 139.1921 82.9807 0)
       (effects (font (size 1.27 1.27)) (justify right))
     )
-    (property "Note" "Output limiting" (id 5) (at 139.065 81.915 90)
+    (property "Note" "" (id 5) (at 139.065 81.915 90)
       (effects (font (size 1.27 1.27)) hide)
     )
@@
       (effects (font (size 1.27 1.27)) hide)
     )
-    (property "ManufacturerPartNum" "MFR-12*" (id 5) (at 38.1 82.55 0)
+    (property "ManufacturerPartNum" "MFR-12FTF52-1M" (id 5) (at 38.1 82.55 0)
       (effects (font (size 1.27 1.27)) hide)
     )
@@
       (effects (font (size 1.27 1.27)) hide)
     )
-    (property "DistributorPartNum" "603-MFR-12*" (id 7) (at 38.1 82.55 0)
-      (effects (font (size 1.27 1.27)) hide)
-    )
-    (property "DistributorPartLink" "https://www.mouser.ca/c/?m=YAGEO&power+rating=166+mW+(1%2f6+W)&tolerance=1+%25&instock=y" (id 8) (at 38.1 82.55 0)
-      (effects (font (size 1.27 1.27)) hide)
-    )
-    (property "Value2" "1%, 1/6 W" (id 9) (at 43.053 82.55 90)
-      (effects (font (size 1.27 1.27)) hide)
-    )
+    (property "DistributorPartNum" "603-MFR-12FTF52-1M" (id 7) (at 38.1 82.55 0)
+      (effects (font (size 1.27 1.27)) hide)
+    )
+    (property "DistributorPartLink" "https://www.mouser.ca/ProductDetail/YAGEO/MFR-12FTF52-1M?qs=oAGoVhmvjhw%2F%2F4epxEjLtQ%3D%3D" (id 8) (at 38.1 82.55 0)
+      (effects (font (size 1.27 1.27)) hide)
+    )
+    (property "Value2" "1% 1/6W" (id 9) (at 43.053 82.55 90)
+      (effects (font (size 1.27 1.27)) hide)
+    )
