File: modules/Mixer1/PanelPower.kicad_sch (KiCad schematic)
At the start: 45 parts, among them J1 WQP-PJ398, J10 Conn_PCB_Back, J11 Conn_PCB_Front, J12 Conn_PCB_Back, J13 Conn_Eurorack_10, J2 WQP-PJ398, J3 WQP-PJ398, J4 WQP-PJ398, J5 WQP-PJ398, J6 WQP-PJ398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

Commit message: Mixer1 - wip
Other:
- title: Eurorack Dual Mixer -> Front Panel & Power - Eurorack Mixer
Changed lines of the file:
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@@
   (paper "A4")
   (title_block
-    (title "Eurorack Dual Mixer")
-    (date "2022-10-03")
-    (rev "1.2")
+    (title "Front Panel & Power - Eurorack Mixer")
+    (date "2022-11-13")
+    (rev "1.0")
     (company "Len Popp")
     (comment 1 "Copyright © 2022 Len Popp CC BY")
-    (comment 2 "Layout designed for 8HP module using Delptronics Module Construction Set")
-    (comment 3 "Eurorack 2-channel 3:1 mixer module - 8HP")
+    (comment 2 "Eurorack 3:1 mixer module - 4HP")
   )

Commit message: Mixer1 - wip
Parts:
- removed C7, C8: 100N, -lmp-misc:C_Disc_D5.0mm_W2.5mm_P2.50mm, symbol -lmp:CC_100N
- removed D2: LED_Dual_5mm_ACA, LED_THT:LED_D5.0mm-3, symbol -lmp-synth:LED_Dual_5mm_Red_Green_ACA
- removed H1, H10, H5, H6: HW_Screw_M3x0.50x6, symbol -lmp-synth:HW_Screw_M3x0.50x6
- removed H2, H4, H7, H9: MountingHole_M3, -lmp-holes:MountingHole_PCB_3.2mm_M3, symbol -lmp-holes:MountingHole_PCB_M3
- removed H3, H8: HW_Standoff_F-F_11mm_M3x0.50, symbol -lmp-synth:HW_Standoff_F-F_11mm_M3x0.50
- removed J11: Conn_PCB_Front, Connector_PinSocket_2.54mm:PinSocket_1x09_P2.54mm_Vertical, symbol Connector_Generic:Conn_01x09
- removed J12: Conn_PCB_Back, Connector_PinHeader_2.54mm:PinHeader_1x09_P2.54mm_Vertical, symbol Connector_Generic:Conn_01x09
- removed J5, J6, J7, J8: WQP-PJ398, -lmp-synth:Jack_3.5mm_QingPu_WQP-PJ398SM_Vertical, symbol -lmp-synth:Jack_WQP-PJ398
- removed RV5, RV6, RV7, RV8: 100K, -lmp-synth:Potentiometer_Alpha_RD901F-40-00D_Single_Vertical, symbol -lmp-synth:R_POT_Panel_PCB_Alpha
- removed U2: TL074, Package_DIP:DIP-14_W7.62mm, symbol -lmp-opamp:TL074
- removed U3: TL072, Package_DIP:DIP-8_W7.62mm, symbol -lmp-opamp:TL072
- D1: Label Level 1 -> Level
- J1, RV1: Label Input 1-1 -> Input 1
- J2, RV2: Label Input 1-2 -> Input 2
- J3, RV3: Label Input 1-3 -> Input 3
- J4: Label Output 1 -> Output
- RV4: Label Gain 1 -> Gain
Connections:
- net GND: now also J10.9 (Pin_9), J4.TN, J9.9 (Pin_9)
- net GAIN-1 renamed GAIN
- net GAIN-ATTEN-1 renamed GAIN-ATTEN
- net IN-1-1 renamed IN-1
- net IN-1-2 renamed IN-2
- net IN-1-3 renamed IN-3
- net IN-ATTEN-1-1 renamed IN-ATTEN-1
- net IN-ATTEN-1-2 renamed IN-ATTEN-2
- net IN-ATTEN-1-3 renamed IN-ATTEN-3
- net LED-GREEN-1 renamed LED-GREEN
- net LED-RED-1 renamed LED-RED
- removed net OUT-1: J10.9 (Pin_9), J4.T, J9.9 (Pin_9)
- net OUT-1-NORMAL renamed OUT
- net OUT: now also J4.T; no longer J4.TN
- no-connect marks 1 -> 0
Other:
- note added: "TL071"
- note added: "U2"
- note removed: "Channel 1"
- note removed: "Channel 2"
- note removed: "Hardware"
- note removed: "OUT-1 is normalled to mix with channel 2"
- moved on the sheet: A1, C1, C2, C3, C4, C5, C6, J13, U1E
