File: modules/Mixer1/Mixer1.kicad_pcb (KiCad board)
At the start: 2 copper layers, 91.4 x 108.2 mm, 79 parts, among them J1 WQP-PJ398, J10 Conn_PCB_Back, J11 Conn_PCB_Front, J12 Conn_PCB_Back, J13 Conn_Eurorack_10, J2 WQP-PJ398, J3 WQP-PJ398, J4 WQP-PJ398, J5 WQP-PJ398, J6 WQP-PJ398, J7 WQP-PJ398, J8 WQP-PJ398, J9 Conn_PCB_Front, U1 TL074, U2 TL074, U3 TL072

Commit message: Mixer1 - wip
Other:
- board text added: "1Mix"
- board text removed: "2Mix"
Changed lines of the file:
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@@
   (paper "A4")
   (title_block
-    (title "Eurorack Dual Mixer")
-    (date "2022-10-03")
-    (rev "1.2")
+    (title "Eurorack Mixer")
+    (date "2022-11-13")
+    (rev "1.0")
     (company "Len Popp")
     (comment 1 "Copyright © 2022 Len Popp CC BY")
-    (comment 2 "Front panel layout matches 8HP Delptronics Module Construction Set")
-    (comment 3 "Board settings comply with requirements of OSH Park https://oshpark.com/")
-    (comment 4 "Eurorack 2-channel 3:1 mixer module - 8HP")
+    (comment 2 "Board settings comply with requirements of OSH Park https://oshpark.com/")
+    (comment 3 "Eurorack 3:1 mixer module - 4HP")
   )
   (layers
@@
     (effects (font (size 1 1) (thickness 0.15)) (justify right))
   )
-  (gr_text "2Mix" (at 153.035 41.798) (layer "F.SilkS")
+  (gr_text "1Mix" (at 153.035 41.798) (layer "F.SilkS")
     (effects (font (size 1.524 1.524) (thickness 0.2286)) (justify left))
   )
-  (gr_text "2Mix" (at 120.65 110.38) (layer "F.SilkS")
+  (gr_text "1Mix" (at 120.65 110.38) (layer "F.SilkS")
     (effects (font (size 1.524 1.524) (thickness 0.2286)))
   )

Commit message: Mixer1 - wip
Other:
- board text added: "1.95"
- board text added: "2.7"
- board text added: "3.45"
- board text added: "4,3.2"
- board text added: "4.2"
- board text added: "4.4557"
- board text added: "4.657"
- board text added: "5.21"
- board text added: "6.0134,3.2"
- board text added: "7.41,5.5"
- board text added: "7.5,3.2"
Changed lines of the file:
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@@
+    (effects (font (size 1.016 1.016) (thickness 0.1524)))
+  )
+  (gr_text "7.5,3.2" (at 196.088 81.153) (layer "Cmts.User")
+    (effects (font (size 1.016 1.016) (thickness 0.1524)))
+  )
+  (gr_text "4.657" (at 96.774 118.745) (layer "Cmts.User")
+    (effects (font (size 1.016 1.016) (thickness 0.1524)))
+  )
+  (gr_text "7.41,5.5" (at 195.834 126.873) (layer "Cmts.User")
+    (effects (font (size 1.016 1.016) (thickness 0.1524)))
+  )
+  (gr_text "1.95" (at 97.155 49.149) (layer "Cmts.User")
+    (effects (font (size 1.016 1.016) (thickness 0.1524)))
+  )
+  (gr_text "3.45" (at 96.901 88.138) (layer "Cmts.User")
+    (effects (font (size 1.016 1.016) (thickness 0.1524)))
+  )
+  (gr_text "5.21" (at 96.901 132.461) (layer "Cmts.User")
+    (effects (font (size 1.016 1.016) (thickness 0.1524)))
+  )
+  (gr_text "4.2" (at 96.647 106.045) (layer "Cmts.User")
+    (effects (font (size 1.016 1.016) (thickness 0.1524)))
+  )
+  (gr_text "2.7" (at 97.282 68.326) (layer "Cmts.User")
+    (effects (font (size 1.016 1.016) (thickness 0.1524)))
+  )
+  (gr_text "4,3.2" (at 97.155 81.153) (layer "Cmts.User")
+    (effects (font (size 1.016 1.016) (thickness 0.1524)))
+  )
+  (gr_text "6.0134,3.2" (at 149.733 79.248) (layer "Cmts.User")
+    (effects (font (size 1.016 1.016) (thickness 0.1524)))
+  )
+  (gr_text "4.4557" (at 96.52 112.903) (layer "Cmts.User")
     (effects (font (size 1.016 1.016) (thickness 0.1524)))
   )

Commit message: Mixer1 - wip
Parts:
- removed C10, C12, C13: 5P6, -lmp-misc:C_Disc_D5.0mm_W2.5mm_P2.50mm
- removed C11, C14: 100N, -lmp-misc:C_Disc_D5.0mm_W2.5mm_P2.50mm
- removed D4, D5, D6: 1N4148, Diode_THT:D_DO-35_SOD27_P7.62mm_Horizontal
- removed H2, H4, H7, H9: MountingHole_M3, -lmp-holes:MountingHole_PCB_3.2mm_M3
- removed J10, J12: Conn_PCB_Back, Connector_PinHeader_2.54mm:PinHeader_1x09_P2.54mm_Vertical
- removed J11, J9: Conn_PCB_Front, Connector_PinSocket_2.54mm:PinSocket_1x09_P2.54mm_Vertical
- removed J13: Conn_Eurorack_10, -lmp-synth:IDC-Header-Eurorack-10-TH
- removed J8: WQP-PJ398, -lmp-synth:Jack_3.5mm_QingPu_WQP-PJ398SM_Vertical
- removed R16, R17, R18, R20: 100K, -lmp-misc:R_Axial_DIN0207_L6.3mm_D2.5mm_P7.62mm_Horizontal
- removed R19: 51R, -lmp-misc:R_Axial_DIN0207_L6.3mm_D2.5mm_P10.16mm_Horizontal
- removed R21, R22: 10K, -lmp-misc:R_Axial_DIN0207_L6.3mm_D2.5mm_P7.62mm_Horizontal
- removed R23: 4K7, -lmp-misc:R_Axial_DIN0207_L6.3mm_D2.5mm_P7.62mm_Horizontal
- removed R24: 75K, -lmp-misc:R_Axial_DIN0207_L6.3mm_D2.5mm_P7.62mm_Horizontal
- removed R25: 11K, -lmp-misc:R_Axial_DIN0207_L6.3mm_D2.5mm_P7.62mm_Horizontal
- removed R26: 36K, -lmp-misc:R_Axial_DIN0207_L6.3mm_D2.5mm_P7.62mm_Horizontal
- removed R27: 200R, -lmp-misc:R_Axial_DIN0207_L6.3mm_D2.5mm_P7.62mm_Horizontal
- removed RV5, RV6, RV7, RV8: 100K, -lmp-synth:Potentiometer_Alpha_RD901F-40-00D_Single_Vertical
- removed U3: TL072, Package_DIP:DIP-8_W7.62mm
- C7: value 100N -> 5P6
- D2: value LED_Dual_5mm_ACA -> 1N4148; footprint LED_THT:LED_D5.0mm-3 -> Diode_THT:D_DO-35_SOD27_P7.62mm_Horizontal
- J5: value WQP-PJ398 -> Conn_PCB_Front; footprint -lmp-synth:Jack_3.5mm_QingPu_WQP-PJ398SM_Vertical -> Connector_PinSocket_2.54mm:PinSocket_1x09_P2.54mm_Vertical
- J6: value WQP-PJ398 -> Conn_PCB_Back; footprint -lmp-synth:Jack_3.5mm_QingPu_WQP-PJ398SM_Vertical -> Connector_PinHeader_2.54mm:PinHeader_1x09_P2.54mm_Horizontal
- J7: value WQP-PJ398 -> Conn_Eurorack_10; footprint -lmp-synth:Jack_3.5mm_QingPu_WQP-PJ398SM_Vertical -> -lmp-synth:IDC-Header-Eurorack-10-TH
- R1: value 100K -> 75K
- R10, R9: value 10K -> 100K
- R11: value 4K7 -> 100K
- R12: value 100K -> 51R; footprint -lmp-misc:R_Axial_DIN0207_L6.3mm_D2.5mm_P7.62mm_Horizontal -> -lmp-misc:R_Axial_DIN0207_L6.3mm_D2.5mm_P10.16mm_Horizontal
- R13, R14: value 100K -> 10K
- R15: value 100K -> 4K7
- R2: value 100K -> 11K
- R3: value 100K -> 36K
- R4: value 100K -> 200R
- R7: value 51R -> 100K; footprint -lmp-misc:R_Axial_DIN0207_L6.3mm_D2.5mm_P10.16mm_Horizontal -> -lmp-misc:R_Axial_DIN0207_L6.3mm_D2.5mm_P7.62mm_Horizontal
- U2: value TL074 -> TL071; footprint Package_DIP:DIP-14_W7.62mm -> Package_DIP:DIP-8_W7.62mm
- moved J4 145.3 mm to (228.1, 40.2)
- moved J1 137.5 mm to (228.1, 55.2)
- moved J2 127.3 mm to (232.1, 114.9)
- moved RV2 127.2 mm to (218.6, 132.6), turned to 0 degrees
- moved D1 120.2 mm to (227.5, 95.8)
- moved RV1 119.2 mm to (225.5, 72.8), turned to 0 degrees
- moved RV4 107.6 mm to (210.7, 72.8), turned to 0 degrees
- moved J3 106.3 mm to (222.0, 114.9)
- moved J5 106.3 mm to (198.0, 40.7)
- moved J6 98.6 mm to (198.0, 65.7)
- moved RV3 93.8 mm to (202.0, 96.5), turned to 0 degrees
- moved R15 84.9 mm to (199.6, 131.4), turned to 0 degrees
- moved R13 80.6 mm to (232.1, 87.8)
- moved R3 75.4 mm to (199.6, 135.5), turned to 0 degrees
- moved R14 72.7 mm to (197.8, 120.8)
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Connections:
- net IN-1-1 renamed IN-1
- net IN-1-2 renamed IN-2
- net IN-1-3 renamed IN-3
- C7 pad 1: +12V -> Net-(C7-Pad1)
- C7 pad 2: GND -> GAIN
- C8 pad 1: GND -> Net-(C8-Pad1)
- C8 pad 2: -12V -> GND
- C9 pad 2: GAIN-1 -> Net-(C9-Pad2)
- D1 pad 1: LED-RED-1 -> LED-RED
- D1 pad 3: LED-GREEN-1 -> LED-GREEN
- D2 pad 1: LED-RED-2 -> Net-(C8-Pad1)
- D2 pad 2: GND -> Net-(C9-Pad2)
- D3 pad 1: Net-(C11-Pad1) -> LED-RED
- D3 pad 2: Net-(C10-Pad2) -> GND
- J4 pad T: OUT-1 -> OUT
- J4 pad TN: OUT-1-NORMAL -> GND
- R1 pad 1: IN-ATTEN-1-1 -> +12V
- R1 pad 2: Net-(C9-Pad1) -> VREF-5
- R10 pad 1: Net-(R10-Pad1) -> GAIN-ATTEN
- R10 pad 2: LED-GREEN-1 -> Net-(C9-Pad1)
- R11 pad 1: Net-(R11-Pad1) -> Net-(C9-Pad1)
- R11 pad 2: LED-RED-1 -> Net-(C9-Pad2)
- R12 pad 1: IN-ATTEN-2-1 -> Net-(C9-Pad2)
- R12 pad 2: Net-(C12-Pad1) -> OUT
- R13 pad 1: IN-ATTEN-2-2 -> Net-(R13-Pad1)
- R13 pad 2: Net-(C12-Pad1) -> LED-GREEN
- R14 pad 1: IN-ATTEN-2-3 -> Net-(R14-Pad1)
- R14 pad 2: Net-(C12-Pad1) -> LED-GREEN
- R15 pad 1: OUT-1-NORMAL -> Net-(R15-Pad1)
- R15 pad 2: Net-(C12-Pad1) -> LED-RED
- R2 pad 1: IN-ATTEN-1-2 -> VREF-5
- R2 pad 2: Net-(C9-Pad1) -> VREF-4
- R3 pad 1: IN-ATTEN-1-3 -> VREF-4
- R3 pad 2: Net-(C9-Pad1) -> VREF-LO
- R4 pad 1: Net-(C9-Pad1) -> VREF-LO
- R4 pad 2: GAIN-1 -> GND
- R5 pad 1: GAIN-ATTEN-1 -> IN-ATTEN-1
- R5 pad 2: Net-(C10-Pad1) -> Net-(C7-Pad1)
- R6 pad 1: Net-(C10-Pad1) -> IN-ATTEN-2
- R6 pad 2: Net-(C10-Pad2) -> Net-(C7-Pad1)
- R7 pad 1: Net-(C10-Pad2) -> IN-ATTEN-3
- R7 pad 2: OUT-1 -> Net-(C7-Pad1)
- R8 pad 1: GND -> Net-(C7-Pad1)
- R8 pad 2: Net-(C11-Pad1) -> GAIN
- R9 pad 1: Net-(R9-Pad1) -> GND
- R9 pad 2: LED-GREEN-1 -> Net-(C8-Pad1)
- RV1 pad 2: IN-ATTEN-1-1 -> IN-ATTEN-1
- RV2 pad 2: IN-ATTEN-1-2 -> IN-ATTEN-2
- RV3 pad 2: IN-ATTEN-1-3 -> IN-ATTEN-3
- RV4 pad 2: GAIN-ATTEN-1 -> GAIN-ATTEN
- RV4 pad 3: GAIN-1 -> GAIN
- U1 pad 1: GAIN-2 -> GAIN
- U1 pad 10: GND -> VREF-5
- U1 pad 14: GAIN-1 -> Net-(C9-Pad2)
- U1 pad 2: Net-(C12-Pad1) -> Net-(C7-Pad1)
- U1 pad 5: GND -> Net-(C8-Pad1)
- U1 pad 6: Net-(C13-Pad1) -> VREF-LO
- U1 pad 7: Net-(C13-Pad2) -> Net-(R14-Pad1)
- U1 pad 8: Net-(C10-Pad2) -> Net-(R13-Pad1)
- U1 pad 9: Net-(C10-Pad1) -> Net-(C8-Pad1)
- U2 pad 1: Net-(R21-Pad1) -> unconnected-(U2-Pad1)
- U2 pad 2: Net-(C14-Pad1) -> VREF-4
- U2 pad 3: VREF-5 -> Net-(C8-Pad1)
- U2 pad 4: +12V -> -12V
- U2 pad 5: Net-(C14-Pad1) -> unconnected-(U2-Pad5)
- U2 pad 6: VREF-LO -> Net-(R15-Pad1)
- U2 pad 7: Net-(R22-Pad1) -> +12V
- U2 pad 8: Net-(R9-Pad1) -> unconnected-(U2-Pad8)
Routing:
- net -12V: track 142.6 -> 0.00 mm, vias 2 -> 0
- net +12V: track 138.0 -> 0.00 mm
- net OUT-1-NORMAL: track 111.8 -> 0.00 mm
- net IN-2-1: track 93.3 -> 0.00 mm
- net IN-2-2: track 89.8 -> 0.00 mm, vias 1 -> 0
- net IN-1: track 87.2 -> 0.00 mm
- net IN-2: track 84.8 -> 0.00 mm, vias 1 -> 0
- net GAIN-2: track 74.2 -> 0.00 mm
- net GAIN-1: track 71.8 -> 0.00 mm
- net OUT-1: track 64.9 -> 0.00 mm
- net LED-RED-1: track 63.1 -> 0.00 mm
- net OUT-2: track 62.2 -> 0.00 mm
- net LED-RED-2: track 60.1 -> 0.00 mm
- net Net-(C14-Pad1): track 60.1 -> 0.00 mm
- net Net-(C11-Pad1): track 59.4 -> 0.00 mm, vias 1 -> 0
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
Commit message: Mixer1 - wip
Parts:
- G2, G4, J5, J6: moved to B.Cu
- moved J4 127.0 mm to (140.7, 132.3)
- moved J1 116.1 mm to (130.7, 118.3)
- moved RV2 106.7 mm to (133.2, 68.6), turned to 90 degrees
- moved J2 102.9 mm to (130.7, 132.3)
- moved D1 95.9 mm to (133.2, 113.2)
- moved RV1 95.2 mm to (133.2, 49.5), turned to 90 degrees
- moved D3 88.6 mm to (148.8, 114.0)
- moved R13 88.6 mm to (148.8, 117.8)
- moved RV4 84.6 mm to (133.2, 106.7), turned to 90 degrees
- moved J5 81.7 mm to (127.0, 81.3), turned to 180 degrees
- moved J3 81.3 mm to (140.7, 118.3)
- moved R1 74.7 mm to (148.6, 67.3)
- moved R5 74.7 mm to (148.6, 63.3)
- moved R4 70.5 mm to (150.9, 82.9)
- moved R9 70.5 mm to (150.9, 87.0)
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Routing:
- net IN-1: track 0.00 -> 86.8 mm
- net IN-2: track 0.00 -> 82.4 mm, vias 0 -> 1
- net OUT: track 0.00 -> 56.7 mm, vias 0 -> 1
- net IN-3: track 0.00 -> 46.5 mm, vias 0 -> 1
- net IN-ATTEN-1: track 0.00 -> 35.3 mm
- net LED-GREEN: track 0.00 -> 30.8 mm
- net GAIN: track 0.00 -> 26.7 mm
- net LED-RED: track 0.00 -> 24.9 mm
- net GAIN-ATTEN: track 0.00 -> 21.6 mm
- net IN-ATTEN-2: track 0.00 -> 20.9 mm
- net IN-ATTEN-3: track 0.00 -> 10.6 mm
Other:
- board size 91.4 x 108.2 mm -> 91.1 x 108.2 mm
- board text removed: "1.95"
- board text removed: "2.7"
- board text removed: "3.45"
- board text removed: "4,3.2"
- board text removed: "4.2"
- board text removed: "4.4557"
- board text removed: "4.657"
- board text removed: "5.21"
- board text removed: "6.0134,3.2"
- board text removed: "7.41,5.5"
- board text removed: "7.5,3.2"

Commit message: Mixer1 - wip
Parts:
- moved R14 77.9 mm to (204.5, 66.5)
- moved R7 72.0 mm to (180.2, 75.7)
- moved R3 66.6 mm to (205.9, 97.3), turned to 180 degrees
- moved R9 61.7 mm to (212.1, 79.2), turned to 180 degrees
- moved R2 60.6 mm to (205.1, 101.2)
- moved R13 60.1 mm to (201.7, 89.2), turned to 180 degrees
- moved C8 58.9 mm to (205.3, 75.6)
- moved C7 57.9 mm to (190.9, 69.1), turned to 90 degrees
- moved R1 56.7 mm to (194.1, 101.2)
- moved C4 56.7 mm to (207.8, 71.9), turned to 180 degrees
- moved R8 52.8 mm to (180.2, 65.8)
- moved R4 48.5 mm to (198.2, 93.5)
- moved C6 48.2 mm to (207.8, 106.3), turned to 180 degrees
- moved C9 48.2 mm to (188.7, 82.4)
- moved R15 45.8 mm to (190.9, 108.0), turned to 180 degrees
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Connections:
- U1 pad 12: GND -> Net-(C8-Pad1)
- U1 pad 13: Net-(C9-Pad1) -> VREF-LO
- U1 pad 14: Net-(C9-Pad2) -> Net-(R14-Pad1)
- U1 pad 5: Net-(C8-Pad1) -> GND
- U1 pad 6: VREF-LO -> Net-(C9-Pad1)
- U1 pad 7: Net-(R14-Pad1) -> Net-(C9-Pad2)
Routing:
- net -12V: track 0.00 -> 89.8 mm, vias 0 -> 1
- net +12V: track 0.00 -> 82.0 mm, vias 0 -> 2
- net Net-(C8-Pad1): track 0.00 -> 54.4 mm, vias 0 -> 2
- net LED-GREEN: track 30.8 -> 80.8 mm, vias 0 -> 1
- net GAIN: track 26.7 -> 61.4 mm
- net VREF-LO: track 0.00 -> 30.2 mm
- net LED-RED: track 24.9 -> 54.3 mm
- net VREF-5: track 0.00 -> 29.3 mm
- net VREF-4: track 0.00 -> 25.7 mm
- net Net-(C7-Pad1): track 0.00 -> 21.8 mm
- net Net-(C9-Pad2): track 0.00 -> 16.2 mm
- net GAIN-ATTEN: track 21.6 -> 36.5 mm
- net IN-ATTEN-2: track 20.9 -> 34.5 mm
- net IN-ATTEN-1: track 35.3 -> 48.9 mm
- net IN-ATTEN-3: track 10.6 -> 22.6 mm
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
Commit message: Mixer1 - wip
Parts:
- moved G3 88.7 mm to (180.8, 128.0)
- moved G1 84.6 mm to (188.6, 128.3)
- moved C1 11.2 mm to (199.5, 118.6)
- moved J7 11.2 mm to (210.9, 128.8)
- moved C2 11.2 mm to (199.7, 128.0)
- moved G2 1.35 mm to (140.1, 93.1)
- moved G4 1.20 mm to (131.6, 93.0)
Routing:
- net -12V: track 89.8 -> 77.9 mm
- net +12V: track 82.0 -> 70.2 mm
- net IN-1: track 86.8 -> 89.3 mm
- net IN-2: track 82.4 -> 83.5 mm
- net GAIN: track 61.4 -> 60.5 mm
- net OUT: track 65.4 -> 65.9 mm
Other:
- board size 91.1 x 108.2 mm -> 88.8 x 108.2 mm

Commit message: Mixer1: gerber files
Routing:
- net GAIN-ATTEN: track 36.5 -> 35.7 mm
Changed lines of the file:
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@@
       (drillshape 0)
       (scaleselection 1)
-      (outputdirectory "gerbers/")
+      (outputdirectory "gerbers/gerbers/")
     )
   )
@@
   (segment (start 202.992004 128.778) (end 202.230004 128.016) (width 0.762) (layer "B.Cu") (net 3))
   (segment (start 201.676 74.168) (end 202.966 74.168) (width 0.762) (layer "B.Cu") (net 3))
+  (segment (start 181.864 84.836) (end 181.864 78.359) (width 0.381) (layer "F.Cu") (net 4))
   (segment (start 194.056 66.548) (end 190.921 66.548) (width 0.381) (layer "F.Cu") (net 4))
-  (segment (start 181.864 78.359) (end 186.055 74.168) (width 0.381) (layer "F.Cu") (net 4))
+  (segment (start 184.658 68.961) (end 187.833 65.786) (width 0.381) (layer "F.Cu") (net 4))
+  (segment (start 177.8 88.9) (end 181.864 84.836) (width 0.381) (layer "F.Cu") (net 4))
   (segment (start 136.906 104.775) (end 136.906 91.567) (width 0.381) (layer "F.Cu") (net 4))
   (segment (start 138.18 106.049) (end 136.906 104.775) (width 0.381) (layer "F.Cu") (net 4))
-  (segment (start 177.8 88.9) (end 181.864 84.836) (width 0.381) (layer "F.Cu") (net 4))
   (segment (start 187.833 65.786) (end 190.079 65.786) (width 0.381) (layer "F.Cu") (net 4))
   (segment (start 135.128 89.789) (end 127.889 89.789) (width 0.381) (layer "F.Cu") (net 4))
+  (segment (start 181.864 78.359) (end 184.658 75.565) (width 0.381) (layer "F.Cu") (net 4))
   (segment (start 190.079 65.786) (end 190.881 66.588) (width 0.381) (layer "F.Cu") (net 4))
-  (segment (start 186.055 67.564) (end 187.833 65.786) (width 0.381) (layer "F.Cu") (net 4))
   (segment (start 136.906 91.567) (end 135.128 89.789) (width 0.381) (layer "F.Cu") (net 4))
-  (segment (start 181.864 84.836) (end 181.864 78.359) (width 0.381) (layer "F.Cu") (net 4))
+  (segment (start 184.658 75.565) (end 184.658 68.961) (width 0.381) (layer "F.Cu") (net 4))
   (segment (start 190.921 66.548) (end 190.881 66.588) (width 0.381) (layer "F.Cu") (net 4))
   (segment (start 138.18 106.68) (end 138.18 106.049) (width 0.381) (layer "F.Cu") (net 4))
   (segment (start 127.889 89.789) (end 127 88.9) (width 0.381) (layer "F.Cu") (net 4))
-  (segment (start 186.055 74.168) (end 186.055 67.564) (width 0.381) (layer "F.Cu") (net 4))
   (segment (start 191.262 78.994) (end 193.802 78.994) (width 0.381) (layer "F.Cu") (net 5))
   (segment (start 188.742 82.423) (end 188.742 83.673) (width 0.381) (layer "F.Cu") (net 5))
@@
   (segment (start 188.087 103.124) (end 183.261 107.95) (width 0.381) (layer "F.Cu") (net 9))
   (segment (start 183.261 107.95) (end 183.261 114.808) (width 0.381) (layer "F.Cu") (net 9))
-  (segment (start 134.493 97.155) (end 131.318 93.98) (width 0.381) (layer "F.Cu") (net 10))
-  (segment (start 134.874 109.347) (end 132.08 109.347) (width 0.381) (layer "F.Cu") (net 10))
-  (segment (start 131.191 108.458) (end 131.191 104.902) (width 0.381) (layer "F.Cu") (net 10))
+  (segment (start 131.191 104.902) (end 134.493 101.6) (width 0.381) (layer "F.Cu") (net 10))
   (segment (start 189.23 93.98) (end 187.325 93.98) (width 0.381) (layer "F.Cu") (net 10))
   (segment (start 194.056 89.154) (end 189.23 93.98) (width 0.381) (layer "F.Cu") (net 10))
-  (segment (start 138.26 112.733) (end 134.874 109.347) (width 0.381) (layer "F.Cu") (net 10))
   (segment (start 207.137 78.994) (end 212.09 74.041) (width 0.381) (layer "F.Cu") (net 10))
+  (segment (start 130.937 93.98) (end 127 93.98) (width 0.381) (layer "F.Cu") (net 10))
+  (segment (start 134.493 97.536) (end 130.937 93.98) (width 0.381) (layer "F.Cu") (net 10))
+  (segment (start 134.493 101.6) (end 134.493 97.536) (width 0.381) (layer "F.Cu") (net 10))
+  (segment (start 134.874 109.347) (end 132.08 109.347) (width 0.381) (layer "F.Cu") (net 10))
   (segment (start 138.26 113.175) (end 138.26 112.733) (width 0.381) (layer "F.Cu") (net 10))
-  (segment (start 134.493 101.6) (end 134.493 97.155) (width 0.381) (layer "F.Cu") (net 10))
-  (segment (start 132.08 109.347) (end 131.191 108.458) (width 0.381) (layer "F.Cu") (net 10))
-  (segment (start 131.318 93.98) (end 127 93.98) (width 0.381) (layer "F.Cu") (net 10))
   (segment (start 187.325 93.98) (end 177.8 93.98) (width 0.381) (layer "F.Cu") (net 10))
-  (segment (start 131.191 104.902) (end 134.493 101.6) (width 0.381) (layer "F.Cu") (net 10))
+  (segment (start 131.191 108.458) (end 131.191 104.902) (width 0.381) (layer "F.Cu") (net 10))
+  (segment (start 138.26 112.733) (end 134.874 109.347) (width 0.381) (layer "F.Cu") (net 10))
   (segment (start 212.09 74.041) (end 212.09 66.548) (width 0.381) (layer "F.Cu") (net 10))
+  (segment (start 132.08 109.347) (end 131.191 108.458) (width 0.381) (layer "F.Cu") (net 10))
   (via (at 207.137 78.994) (size 0.762) (drill 0.381) (layers "F.Cu" "B.Cu") (net 10))
   (segment (start 199.263 85.344) (end 195.453 89.154) (width 0.381) (layer "B.Cu") (net 10))
@@
   (segment (start 207.137 78.994) (end 200.787 85.344) (width 0.381) (layer "B.Cu") (net 10))
   (segment (start 200.787 85.344) (end 199.263 85.344) (width 0.381) (layer "B.Cu") (net 10))
-  (segment (start 138.176 102.616) (end 138.176 91.186) (width 0.381) (layer "F.Cu") (net 11))
-  (segment (start 140.680284 113.319716) (end 140.680284 105.120284) (width 0.381) (layer "F.Cu") (net 11))
+  (segment (start 134.874 119.126) (end 140.081 113.919) (width 0.381) (layer "F.Cu") (net 11))
+  (segment (start 140.081 104.521) (end 138.176 102.616) (width 0.381) (layer "F.Cu") (net 11))
+  (segment (start 143.002 54.352) (end 138.18 49.53) (width 0.381) (layer "F.Cu") (net 11))
   (segment (start 138.176 91.186) (end 143.002 86.36) (width 0.381) (layer "F.Cu") (net 11))
   (segment (start 134.874 125.5338) (end 134.874 119.126) (width 0.381) (layer "F.Cu") (net 11))
-  (segment (start 140.680284 105.120284) (end 138.176 102.616) (width 0.381) (layer "F.Cu") (net 11))
-  (segment (start 143.002 54.352) (end 138.18 49.53) (width 0.381) (layer "F.Cu") (net 11))
   (segment (start 143.002 86.36) (end 143.002 54.352) (width 0.381) (layer "F.Cu") (net 11))
-  (segment (start 134.874 119.126) (end 140.680284 113.319716) (width 0.381) (layer "F.Cu") (net 11))
   (segment (start 130.72 129.6878) (end 134.874 125.5338) (width 0.381) (layer "F.Cu") (net 11))
+  (segment (start 138.176 102.616) (end 138.176 91.186) (width 0.381) (layer "F.Cu") (net 11))
+  (segment (start 140.081 113.919) (end 140.081 104.521) (width 0.381) (layer "F.Cu") (net 11))
   (segment (start 142.875 112.903) (end 136.906 118.872) (width 0.381) (layer "F.Cu") (net 12))
   (segment (start 136.906 137.548) (end 130.72 143.734) (width 0.381) (layer "F.Cu") (net 12))
@@
   (segment (start 144.399 93.853) (end 144.399 93.849) (width 0.381) (layer "B.Cu") (net 13))
   (segment (start 144.399 93.849) (end 138.18 87.63) (width 0.381) (layer "B.Cu") (net 13))
-  (segment (start 128.905 100.584) (end 127.381 99.06) (width 0.381) (layer "F.Cu") (net 14))
+  (segment (start 127.762 103.759) (end 128.905 102.616) (width 0.381) (layer "F.Cu") (net 14))
   (segment (start 177.927 99.187) (end 177.8 99.06) (width 0.381) (layer "F.Cu") (net 14))
-  (segment (start 127.762 140.462) (end 127.762 110.49) (width 0.381) (layer "F.Cu") (net 14))
-  (segment (start 186.436 99.187) (end 177.927 99.187) (width 0.381) (layer "F.Cu") (net 14))
-  (segment (start 127.762 110.49) (end 128.905 109.347) (width 0.381) (layer "F.Cu") (net 14))
   (segment (start 127.381 99.06) (end 127 99.06) (width 0.381) (layer "F.Cu") (net 14))
-  (segment (start 128.905 109.347) (end 128.905 100.584) (width 0.381) (layer "F.Cu") (net 14))
+  (segment (start 128.905 100.584) (end 127.381 99.06) (width 0.381) (layer "F.Cu") (net 14))
+  (segment (start 128.905 102.616) (end 128.905 100.584) (width 0.381) (layer "F.Cu") (net 14))
+  (segment (start 186.436 99.187) (end 177.927 99.187) (width 0.381) (layer "F.Cu") (net 14))
+  (segment (start 127.762 140.462) (end 127.762 103.759) (width 0.381) (layer "F.Cu") (net 14))
   (via (at 127.762 140.462) (size 0.762) (drill 0.381) (layers "F.Cu" "B.Cu") (net 14))
   (segment (start 138.738 141.732) (end 129.413 141.732) (width 0.381) (layer "B.Cu") (net 14))
@@
   (segment (start 180.721 76.2) (end 180.213 75.692) (width 0.381) (layer "F.Cu") (net 17))
   (segment (start 134.874 85.598) (end 127.762 85.598) (width 0.381) (layer "F.Cu") (net 17))
-  (segment (start 135.68 106.68) (end 135.68 95.421) (width 0.381) (layer "F.Cu") (net 18))
-  (segment (start 135.68 95.421) (end 131.699 91.44) (width 0.381) (layer "F.Cu") (net 18))
   (segment (start 183.642 85.598) (end 177.8 91.44) (width 0.381) (layer "F.Cu") (net 18))
-  (segment (start 131.699 91.44) (end 127 91.44) (width 0.381) (layer "F.Cu") (net 18))
+  (segment (start 130.3655 91.44) (end 127 91.44) (width 0.381) (layer "F.Cu") (net 18))
+  (segment (start 135.68 96.7545) (end 130.3655 91.44) (width 0.381) (layer "F.Cu") (net 18))
+  (segment (start 135.68 106.68) (end 135.68 96.7545) (width 0.381) (layer "F.Cu") (net 18))
   (segment (start 183.642 78.994) (end 183.642 85.598) (width 0.381) (layer "F.Cu") (net 18))
   (segment (start 201.676 89.154) (end 201.676 81.788) (width 0.381) (layer "F.Cu") (net 19))

Commit message: Mixer1: - clean up schematic - fix output jack connection
Connections:
- J4 pad TN: GND -> unconnected-(J4-PadTN)
