File: modules/VCF-SV/proto/proto.kicad_pcb (KiCad board)
At the start: 6 copper layers, 40.6 x 101.6 mm, 34 parts, among them J1 Conn_01x09, U1 TL074, U2 CEM3320

Commit message: VCF-SV: proto - update pcb.png
Other:
- board text added: "15"
- board text added: "20"
- board text added: "25"
- board text added: "30"
- board text added: "35"
- board text added: "40"
- board text removed: "21"
- board text removed: "31"
- board text removed: "41"
Changed lines of the file:
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@@
   (gr_line (start 82.55 135.89) (end 82.55 34.29) (layer "Edge.Cuts") (width 0.1))
   (gr_line (start 82.55 34.29) (end 123.19 34.29) (layer "Edge.Cuts") (width 0.1))
-  (gr_text "21" (at 80.645 60.96) (layer "Cmts.User")
+  (gr_text "20" (at 80.645 58.305159) (layer "Cmts.User")
+    (effects (font (size 1.524 1.524) (thickness 0.2286)))
+  )
+  (gr_text "25" (at 125.095 71.12) (layer "Cmts.User")
     (effects (font (size 1.524 1.524) (thickness 0.2286)))
   )
   (gr_text "CV1" (at 104.14 134.62) (layer "Cmts.User")
     (effects (font (size 1.524 1.524) (thickness 0.254)))
+  )
+  (gr_text "15" (at 80.563391 45.605159) (layer "Cmts.User")
+    (effects (font (size 1.524 1.524) (thickness 0.2286)))
   )
   (gr_text "11" (at 125.095 35.56) (layer "Cmts.User")
@@
     (effects (font (size 1.524 1.524) (thickness 0.2286)))
   )
-  (gr_text "31" (at 125.095 86.36) (layer "Cmts.User")
+  (gr_text "30" (at 125.349 83.82) (layer "Cmts.User")
     (effects (font (size 1.524 1.524) (thickness 0.2286)))
   )
-  (gr_text "31" (at 80.645 86.36) (layer "Cmts.User")
+  (gr_text "30" (at 80.645 83.705159) (layer "Cmts.User")
     (effects (font (size 1.524 1.524) (thickness 0.2286)))
   )
-  (gr_text "21" (at 125.095 60.96) (layer "Cmts.User")
+  (gr_text "15" (at 125.095 45.72) (layer "Cmts.User")
+    (effects (font (size 1.524 1.524) (thickness 0.2286)))
+  )
+  (gr_text "20" (at 125.222 58.42) (layer "Cmts.User")
     (effects (font (size 1.524 1.524) (thickness 0.2286)))
   )
@@
     (effects (font (size 1.524 1.524) (thickness 0.254)))
   )
-  (gr_text "41" (at 125.095 111.76) (layer "Cmts.User")
+  (gr_text "25" (at 80.645 71.005159) (layer "Cmts.User")
     (effects (font (size 1.524 1.524) (thickness 0.2286)))
   )
-  (gr_text "41" (at 80.645 111.76) (layer "Cmts.User")
+  (gr_text "40" (at 125.222 109.22) (layer "Cmts.User")
     (effects (font (size 1.524 1.524) (thickness 0.2286)))
   )
+  (gr_text "40" (at 80.645 109.105159) (layer "Cmts.User")
+    (effects (font (size 1.524 1.524) (thickness 0.2286)))
+  )
+  (gr_text "35" (at 125.095 96.52) (layer "Cmts.User")
+    (effects (font (size 1.524 1.524) (thickness 0.2286)))
+  )
+  (gr_text "35" (at 80.645 96.405159) (layer "Cmts.User")
+    (effects (font (size 1.524 1.524) (thickness 0.2286)))
+  )

Commit message: VCF-SV: proto - update pcb.png
Other:
- board text added: "X"
Changed lines of the file:
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@@
     (effects (font (size 1.524 1.524) (thickness 0.2286)))
+  )
+  (gr_text "X" (at 85.09 83.82) (layer "Cmts.User")
+    (effects (font (size 1.27 1.27) (thickness 0.2032)))
   )
   (gr_text "25" (at 125.095 71.12) (layer "Cmts.User")
     (effects (font (size 1.524 1.524) (thickness 0.2286)))
   )
+  (gr_text "X" (at 132.08 38.735) (layer "Cmts.User")
+    (effects (font (size 1.27 1.27) (thickness 0.2032)))
+  )
   (gr_text "CV1" (at 104.14 134.62) (layer "Cmts.User")
     (effects (font (size 1.524 1.524) (thickness 0.254)))
+  )
+  (gr_text "X" (at 115.558799 64.761116) (layer "Cmts.User")
+    (effects (font (size 1.27 1.27) (thickness 0.2032)))
+  )
+  (gr_text "X" (at 102.87 50.8) (layer "Cmts.User")
+    (effects (font (size 1.27 1.27) (thickness 0.2032)))
+  )
+  (gr_text "X" (at 86.995 88.9) (layer "Cmts.User")
+    (effects (font (size 1.27 1.27) (thickness 0.2032)))
+  )
+  (gr_text "X" (at 87.581019 104.207266) (layer "Cmts.User")
+    (effects (font (size 1.27 1.27) (thickness 0.2032)))
+  )
+  (gr_text "X" (at 87.63 101.6) (layer "Cmts.User")
+    (effects (font (size 1.27 1.27) (thickness 0.2032)))
   )
   (gr_text "15" (at 80.563391 45.605159) (layer "Cmts.User")
@@
     (effects (font (size 1.524 1.524) (thickness 0.2286)))
   )
+  (gr_text "X" (at 120.015 52.705) (layer "Cmts.User")
+    (effects (font (size 1.27 1.27) (thickness 0.2032)))
+  )
+  (gr_text "X" (at 95.25 86.36) (layer "Cmts.User")
+    (effects (font (size 1.27 1.27) (thickness 0.2032)))
+  )
   (gr_text "30" (at 125.349 83.82) (layer "Cmts.User")
     (effects (font (size 1.524 1.524) (thickness 0.2286)))
+  )
+  (gr_text "X" (at 104.09043 36.783336) (layer "Cmts.User")
+    (effects (font (size 1.27 1.27) (thickness 0.2032)))
+  )
+  (gr_text "X" (at 111.76 45.72) (layer "Cmts.User")
+    (effects (font (size 1.27 1.27) (thickness 0.2032)))
   )
   (gr_text "30" (at 80.645 83.705159) (layer "Cmts.User")
     (effects (font (size 1.524 1.524) (thickness 0.2286)))
   )
+  (gr_text "X" (at 119.38 39.37) (layer "Cmts.User")
+    (effects (font (size 1.27 1.27) (thickness 0.2032)))
+  )
+  (gr_text "X" (at 102.830169 104.08124) (layer "Cmts.User")
+    (effects (font (size 1.27 1.27) (thickness 0.2032)))
+  )
+  (gr_text "X" (at 104.14 71.755) (layer "Cmts.User")
+    (effects (font (size 1.27 1.27) (thickness 0.2032)))
+  )
+  (gr_text "X" (at 103.505 46.99) (layer "Cmts.User")
+    (effects (font (size 1.27 1.27) (thickness 0.2032)))
+  )
+  (gr_text "X" (at 118.11 104.14) (layer "Cmts.User")
+    (effects (font (size 1.27 1.27) (thickness 0.2032)))
+  )
   (gr_text "15" (at 125.095 45.72) (layer "Cmts.User")
     (effects (font (size 1.524 1.524) (thickness 0.2286)))
+  )
+  (gr_text "X" (at 86.950889 68.541898) (layer "Cmts.User")
+    (effects (font (size 1.27 1.27) (thickness 0.2032)))
+  )
+  (gr_text "X" (at 87.581019 66.021377) (layer "Cmts.User")
+    (effects (font (size 1.27 1.27) (thickness 0.2032)))
   )
   (gr_text "20" (at 125.222 58.42) (layer "Cmts.User")
@@
     (effects (font (size 1.524 1.524) (thickness 0.254)))
   )
+  (gr_text "X" (at 116.84 71.12) (layer "Cmts.User")
+    (effects (font (size 1.27 1.27) (thickness 0.2032)))
+  )
+  (gr_text "X" (at 118.745 35.56) (layer "Cmts.User")
+    (effects (font (size 1.27 1.27) (thickness 0.2032)))
+  )
+  (gr_text "X" (at 114.3 80.01) (layer "Cmts.User")
+    (effects (font (size 1.27 1.27) (thickness 0.2032)))
+  )
   (gr_text "25" (at 80.645 71.005159) (layer "Cmts.User")
     (effects (font (size 1.524 1.524) (thickness 0.2286)))
   )
+  (gr_text "X" (at 102.87 60.325) (layer "Cmts.User")
+    (effects (font (size 1.27 1.27) (thickness 0.2032)))
+  )
+  (gr_text "X" (at 114.3 59.69) (layer "Cmts.User")
+    (effects (font (size 1.27 1.27) (thickness 0.2032)))
+  )
   (gr_text "40" (at 125.222 109.22) (layer "Cmts.User")
     (effects (font (size 1.524 1.524) (thickness 0.2286)))
+  )
+  (gr_text "X" (at 111.76 70.485) (layer "Cmts.User")
+    (effects (font (size 1.27 1.27) (thickness 0.2032)))
+  )
+  (gr_text "X" (at 88.9 73.66) (layer "Cmts.User")
+    (effects (font (size 1.27 1.27) (thickness 0.2032)))
+  )
+  (gr_text "X" (at 88.265 78.74) (layer "Cmts.User")
+    (effects (font (size 1.27 1.27) (thickness 0.2032)))
+  )
+  (gr_text "X" (at 93.98 60.96) (layer "Cmts.User")
+    (effects (font (size 1.27 1.27) (thickness 0.2032)))
+  )
+  (gr_text "X" (at 109.22 83.82) (layer "Cmts.User")
+    (effects (font (size 1.27 1.27) (thickness 0.2032)))
+  )
+  (gr_text "X" (at 102.830169 53.292747) (layer "Cmts.User")
+    (effects (font (size 1.27 1.27) (thickness 0.2032)))
+  )
+  (gr_text "X" (at 118.11 73.66) (layer "Cmts.User")
+    (effects (font (size 1.27 1.27) (thickness 0.2032)))
+  )
+  (gr_text "X" (at 118.07932 43.084638) (layer "Cmts.User")
+    (effects (font (size 1.27 1.27) (thickness 0.2032)))
   )
   (gr_text "40" (at 80.645 109.105159) (layer "Cmts.User")
@@
     (effects (font (size 1.524 1.524) (thickness 0.2286)))
   )
+  (gr_text "X" (at 118.07932 106.601761) (layer "Cmts.User")
+    (effects (font (size 1.27 1.27) (thickness 0.2032)))
+  )
+  (gr_text "X" (at 120.65 43.815) (layer "Cmts.User")
+    (effects (font (size 1.27 1.27) (thickness 0.2032)))
+  )
+  (gr_text "X" (at 111.651992 57.073528) (layer "Cmts.User")
+    (effects (font (size 1.27 1.27) (thickness 0.2032)))
+  )
+  (gr_text "X" (at 87.63 106.68) (layer "Cmts.User")
+    (effects (font (size 1.27 1.27) (thickness 0.2032)))
+  )
   (gr_text "35" (at 80.645 96.405159) (layer "Cmts.User")

Commit message: VCF-SV: proto - update pcb.png
Routing:
- net Net-(R10-Pad1): track 51.4 -> 59.0 mm
Other:
- board text added: "TODO: 4 jumpers"
Changed lines of the file:
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@@
     (effects (font (size 1.524 1.524) (thickness 0.2286)))
   )
-  (gr_text "X" (at 85.09 83.82) (layer "Cmts.User")
+  (gr_text "X" (at 114.935 85.09) (layer "Cmts.User")
+    (effects (font (size 1.27 1.27) (thickness 0.2032)))
+  )
+  (gr_text "X" (at 111.76 95.885) (layer "Cmts.User")
+    (effects (font (size 1.27 1.27) (thickness 0.2032)))
+  )
+  (gr_text "X" (at 85.725 83.82) (layer "Cmts.User")
+    (effects (font (size 1.27 1.27) (thickness 0.2032)))
+  )
+  (gr_text "X" (at 102.87 114.3) (layer "Cmts.User")
+    (effects (font (size 1.27 1.27) (thickness 0.2032)))
+  )
+  (gr_text "X" (at 85.725 113.03) (layer "Cmts.User")
     (effects (font (size 1.27 1.27) (thickness 0.2032)))
   )
@@
     (effects (font (size 1.27 1.27) (thickness 0.2032)))
   )
-  (gr_text "X" (at 86.995 88.9) (layer "Cmts.User")
+  (gr_text "X" (at 87.63 88.9) (layer "Cmts.User")
     (effects (font (size 1.27 1.27) (thickness 0.2032)))
   )
@@
     (effects (font (size 1.27 1.27) (thickness 0.2032)))
   )
+  (gr_text "X" (at 93.323244 101.545591) (layer "Cmts.User")
+    (effects (font (size 1.27 1.27) (thickness 0.2032)))
+  )
+  (gr_text "X" (at 119.953667 90.114608) (layer "Cmts.User")
+    (effects (font (size 1.27 1.27) (thickness 0.2032)))
+  )
   (gr_text "15" (at 80.563391 45.605159) (layer "Cmts.User")
     (effects (font (size 1.524 1.524) (thickness 0.2286)))
@@
     (effects (font (size 1.524 1.524) (thickness 0.2286)))
   )
+  (gr_text "X" (at 101.6 99.06) (layer "Cmts.User")
+    (effects (font (size 1.27 1.27) (thickness 0.2032)))
+  )
   (gr_text "X" (at 120.015 52.705) (layer "Cmts.User")
     (effects (font (size 1.27 1.27) (thickness 0.2032)))
@@
     (effects (font (size 1.27 1.27) (thickness 0.2032)))
   )
+  (gr_text "X" (at 120.015 114.3) (layer "Cmts.User")
+    (effects (font (size 1.27 1.27) (thickness 0.2032)))
+  )
+  (gr_text "X" (at 120.015 82.55) (layer "Cmts.User")
+    (effects (font (size 1.27 1.27) (thickness 0.2032)))
+  )
   (gr_text "30" (at 125.349 83.82) (layer "Cmts.User")
     (effects (font (size 1.524 1.524) (thickness 0.2286)))
@@
     (effects (font (size 1.27 1.27) (thickness 0.2032)))
   )
+  (gr_text "X" (at 88.9 92.71) (layer "Cmts.User")
+    (effects (font (size 1.27 1.27) (thickness 0.2032)))
+  )
   (gr_text "X" (at 111.76 45.72) (layer "Cmts.User")
     (effects (font (size 1.27 1.27) (thickness 0.2032)))
@@
     (effects (font (size 1.27 1.27) (thickness 0.2032)))
   )
+  (gr_text "TODO: 4 jumpers" (at 130.81 106.68) (layer "Cmts.User")
+    (effects (font (size 1 1) (thickness 0.15)))
+  )
   (gr_text "X" (at 102.830169 104.08124) (layer "Cmts.User")
     (effects (font (size 1.27 1.27) (thickness 0.2032)))
@@
   )
   (gr_text "X" (at 87.581019 66.021377) (layer "Cmts.User")
+    (effects (font (size 1.27 1.27) (thickness 0.2032)))
+  )
+  (gr_text "X" (at 106.68 85.725) (layer "Cmts.User")
     (effects (font (size 1.27 1.27) (thickness 0.2032)))
   )
@@
     (effects (font (size 1.27 1.27) (thickness 0.2032)))
   )
+  (gr_text "X" (at 102.235 71.755) (layer "Cmts.User")
+    (effects (font (size 1.27 1.27) (thickness 0.2032)))
+  )
   (gr_text "X" (at 118.745 35.56) (layer "Cmts.User")
     (effects (font (size 1.27 1.27) (thickness 0.2032)))
   )
+  (gr_text "X" (at 91.44 110.49) (layer "Cmts.User")
+    (effects (font (size 1.27 1.27) (thickness 0.2032)))
+  )
   (gr_text "X" (at 114.3 80.01) (layer "Cmts.User")
     (effects (font (size 1.27 1.27) (thickness 0.2032)))
@@
     (effects (font (size 1.524 1.524) (thickness 0.2286)))
   )
+  (gr_text "X" (at 109.22 107.315) (layer "Cmts.User")
+    (effects (font (size 1.27 1.27) (thickness 0.2032)))
+  )
+  (gr_text "X" (at 99.06 93.345) (layer "Cmts.User")
+    (effects (font (size 1.27 1.27) (thickness 0.2032)))
+  )
   (gr_text "X" (at 111.76 70.485) (layer "Cmts.User")
     (effects (font (size 1.27 1.27) (thickness 0.2032)))
@@
     (effects (font (size 1.27 1.27) (thickness 0.2032)))
   )
+  (gr_text "X" (at 84.455 79.375) (layer "Cmts.User")
+    (effects (font (size 1.27 1.27) (thickness 0.2032)))
+  )
   (gr_text "40" (at 80.645 109.105159) (layer "Cmts.User")
     (effects (font (size 1.524 1.524) (thickness 0.2286)))
@@
     (effects (font (size 1.524 1.524) (thickness 0.2286)))
   )
+  (gr_text "X" (at 109.22 97.79) (layer "Cmts.User")
+    (effects (font (size 1.27 1.27) (thickness 0.2032)))
+  )
   (gr_text "X" (at 118.07932 106.601761) (layer "Cmts.User")
     (effects (font (size 1.27 1.27) (thickness 0.2032)))
@@
     (effects (font (size 1.27 1.27) (thickness 0.2032)))
   )
+  (gr_text "X" (at 113.665 113.03) (layer "Cmts.User")
+    (effects (font (size 1.27 1.27) (thickness 0.2032)))
+  )
+  (gr_text "X" (at 102.235 78.74) (layer "Cmts.User")
+    (effects (font (size 1.27 1.27) (thickness 0.2032)))
+  )
   (gr_text "X" (at 111.651992 57.073528) (layer "Cmts.User")
     (effects (font (size 1.27 1.27) (thickness 0.2032)))
@@
   (gr_text "35" (at 80.645 96.405159) (layer "Cmts.User")
     (effects (font (size 1.524 1.524) (thickness 0.2286)))
+  )
+  (gr_text "X" (at 96.463624 112.976574) (layer "Cmts.User")
+    (effects (font (size 1.27 1.27) (thickness 0.2032)))
   )
   (segment (start 99.06 119.38) (end 88.9 119.38) (width 0.4064) (layer "F.Cu") (net 0))
@@
   (via (at 91.44 93.98) (size 0.8) (drill 0.4) (layers "F.Cu" "B.Cu") (net 29))
   (via (at 91.44 63.5) (size 0.8) (drill 0.4) (layers "F.Cu" "B.Cu") (net 29))
-  (segment (start 90.17 90.913949) (end 90.17 66.566051) (width 0.4064) (layer "In1.Cu") (net 29))
-  (arc (start 91.44 93.98) (mid 90.500063 92.573283) (end 90.17 90.913949) (width 0.4064) (layer "In1.Cu") (net 29))
-  (arc (start 90.17 66.566051) (mid 90.500062 64.906717) (end 91.44 63.5) (width 0.4064) (layer "In1.Cu") (net 29))
+  (segment (start 91.44 63.5) (end 91.44 67.681975) (width 0.4064) (layer "In1.Cu") (net 29))
+  (segment (start 84.6232 73.77998) (end 84.6232 87.881994) (width 0.4064) (layer "In1.Cu") (net 29))
+  (segment (start 87.738949 70.485) (end 87.258025 70.485) (width 0.4064) (layer "In1.Cu") (net 29))
+  (segment (start 90.959076 93.98) (end 91.44 93.98) (width 0.4064) (layer "In1.Cu") (net 29))
+  (arc (start 85.725 71.12) (mid 84.909548 72.34041) (end 84.6232 73.77998) (width 0.4064) (layer "In1.Cu") (net 29))
+  (arc (start 87.258025 70.485) (mid 86.428357 70.650031) (end 85.725 71.12) (width 0.4064) (layer "In1.Cu") (net 29))
+  (arc (start 84.6232 87.881994) (mid 85.07458 90.151232) (end 86.36 92.075) (width 0.4064) (layer "In1.Cu") (net 29))
+  (arc (start 91.44 67.681975) (mid 91.274969 68.511642) (end 90.805 69.215) (width 0.4064) (layer "In1.Cu") (net 29))
+  (arc (start 90.805 69.215) (mid 89.398284 70.154937) (end 87.738949 70.485) (width 0.4064) (layer "In1.Cu") (net 29))
+  (arc (start 86.36 92.075) (mid 88.470074 93.484907) (end 90.959076 93.98) (width 0.4064) (layer "In1.Cu") (net 29))
   (segment (start 116.84 60.96) (end 106.68 60.96) (width 0.4064) (layer "F.Cu") (net 30))
   (segment (start 116.84 76.2) (end 106.68 76.2) (width 0.4064) (layer "F.Cu") (net 31))

Commit message: VCF-SV: proto - update pcb.png
Parts:
- moved R3 10.8 mm to (96.5, 91.4), turned to -90 degrees
- moved R8 2.54 mm to (91.4, 99.1)
- moved R9 2.54 mm to (94.0, 96.5)
Routing:
- net -12V: track 165.2 -> 190.5 mm, vias 6 -> 7
- net (no net): track 193.0 -> 182.9 mm
Other:
- board text removed: "TODO: 4 jumpers"
- board text removed: "X"

Commit message: VCF-SV: proto - wip
Routing:
- net OUT: track 60.0 -> 57.5 mm
Changed lines of the file:
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@@
   (gr_circle (center 111.76 91.44) (end 112.895923 91.44) (layer "Dwgs.User") (width 0.2032) (fill none))
   (gr_circle (center 116.721092 111.675049) (end 117.857015 111.675049) (layer "Dwgs.User") (width 0.2032) (fill none))
-  (gr_circle (center 116.84 96.52) (end 117.975923 96.52) (layer "Dwgs.User") (width 0.2032) (fill none))
+  (gr_circle (center 116.84 99.06) (end 117.975923 99.06) (layer "Dwgs.User") (width 0.2032) (fill none))
   (gr_circle (center 111.76 101.6) (end 112.895923 101.6) (layer "Dwgs.User") (width 0.2032) (fill none))
   (gr_line (start 123.19 135.89) (end 82.55 135.89) (layer "Edge.Cuts") (width 0.1))
@@
   (segment (start 109.22 96.52) (end 106.68 96.52) (width 0.4064) (layer "F.Cu") (net 17))
   (via (at 109.22 96.52) (size 0.8) (drill 0.4) (layers "F.Cu" "B.Cu") (net 17))
-  (via (at 116.84 96.52) (size 0.8) (drill 0.4) (layers "F.Cu" "B.Cu") (net 17))
+  (via (at 116.84 99.06) (size 0.8) (drill 0.4) (layers "F.Cu" "B.Cu") (net 17))
   (via (at 109.22 99.06) (size 0.8) (drill 0.4) (layers "F.Cu" "B.Cu") (net 17))
-  (segment (start 115.57 99.586051) (end 115.57 113.048693) (width 0.4064) (layer "In1.Cu") (net 17))
+  (segment (start 115.57 102.126051) (end 115.57 113.048693) (width 0.4064) (layer "In1.Cu") (net 17))
   (arc (start 115.57 113.048693) (mid 113.589626 123.004703) (end 107.95 131.445) (width 0.4064) (layer "In1.Cu") (net 17))
-  (arc (start 116.84 96.52) (mid 115.900062 97.926716) (end 115.57 99.586051) (width 0.4064) (layer "In1.Cu") (net 17))
+  (arc (start 116.84 99.06) (mid 115.900062 100.466716) (end 115.57 102.126051) (width 0.4064) (layer "In1.Cu") (net 17))
   (segment (start 109.22 96.52) (end 109.22 99.06) (width 0.4064) (layer "In4.Cu") (net 17))
   (segment (start 99.06 116.84) (end 88.9 116.84) (width 0.4064) (layer "F.Cu") (net 18))

Commit message: VCF-SV: proto - notch output wip
Parts:
- added R22: 47K, -lmp-stripboard:SB_Gen_7, F.Cu at (116.8, 83.8)
- added R23: 47K, -lmp-stripboard:SB_Gen_4, F.Cu at (111.8, 91.4)
- R12: value 200K -> 300K
- moved C10 2.54 mm to (114.3, 88.9)
- moved C5 2.54 mm to (114.3, 81.3)
Connections:
- U1 pad 12: /LP -> Net-(U1-Pad12)
Routing:
- net /LP: track 30.5 -> 10.2 mm, vias 2 -> 0
- net Net-(U1-Pad12): track 0.00 -> 10.2 mm

Commit message: VCF-SV: proto - notch output wip
Parts:
- R22: footprint -lmp-stripboard:SB_Gen_7 -> -lmp-stripboard:SB_Gen_1
- R23: footprint -lmp-stripboard:SB_Gen_4 -> -lmp-stripboard:SB_Gen_1
- moved R22 38.4 mm to (111.8, 121.9)
- moved C5 38.1 mm to (114.3, 119.4)
- moved C10 38.1 mm to (91.4, 119.4)
- moved R23 35.5 mm to (94.0, 122.1)
Routing:
- net Net-(R22-Pad2): track 10.2 -> 73.1 mm, vias 0 -> 4
- net Net-(C10-Pad1): track 43.8 -> 92.8 mm, vias 2 -> 4
- net Net-(C4-Pad2): track 42.3 -> 91.2 mm, vias 2 -> 4
- net (no net): track 182.9 -> 142.2 mm
- net OUT: track 57.5 -> 58.6 mm
Other:
- board text added: "HP"
- board text added: "LP"
