File: modules/VCF-SV/VCF-SV.kicad_sch (KiCad schematic)
At the start: 45 parts, among them U1 CEM3320, U2 TL074, U3 TL072

Commit message: VCF-SV: wip
Other:
- note added: "TODO: Backwards!"
Changed lines of the file:
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@@
     (effects (font (size 1.27 1.27) (thickness 0.254) bold) (justify left bottom))
+  )
+  (text "TODO: Backwards!" (at 27.94 111.76 0)
+    (effects (font (size 1.27 1.27)) (justify left bottom))
   )
   (text "Front Panel & Power" (at 304.8 21.59 0)

Commit message: VCF-SV: wip
Other:
- note added: "TODO: Updates from prototype"
Changed lines of the file:
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@@
+    (effects (font (size 1.27 1.27)) (justify left bottom))
+  )
+  (text "TODO: Updates from prototype" (at 201.93 90.17 0)
     (effects (font (size 1.27 1.27)) (justify left bottom))
   )

Commit message: VCF-SV: wip
Other:
- note added: "TODO: Reversing attenuator see TLN-428"
- note removed: "TODO: Backwards!"
Changed lines of the file:
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@@
+    (effects (font (size 1.27 1.27)) (justify left bottom))
+  )
+  (text "TODO: Reversing attenuator\nsee TLN-428" (at 17.78 114.3 0)
     (effects (font (size 1.27 1.27)) (justify left bottom))
   )
@@
   (text "Audio Input" (at 22.86 20.32 0)
     (effects (font (size 1.27 1.27) (thickness 0.254) bold) (justify left bottom))
-  )
-  (text "TODO: Backwards!" (at 27.94 111.76 0)
-    (effects (font (size 1.27 1.27)) (justify left bottom))
   )
   (text "Front Panel & Power" (at 304.8 21.59 0)
@@
       (reference "#PWR0121") (unit 1) (value "-12V") (footprint "")
     )
+    (path "/00000000-0000-0000-0000-000060cbfb6a/8d480f83-99a4-40a0-834e-e357fe87211f"
+      (reference "#PWR?") (unit 1) (value "GND") (footprint "")
+    )
+    (path "/00000000-0000-0000-0000-000060cbfb6a/e666764c-3bc8-48ef-8f90-030ff269b3f6"
+      (reference "#PWR?") (unit 1) (value "GND") (footprint "")
+    )
     (path "/00000000-0000-0000-0000-000060cbfb6a/ffa83238-2555-4a28-9cf2-ee04a99c5d51"

Commit message: VCF-SV: wip
Parts:
- R7: value 130K -> 100K; Note (none) -> *changed
Changed lines of the file:
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@@
   (symbol (lib_id "-lmp:R_1%_0W166") (at 41.91 176.53 90) (unit 1)
     (in_bom yes) (on_board yes) (fields_autoplaced)
-    (property "Reference" "R7" (id 0) (at 41.91 171.8142 90))
-    (property "Value" "130K" (id 1) (at 41.91 174.3511 90))
+    (property "Reference" "R7" (id 0) (at 41.91 169.2774 90))
+    (property "Value" "100K" (id 1) (at 41.91 171.8143 90))
     (property "Footprint" "-lmp-misc:R_Axial_DIN0207_L6.3mm_D2.5mm_P7.62mm_Horizontal" (id 2) (at 41.91 178.308 90)
       (effects (font (size 1.27 1.27)) hide)
@@
       (effects (font (size 1.27 1.27)) hide)
     )
+    (property "Note" "*changed" (id 10) (at 41.91 174.3512 90))
     (pin "1")
     (pin "2")
@@
     )
     (path "/ccd11566-81bf-43ae-8e46-e65fe09df230"
-      (reference "R7") (unit 1) (value "130K") (footprint "-lmp-misc:R_Axial_DIN0207_L6.3mm_D2.5mm_P7.62mm_Horizontal")
+      (reference "R7") (unit 1) (value "100K") (footprint "-lmp-misc:R_Axial_DIN0207_L6.3mm_D2.5mm_P7.62mm_Horizontal")
     )
     (path "/5f67bdba-b7b8-4799-92c8-494682322525"

Commit message: VCF-SV: update from prototype - wip
Parts:
- removed C11: 4U7, -lmp-misc:CP_Radial_D4.0mm_P2.50mm, symbol -lmp:CP
- added R29, R31, R32: 100K, -lmp-misc:R_Axial_DIN0207_L6.3mm_D2.5mm_P7.62mm_Horizontal, symbol -lmp:R_1%_0W166
- added R30: 1M, -lmp-misc:R_Axial_DIN0207_L6.3mm_D2.5mm_P7.62mm_Horizontal, symbol -lmp:R_1%_0W166
- R1: value 100K -> 200K
- R12: value 49K9 -> 39K
- R14: value 200K -> 300K
- R2: value 240K -> 130K
- R25: value 100K -> 68K
- R3: value 200K -> 100K
- R7: value 100K -> 130K; Note *changed -> (none)
Connections:
- net GND: now also R30.2, R31.1
- net OUT-AUDIO-LP-HP: now also R32.2; no longer U3.2 (-)
- net OUT-HP: now also C8.2, R20.2, R22.1, U1.7 (OUT)
- net OUT-LP: now also C12.2, R23.2, U1.15 (OUT); no longer C16.2
- net OUT-LP-HP: now also C16.1; no longer U3.3 (+)
- net OUT-BP: now reaches C14.2, R16.2, R17.1, R25.1
- net at R11.2, R15.1, U2.2 (-): now also R29.2
- net CV-RES-MOD renamed CV-RES-MOD-P
- new net: C16.2, R30.1, U3.3 (+)
- new net: R31.2, R32.1, U3.2 (-)
- new net CV-RES-MOD-N: R29.1
Other:
- note added: "Can be trimmed so the 1V/octave CV input tracks pitch. If that doesn't matter, the trimmers and the thermistor may be replaced by fixed resistors."
- note added: "Increasing current into Q-CTRL increases feedback but reduces resonance."
- note added: "Output level varies with resonance and waveform. The gain settings here are a compromise."
- note added: "Reversing attenuator for resonance CV"
- note added: "State-Variable Filter"
- note added: "Turning the resonance pot fully CW should provoke oscillation. The resonance CV goes through a reversing attenuator pot."
- note added: "from Lo/Hi/Notch control"
- note added: "to Lo/Hi/Notch control"
- note removed: "Can be trimmed so the CV inputs track 1V/octave. If that doesn't matter, the trimmers and thermistor may be replaced by fixed resistors."
- note removed: "Filter"
- note removed: "TODO: Reversing attenuator see TLN-428"
- note removed: "TODO: Updates from prototype"
- note removed: "TODO: capacitor needed?"
- note removed: "TODO: check output levels"
- note removed: "TODO: good value for R12"
- note removed: "This should allow each CV input to provoke self-resonance near its maximum value."
- note removed: "from hi/lo/notch pot"
- note removed: "to hi/lo/notch pot"
- moved on the sheet: C13, C14, C15, C16, R15, R18, R19, R24, R25, R26, U1B, U1C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

Commit message: VCF-SV: update from prototype - wip
Parts:
- renumbered C12 to C11, C13 to C12, C14 to C13, C15 to C14, C16 to C15
Changed lines of the file:
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@@
   (symbol (lib_id "-lmp:CC") (at 144.78 25.4 90) (unit 1)
     (in_bom yes) (on_board yes) (fields_autoplaced)
-    (property "Reference" "C12" (id 0) (at 144.78 19.5412 90))
+    (property "Reference" "C11" (id 0) (at 144.78 19.5412 90))
     (property "Value" "18P" (id 1) (at 144.78 22.0781 90))
     (property "Footprint" "-lmp-misc:C_Disc_D5.0mm_W2.5mm_P2.50mm" (id 2) (at 148.59 24.4348 0)
@@
   (symbol (lib_id "-lmp:CP") (at 190.5 121.92 90) (unit 1)
     (in_bom yes) (on_board yes) (fields_autoplaced)
-    (property "Reference" "C16" (id 0) (at 189.611 116.0612 90))
+    (property "Reference" "C15" (id 0) (at 189.611 116.0612 90))
     (property "Value" "4U7" (id 1) (at 189.611 118.5981 90))
     (property "Footprint" "-lmp-misc:CP_Radial_D4.0mm_P2.50mm" (id 2) (at 194.31 120.9548 0)
@@
   (symbol (lib_id "-lmp:CF") (at 177.8 72.39 0) (unit 1)
     (in_bom yes) (on_board yes) (fields_autoplaced)
-    (property "Reference" "C15" (id 0) (at 180.721 71.5553 0)
+    (property "Reference" "C14" (id 0) (at 180.721 71.5553 0)
       (effects (font (size 1.27 1.27)) (justify left))
     )
@@
   (symbol (lib_id "-lmp:CP") (at 154.94 72.39 0) (unit 1)
     (in_bom yes) (on_board yes) (fields_autoplaced)
-    (property "Reference" "C14" (id 0) (at 157.861 70.6663 0)
+    (property "Reference" "C13" (id 0) (at 157.861 70.6663 0)
       (effects (font (size 1.27 1.27)) (justify left))
     )
@@
   (symbol (lib_id "-lmp:CF") (at 143.51 72.39 0) (unit 1)
     (in_bom yes) (on_board yes) (fields_autoplaced)
-    (property "Reference" "C13" (id 0) (at 146.431 71.5553 0)
+    (property "Reference" "C12" (id 0) (at 146.431 71.5553 0)
       (effects (font (size 1.27 1.27)) (justify left))
     )
@@
     )
     (path "/34925a35-1201-4393-9c57-abfe3bf7689b"
-      (reference "C12") (unit 1) (value "18P") (footprint "-lmp-misc:C_Disc_D5.0mm_W2.5mm_P2.50mm")
+      (reference "C11") (unit 1) (value "18P") (footprint "-lmp-misc:C_Disc_D5.0mm_W2.5mm_P2.50mm")
     )
     (path "/e267fbbb-901e-43f7-8488-02dbd0205b9a"
-      (reference "C13") (unit 1) (value "150P") (footprint "-lmp-misc:C_Rect_L7.2mm_W4.5mm_P5.00mm")
+      (reference "C12") (unit 1) (value "150P") (footprint "-lmp-misc:C_Rect_L7.2mm_W4.5mm_P5.00mm")
     )
     (path "/72f75d2b-9003-46ce-b4fe-7477bd81008a"
-      (reference "C14") (unit 1) (value "4U7") (footprint "-lmp-misc:CP_Radial_D4.0mm_P2.50mm")
+      (reference "C13") (unit 1) (value "4U7") (footprint "-lmp-misc:CP_Radial_D4.0mm_P2.50mm")
     )
     (path "/4e55baad-05f2-4f94-b453-b701868bb807"
-      (reference "C15") (unit 1) (value "150P") (footprint "-lmp-misc:C_Rect_L7.2mm_W4.5mm_P5.00mm")
+      (reference "C14") (unit 1) (value "150P") (footprint "-lmp-misc:C_Rect_L7.2mm_W4.5mm_P5.00mm")
     )
     (path "/41190185-6086-4a2b-8c08-63056244349f"
-      (reference "C16") (unit 1) (value "4U7") (footprint "-lmp-misc:CP_Radial_D4.0mm_P2.50mm")
+      (reference "C15") (unit 1) (value "4U7") (footprint "-lmp-misc:CP_Radial_D4.0mm_P2.50mm")
     )
     (path "/00000000-0000-0000-0000-000060cbfb6a/00000000-0000-0000-0000-000061a7a513"
@@
     )
     (path "/00000000-0000-0000-0000-000060cbfb6a/00000000-0000-0000-0000-000060c179d1"
-      (reference "J11") (unit 1) (value "Conn_Back_Right_Top") (footprint "Connector_PinHeader_2.54mm:PinHeader_1x14_P2.54mm_Vertical")
+      (reference "J11") (unit 1) (value "Conn_Back_Right_Top") (footprint "Connector_PinHeader_2.54mm:PinHeader_1x15_P2.54mm_Vertical")
     )
     (path "/00000000-0000-0000-0000-000060cbfb6a/00000000-0000-0000-0000-000061b13bc3"

Commit message: VCF-SV: BOM
Parts:
- C11: Distributor (none) -> Mouser; DistributorPartLink (none) -> https://www.mouser.ca/ProductDetail/?qs=s%2FCsB4POEK6rPX34e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; DistributorPartNum (none) -> 594-K180J15C0GF5TL2; Manufacturer (none) -> Murata; ManufacturerPartNum (none) -> K180J15C0GF5TL2
- C12, C14: Distributor (none) -> Mouser; DistributorPartLink (none) -> https://www.mouser.ca/ProductDetail/KEMET/PFR5151J63J11L4BU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; DistributorPartNum (none) -> 80-PFR5151J63J11L4; Manufacturer (none) -> KEMET; ManufacturerPartNum (none) -> PFR5151J63J11L4BULK
- C13, C15, C7: Distributor (none) -> Mouser; DistributorPartLink (none) -> https://www.mouser.ca/ProductDetail/Panasonic/ECE-A1HKA4R7I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; DistributorPartNum (none) -> 667-ECE-A1HKA4R7I; Manufacturer (none) -> Panasonic; ManufacturerPartNum (none) -> ECE-A1HKA4R7I
- C8: Distributor (none) -> Mouser; DistributorPartLink (none) -> https://www.mouser.ca/ProductDetail/TDK/FG18C0G1H100DNT00?q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; DistributorPartNum (none) -> 810-FG18C0G1H100DNT0; Manufacturer (none) -> TDK; ManufacturerPartNum (none) -> FG18C0G1H100DNT00
- R1: DistributorPartLink https://www.mouser.ca/c/?m=YAGEO&power+rating=166+mW+(1%2f6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 -> https://www.mouser.ca/ProductDetail/YAGEO/MFR-12FTF52-200K?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; DistributorPartNum 603-MFR-12* -> 603-MFR-12FTF52-200K; ManufacturerPartNum MFR-12* -> MFR-12FTF52-200K
- R10: renamed from R9; DistributorPartLink https://www.mouser.ca/c/?m=YAGEO&power+rating=166+mW+(1%2f6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 -> https://www.mouser.ca/ProductDetail/YAGEO/MFR-12FTF52-100K?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; DistributorPartNum 603-MFR-12* -> 603-MFR-12FTF52-100K; ManufacturerPartNum MFR-12* -> MFR-12FTF52-100K
- R11: renamed from R10; DistributorPartLink https://www.mouser.ca/c/?m=YAGEO&power+rating=166+mW+(1%2f6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 -> https://www.mouser.ca/ProductDetail/YAGEO/MFR-12FTF52-100K?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; DistributorPartNum 603-MFR-12* -> 603-MFR-12FTF52-100K; ManufacturerPartNum MFR-12* -> MFR-12FTF52-100K
- R12: renamed from R11; DistributorPartLink https://www.mouser.ca/c/?m=YAGEO&power+rating=166+mW+(1%2f6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 -> https://www.mouser.ca/ProductDetail/YAGEO/MFR-12FTF52-100K?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; DistributorPartNum 603-MFR-12* -> 603-MFR-12FTF52-100K; ManufacturerPartNum MFR-12* -> MFR-12FTF52-100K
- R13: renamed from R12; DistributorPartLink https://www.mouser.ca/c/?m=YAGEO&power+rating=166+mW+(1%2f6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 -> https://www.mouser.ca/ProductDetail/YAGEO/MFR-12FTF52-39K?q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; DistributorPartNum 603-MFR-12* -> 603-MFR-12FTF52-39K; ManufacturerPartNum MFR-12* -> MFR-12FTF52-39K
- R14: renamed from R13; DistributorPartLink https://www.mouser.ca/c/?m=YAGEO&power+rating=166+mW+(1%2f6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 -> https://www.mouser.ca/ProductDetail/YAGEO/MFR-12FTF52-91K?q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; DistributorPartNum 603-MFR-12* -> 603-MFR-12FTF52-91K; ManufacturerPartNum MFR-12* -> MFR-12FTF52-91K
- R15: renamed from R14; DistributorPartLink https://www.mouser.ca/c/?m=YAGEO&power+rating=166+mW+(1%2f6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 -> https://www.mouser.ca/ProductDetail/YAGEO/MFR-25FRF52-300K?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; DistributorPartNum 603-MFR-12* -> 603-MFR-25FRF52-300K; ManufacturerPartNum MFR-12* -> MFR-25FRF52-300K
- R16: renamed from R15; DistributorPartLink https://www.mouser.ca/c/?m=YAGEO&power+rating=166+mW+(1%2f6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 -> https://www.mouser.ca/ProductDetail/YAGEO/MFR-12FTF52-100K?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; DistributorPartNum 603-MFR-12* -> 603-MFR-12FTF52-100K; ManufacturerPartNum MFR-12* -> MFR-12FTF52-100K
- R17: renamed from R16; DistributorPartLink https://www.mouser.ca/c/?m=YAGEO&power+rating=166+mW+(1%2f6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 -> https://www.mouser.ca/ProductDetail/YAGEO/MFR-12FTF52-240K?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; DistributorPartNum 603-MFR-12* -> 603-MFR-12FTF52-240K; ManufacturerPartNum MFR-12* -> MFR-12FTF52-240K
- R18: renamed from R17; DistributorPartLink https://www.mouser.ca/c/?m=YAGEO&power+rating=166+mW+(1%2f6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 -> https://www.mouser.ca/ProductDetail/YAGEO/MFR-12FTF52-220K?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; DistributorPartNum 603-MFR-12* -> 603-MFR-12FTF52-220K; ManufacturerPartNum MFR-12* -> MFR-12FTF52-220K
- R19: renamed from R18; DistributorPartLink https://www.mouser.ca/c/?m=YAGEO&power+rating=166+mW+(1%2f6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 -> https://www.mouser.ca/ProductDetail/YAGEO/MFR-12FTF52-100K?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; DistributorPartNum 603-MFR-12* -> 603-MFR-12FTF52-100K; ManufacturerPartNum MFR-12* -> MFR-12FTF52-100K
- R2: DistributorPartLink https://www.mouser.ca/c/?m=YAGEO&power+rating=166+mW+(1%2f6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 -> https://www.mouser.ca/ProductDetail/YAGEO/MFR-12FTF52-130K?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; DistributorPartNum 603-MFR-12* -> 603-MFR-12FTF52-130K; ManufacturerPartNum MFR-12* -> MFR-12FTF52-130K
- R20, R3: DistributorPartLink https://www.mouser.ca/c/?m=YAGEO&power+rating=166+mW+(1%2f6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 -> https://www.mouser.ca/ProductDetail/YAGEO/MFR-12FTF52-100K?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; DistributorPartNum 603-MFR-12* -> 603-MFR-12FTF52-100K; ManufacturerPartNum MFR-12* -> MFR-12FTF52-100K
- R21: renamed from R19; DistributorPartLink https://www.mouser.ca/c/?m=YAGEO&power+rating=166+mW+(1%2f6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 -> https://www.mouser.ca/ProductDetail/YAGEO/MFR-25FTE52-2M61?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; DistributorPartNum 603-MFR-12* -> 603-MFR-25FTE52-2M61; ManufacturerPartNum MFR-12* -> MFR-25FTE52-2M61
- R22: renamed from R21; DistributorPartLink https://www.mouser.ca/c/?m=YAGEO&power+rating=166+mW+(1%2f6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 -> https://www.mouser.ca/ProductDetail/YAGEO/MFR-12FTF52-680R?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; DistributorPartNum 603-MFR-12* -> 603-MFR-12FTF52-680R; ManufacturerPartNum MFR-12* -> MFR-12FTF52-680R
- R23: renamed from R22; DistributorPartLink https://www.mouser.ca/c/?m=YAGEO&power+rating=166+mW+(1%2f6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 -> https://www.mouser.ca/ProductDetail/YAGEO/MFR-12FTF52-100K?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; DistributorPartNum 603-MFR-12* -> 603-MFR-12FTF52-100K; ManufacturerPartNum MFR-12* -> MFR-12FTF52-100K
- R24: renamed from R23; DistributorPartLink https://www.mouser.ca/c/?m=YAGEO&power+rating=166+mW+(1%2f6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 -> https://www.mouser.ca/ProductDetail/YAGEO/MFR-12FTF52-91K?q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; DistributorPartNum 603-MFR-12* -> 603-MFR-12FTF52-91K; ManufacturerPartNum MFR-12* -> MFR-12FTF52-91K
- R25: renamed from R24; DistributorPartLink https://www.mouser.ca/c/?m=YAGEO&power+rating=166+mW+(1%2f6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 -> https://www.mouser.ca/ProductDetail/YAGEO/MFR-12FTF52-100K?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; DistributorPartNum 603-MFR-12* -> 603-MFR-12FTF52-100K; ManufacturerPartNum MFR-12* -> MFR-12FTF52-100K
- R26: renamed from R30; DistributorPartLink https://www.mouser.ca/c/?m=YAGEO&power+rating=166+mW+(1%2f6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 -> https://www.mouser.ca/ProductDetail/YAGEO/MFR-12FTE52-1M?qs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; DistributorPartNum 603-MFR-12* -> 603-MFR-12FTE52-1M; ManufacturerPartNum MFR-12* -> MFR-12FTE52-1M
- R27: renamed from R25; DistributorPartLink https://www.mouser.ca/c/?m=YAGEO&power+rating=166+mW+(1%2f6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 -> https://www.mouser.ca/ProductDetail/YAGEO/MFR-12FTF52-68K?q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; DistributorPartNum 603-MFR-12* -> 603-MFR-12FTF52-68K; ManufacturerPartNum MFR-12* -> MFR-12FTF52-68K
- R28: renamed from R31; DistributorPartLink https://www.mouser.ca/c/?m=YAGEO&power+rating=166+mW+(1%2f6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 -> https://www.mouser.ca/ProductDetail/YAGEO/MFR-12FTF52-100K?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; DistributorPartNum 603-MFR-12* -> 603-MFR-12FTF52-100K; ManufacturerPartNum MFR-12* -> MFR-12FTF52-100K
- R29: renamed from R26; DistributorPartLink https://www.mouser.ca/c/?m=YAGEO&power+rating=166+mW+(1%2f6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 -> https://www.mouser.ca/ProductDetail/YAGEO/MFR-12FTF52-100K?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; DistributorPartNum 603-MFR-12* -> 603-MFR-12FTF52-100K; ManufacturerPartNum MFR-12* -> MFR-12FTF52-100K
- R30: renamed from R32; DistributorPartLink https://www.mouser.ca/c/?m=YAGEO&power+rating=166+mW+(1%2f6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 -> https://www.mouser.ca/ProductDetail/YAGEO/MFR-12FTF52-100K?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; DistributorPartNum 603-MFR-12* -> 603-MFR-12FTF52-100K; ManufacturerPartNum MFR-12* -> MFR-12FTF52-100K
- R4: renamed from R29; DistributorPartLink https://www.mouser.ca/c/?m=YAGEO&power+rating=166+mW+(1%2f6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 -> https://www.mouser.ca/ProductDetail/YAGEO/MFR-12FTF52-100K?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; DistributorPartNum 603-MFR-12* -> 603-MFR-12FTF52-100K; ManufacturerPartNum MFR-12* -> MFR-12FTF52-100K
- R5: renamed from R4; DistributorPartLink https://www.mouser.ca/c/?m=YAGEO&power+rating=166+mW+(1%2f6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 -> https://www.mouser.ca/ProductDetail/YAGEO/MFR-12FTF52-120K?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; DistributorPartNum 603-MFR-12* -> 603-MFR-12FTF52-120K; ManufacturerPartNum MFR-12* -> MFR-12FTF52-120K
- R6: renamed from R5; DistributorPartLink https://www.mouser.ca/c/?m=YAGEO&power+rating=166+mW+(1%2f6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 -> https://www.mouser.ca/ProductDetail/YAGEO/MFR-12FTF52-100K?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; DistributorPartNum 603-MFR-12* -> 603-MFR-12FTF52-100K; ManufacturerPartNum MFR-12* -> MFR-12FTF52-100K
- R7: renamed from R6; DistributorPartLink https://www.mouser.ca/c/?m=YAGEO&power+rating=166+mW+(1%2f6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 -> https://www.mouser.ca/ProductDetail/YAGEO/MFR-12FTF52-100K?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; DistributorPartNum 603-MFR-12* -> 603-MFR-12FTF52-100K; ManufacturerPartNum MFR-12* -> MFR-12FTF52-100K
- R8: renamed from R7; DistributorPartLink https://www.mouser.ca/c/?m=YAGEO&power+rating=166+mW+(1%2f6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 -> https://www.mouser.ca/ProductDetail/YAGEO/MFR-12FTF52-130K?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; DistributorPartNum 603-MFR-12* -> 603-MFR-12FTF52-130K; ManufacturerPartNum MFR-12* -> MFR-12FTF52-130K
- R9: renamed from R8; DistributorPartLink https://www.mouser.ca/c/?m=YAGEO&power+rating=166+mW+(1%2f6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 -> https://www.mouser.ca/ProductDetail/YAGEO/MFR-12FTF52-100K?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; DistributorPartNum 603-MFR-12* -> 603-MFR-12FTF52-100K; ManufacturerPartNum MFR-12* -> MFR-12FTF52-100K
- RT1: Distributor (none) -> Thonk; DistributorPartLink (none) -> https://www.thonk.co.uk/shop/tempco-resistor-akaneohm/; DistributorPartNum (none) -> LT16S102F33; Manufacturer (none) -> Akaneohm; ManufacturerPartNum (none) -> LT16S102F33; Note (none) -> Tempco resistor
- RV6: DistributorPartLink https://www.mouser.ca/c/passive-components/potentiometers-t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 -> https://www.mouser.ca/ProductDetail/Bourns/3296W-1-253LF?qs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; DistributorPartNum 652-3296W-* -> 652-3296W-1-253LF; ManufacturerPartNum 3296W-* -> 3296W-1-253LF
- RV7: DistributorPartLink https://www.mouser.ca/c/passive-components/potentiometers-t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 -> https://www.mouser.ca/ProductDetail/Bourns/3296W-1-103LF?qs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; DistributorPartNum 652-3296W-* -> 652-3296W-1-103LF; ManufacturerPartNum 3296W-* -> 3296W-1-103LF
- RV8: DistributorPartLink https://www.mouser.ca/c/passive-components/potentiometers-t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 -> https://www.mouser.ca/ProductDetail/Bourns/3296W-1-202LF?qs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; DistributorPartNum 652-3296W-* -> 652-3296W-1-202LF; ManufacturerPartNum 3296W-* -> 3296W-1-202LF
