File: modules/Switches/prototype/prototype.kicad_sch (KiCad schematic)
At the start: 8 parts, among them J1 Conn_01x09, SW1 SW_Push, U1 TL072

Commit message: Switches module - prototype wip
Parts:
- R3: value R_1K_Output -> 1K
Changed lines of the file:
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@@
       (effects (font (size 1.27 1.27)))
     )
-    (property "Value" "R_1K_Output" (at 120.65 59.6097 90)
+    (property "Value" "1K" (at 120.65 59.6097 90)
       (effects (font (size 1.27 1.27)))
     )
