File: modules/Switches/prototype/fake-vactrol/prototype.kicad_sch (KiCad schematic)
At the start: 8 parts, among them J1 Conn_01x09, SW1 SW_Push, U1 TL072

Commit message: Switches module - add JFET prototype
Other:
- title: Eurorack ProtoModule -> Vactrol Switch Prototype
Changed lines of the file:
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@@
   (paper "A4")
   (title_block
-    (title "Eurorack ProtoModule")
+    (title "Vactrol Switch Prototype")
     (date "2021-10-06")
     (rev "1.0")
