File: modules/Switches/prototype/jfet/prototype.kicad_pcb (KiCad board)
At the start: 6 copper layers, 40.6 x 78.7 mm, 12 parts, among them J1 Conn_01x09, Q1 J109/112, Q2 J109/112, SW1 SW_Push, U1 TL072

Commit message: Switches module - prototype wip
Parts:
- R1: footprint -lmp-misc:R_Axial_DIN0207_L6.3mm_D2.5mm_P7.62mm_Horizontal -> -lmp-stripboard:SB_Gen_1
- R4: footprint -lmp-misc:R_Axial_DIN0207_L6.3mm_D2.5mm_P7.62mm_Horizontal -> -lmp-stripboard:SB_Gen_2
- moved C1 53.9 mm to (88.9, 35.6), turned to 180 degrees
- moved Q2 51.1 mm to (94.0, 81.3), turned to 90 degrees
- moved R5 40.9 mm to (99.1, 30.5)
- moved R4 39.8 mm to (96.5, 30.5), turned to -90 degrees
- moved Q1 39.5 mm to (109.2, 81.3), turned to 90 degrees
- moved R2 38.1 mm to (114.3, 88.9), turned to 90 degrees
- moved R6 25.7 mm to (106.7, 81.3), turned to 180 degrees
- moved R1 19.1 mm to (119.4, 86.4), turned to 180 degrees
Routing:
- net (no net): track 447.0 -> 365.8 mm
- net Net-(Q1-G): track 0.00 -> 79.4 mm, vias 0 -> 4
- net GND: track 175.4 -> 213.5 mm, vias 2 -> 8
- net Net-(Q2-D): track 10.2 -> 23.9 mm, vias 0 -> 1
- net Net-(Q1-D): track 0.00 -> 10.2 mm

Commit message: Switches module - prototype wip
Parts:
- R3: footprint -lmp-stripboard:SB_Gen_3 -> -lmp-stripboard:SB_Gen_2
- moved R3 5.78 mm to (94.0, 89.1)
Connections:
- R3 pad 1: Net-(U1B--) -> Net-(R3-Pad1)
- U1 pad 6: Net-(U1B--) -> IN-OUT-2
- U1 pad 7: Net-(U1B--) -> Net-(R3-Pad1)
Routing:
- net Net-(U1B--): track 22.9 -> 0.00 mm, vias 2 -> 0
- net IN-OUT-2: track 20.4 -> 38.2 mm, vias 1 -> 3
- net Net-(R3-Pad1): track 0.00 -> 10.2 mm
Changed lines of the file:
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@@
   (net 7 "IN-OUT-2")
   (net 8 "Net-(U1A--)")
-  (net 9 "Net-(U1B--)")
+  (net 9 "Net-(R3-Pad1)")
   (net 10 "unconnected-(SW1-Pad1)")
   (net 11 "unconnected-(SW1-Pad3)")
@@
     )
   )
-  (footprint "-lmp-stripboard:SB_Gen_3" (layer "F.Cu")
-    (at 88.9 86.36 -90)
-    (descr "Stripboard, span 3 rows")
+  (footprint "-lmp-stripboard:SB_Gen_2" (layer "F.Cu")
+    (at 93.98 89.125 -90)
+    (descr "Stripboard, span 2 rows")
     (tags "Stripboard")
     (property "Distributor" "Mouser")
@@
     (property "ki_keywords" "R res resistor")
     (attr through_hole)
-    (fp_text reference "R3" (at 3.81 -2.37 -90) (layer "F.SilkS")
-        (effects (font (size 1 1) (thickness 0.15)))
-    )
-    (fp_text value "1K" (at 3.81 2.37 -90) (layer "F.Fab")
-        (effects (font (size 1 1) (thickness 0.15)))
-    )
-    (fp_text user "${REFERENCE}" (at 3.81 0 -90) (layer "F.Fab")
-        (effects (font (size 1 1) (thickness 0.15)))
-    )
-    (fp_line (start 0.54 -1.37) (end 7.08 -1.37)
-      (stroke (width 0.12) (type solid)) (layer "F.SilkS"))
-    (fp_line (start 0.54 -1.04) (end 0.54 -1.37)
-      (stroke (width 0.12) (type solid)) (layer "F.SilkS"))
-    (fp_line (start 0.54 1.04) (end 0.54 1.37)
-      (stroke (width 0.12) (type solid)) (layer "F.SilkS"))
-    (fp_line (start 0.54 1.37) (end 7.08 1.37)
-      (stroke (width 0.12) (type solid)) (layer "F.SilkS"))
-    (fp_line (start 7.08 -1.37) (end 7.08 -1.04)
-      (stroke (width 0.12) (type solid)) (layer "F.SilkS"))
-    (fp_line (start 7.08 1.37) (end 7.08 1.04)
-      (stroke (width 0.12) (type solid)) (layer "F.SilkS"))
-    (fp_line (start -1.05 -1.5) (end -1.05 1.5)
-      (stroke (width 0.05) (type solid)) (layer "F.CrtYd"))
-    (fp_line (start -1.05 1.5) (end 8.67 1.5)
-      (stroke (width 0.05) (type solid)) (layer "F.CrtYd"))
-    (fp_line (start 8.67 -1.5) (end -1.05 -1.5)
-      (stroke (width 0.05) (type solid)) (layer "F.CrtYd"))
-    (fp_line (start 8.67 1.5) (end 8.67 -1.5)
-      (stroke (width 0.05) (type solid)) (layer "F.CrtYd"))
-    (fp_line (start 0 0) (end 0.66 0)
-      (stroke (width 0.1) (type solid)) (layer "F.Fab"))
-    (fp_line (start 0.66 -1.25) (end 0.66 1.25)
-      (stroke (width 0.1) (type solid)) (layer "F.Fab"))
-    (fp_line (start 0.66 1.25) (end 6.96 1.25)
-      (stroke (width 0.1) (type solid)) (layer "F.Fab"))
-    (fp_line (start 6.96 -1.25) (end 0.66 -1.25)
-      (stroke (width 0.1) (type solid)) (layer "F.Fab"))
-    (fp_line (start 6.96 1.25) (end 6.96 -1.25)
-      (stroke (width 0.1) (type solid)) (layer "F.Fab"))
-    (fp_line (start 7.62 0) (end 6.96 0)
-      (stroke (width 0.1) (type solid)) (layer "F.Fab"))
+    (fp_text reference "R3" (at 2.54 -2.37 -90) (layer "F.SilkS")
+        (effects (font (size 1 1) (thickness 0.15)))
+    )
+    (fp_text value "1K" (at 2.54 2.37 -90) (layer "F.Fab")
+        (effects (font (size 1 1) (thickness 0.15)))
+    )
+    (fp_text user "${REFERENCE}" (at 2.54 -2.37 -90) (layer "F.Fab")
+        (effects (font (size 1 1) (thickness 0.15)))
+    )
+    (fp_line (start 1.37 0) (end 3.98 0)
+      (stroke (width 0.12) (type solid)) (layer "F.SilkS"))
+    (fp_circle (center 0 0) (end 1.37 0)
+      (stroke (width 0.12) (type solid)) (fill none) (layer "F.SilkS"))
+    (fp_line (start -1.5 -1.5) (end -1.5 1.5)
+      (stroke (width 0.05) (type solid)) (layer "F.CrtYd"))
+    (fp_line (start -1.5 1.5) (end 6.13 1.5)
+      (stroke (width 0.05) (type solid)) (layer "F.CrtYd"))
+    (fp_line (start 6.13 -1.5) (end -1.5 -1.5)
+      (stroke (width 0.05) (type solid)) (layer "F.CrtYd"))
+    (fp_line (start 6.13 1.5) (end 6.13 -1.5)
+      (stroke (width 0.05) (type solid)) (layer "F.CrtYd"))
+    (fp_line (start 0 0) (end 5.08 0)
+      (stroke (width 0.1) (type solid)) (layer "F.Fab"))
+    (fp_circle (center 0 0) (end 1.25 0)
+      (stroke (width 0.1) (type solid)) (fill none) (layer "F.Fab"))
     (pad "1" thru_hole circle (at 0 0 270) (size 1.6 1.6) (drill 0.8) (layers "*.Cu" "*.Mask")
-      (net 9 "Net-(U1B--)") (pintype "passive"))
-    (pad "2" thru_hole oval (at 7.62 0 270) (size 1.6 1.6) (drill 0.8) (layers "*.Cu" "*.Mask")
+      (net 9 "Net-(R3-Pad1)") (pintype "passive"))
+    (pad "2" thru_hole oval (at 5.08 0 270) (size 1.6 1.6) (drill 0.8) (layers "*.Cu" "*.Mask")
       (net 7 "IN-OUT-2") (pintype "passive"))
-    (model "${KISYS3DMOD}/Resistor_THT.3dshapes/R_Axial_DIN0207_L6.3mm_D2.5mm_P7.62mm_Horizontal.wrl"
+    (model "${KISYS3DMOD}/Resistor_THT.3dshapes/R_Axial_DIN0207_L6.3mm_D2.5mm_P5.08mm_Vertical.wrl"
       (offset (xyz 0 0 0))
       (scale (xyz 1 1 1))
@@
       (net 18 "Net-(Q2-D)") (pinfunction "+") (pintype "input"))
     (pad "6" thru_hole oval (at 7.62 5.08 180) (size 1.6 1.6) (drill 0.8) (layers "*.Cu" "*.Mask")
-      (net 9 "Net-(U1B--)") (pinfunction "-") (pintype "input"))
+      (net 7 "IN-OUT-2") (pinfunction "-") (pintype "input"))
     (pad "7" thru_hole oval (at 7.62 2.54 180) (size 1.6 1.6) (drill 0.8) (layers "*.Cu" "*.Mask")
-      (net 9 "Net-(U1B--)") (pintype "output"))
+      (net 9 "Net-(R3-Pad1)") (pintype "output"))
     (pad "8" thru_hole oval (at 7.62 0 180) (size 1.6 1.6) (drill 0.8) (layers "*.Cu" "*.Mask")
       (net 1 "+12V") (pinfunction "V+") (pintype "power_in"))
@@
     (property "ki_keywords" "R res resistor")
     (attr through_hole)
-    (fp_text reference "R1" (at 1.27 -2.37) (layer "F.SilkS")
-        (effects (font (size 1 1) (thickness 0.15)))
-    )
-    (fp_text value "100k" (at 1.27 2.37) (layer "F.Fab")
-        (effects (font (size 1 1) (thickness 0.15)))
-    )
-    (fp_text user "${REFERENCE}" (at 1.27 -2.37) (layer "F.Fab")
+    (fp_text reference "R1" (at 1.27 -2.37 180) (layer "F.SilkS")
+        (effects (font (size 1 1) (thickness 0.15)))
+    )
+    (fp_text value "100k" (at 1.27 2.37 180) (layer "F.Fab")
+        (effects (font (size 1 1) (thickness 0.15)))
+    )
+    (fp_text user "${REFERENCE}" (at 1.27 -2.37 180) (layer "F.Fab")
         (effects (font (size 1 1) (thickness 0.15)))
     )
@@
     (property "ki_keywords" "R res resistor")
     (attr through_hole)
-    (fp_text reference "R4" (at 2.54 -2.37 90) (layer "F.SilkS")
-        (effects (font (size 1 1) (thickness 0.15)))
-    )
-    (fp_text value "100k" (at 2.54 2.37 90) (layer "F.Fab")
-        (effects (font (size 1 1) (thickness 0.15)))
-    )
-    (fp_text user "${REFERENCE}" (at 2.54 -2.37 90) (layer "F.Fab")
+    (fp_text reference "R4" (at 2.54 -2.37 -90) (layer "F.SilkS")
+        (effects (font (size 1 1) (thickness 0.15)))
+    )
+    (fp_text value "100k" (at 2.54 2.37 -90) (layer "F.Fab")
+        (effects (font (size 1 1) (thickness 0.15)))
+    )
+    (fp_text user "${REFERENCE}" (at 2.54 -2.37 -90) (layer "F.Fab")
         (effects (font (size 1 1) (thickness 0.15)))
     )
@@
   (arc (start 110.49 91.548949) (mid 110.159938 93.208283) (end 109.22 94.615) (width 0.4064) (layer "In4.Cu") (net 6))
   (arc (start 111.76 86.36) (mid 110.820062 87.766715) (end 110.49 89.426051) (width 0.4064) (layer "In4.Cu") (net 6))
-  (segment (start 99.06 93.98) (end 88.9 93.98) (width 0.4064) (layer "F.Cu") (net 7))
+  (segment (start 99.06 86.36) (end 96.52 86.36) (width 0.4064) (layer "F.Cu") (net 7))
+  (segment (start 99.06 93.98) (end 93.98 93.98) (width 0.4064) (layer "F.Cu") (net 7))
+  (segment (start 96.52 86.36) (end 93.98 86.36) (width 0.4064) (layer "F.Cu") (net 7))
+  (segment (start 93.98 86.36) (end 88.9 86.36) (width 0.4064) (layer "F.Cu") (net 7))
+  (segment (start 93.98 93.98) (end 88.9 93.98) (width 0.4064) (layer "F.Cu") (net 7))
   (via (at 99.06 93.98) (size 0.8) (drill 0.4) (layers "F.Cu" "B.Cu") (net 7))
-  (segment (start 106.648089 97.12309) (end 107.95 98.425) (width 0.4064) (layer "In3.Cu") (net 7))
-  (arc (start 99.06 93.98) (mid 103.166644 94.796862) (end 106.648089 97.12309) (width 0.4064) (layer "In3.Cu") (net 7))
+  (via (at 96.52 86.36) (size 0.8) (drill 0.4) (layers "F.Cu" "B.Cu") (net 7))
+  (via (at 96.52 93.98) (size 0.8) (drill 0.4) (layers "F.Cu" "B.Cu") (net 7))
+  (segment (start 96.52 93.98) (end 96.52 86.36) (width 0.4064) (layer "In1.Cu") (net 7))
+  (segment (start 107.95 98.425) (end 106.64809 97.12309) (width 0.25) (layer "In3.Cu") (net 7))
+  (arc (start 106.64809 97.12309) (mid 103.166645 94.796862) (end 99.06 93.98) (width 0.25) (layer "In3.Cu") (net 7))
   (segment (start 116.84 88.9) (end 111.76 88.9) (width 0.4064) (layer "F.Cu") (net 8))
   (segment (start 111.76 91.44) (end 109.22 91.44) (width 0.4064) (layer "F.Cu") (net 8))
@@
   (via (at 111.76 88.9) (size 0.8) (drill 0.4) (layers "F.Cu" "B.Cu") (net 8))
   (segment (start 111.76 91.44) (end 111.76 88.9) (width 0.4064) (layer "In1.Cu") (net 8))
-  (segment (start 99.06 86.36) (end 96.52 86.36) (width 0.4064) (layer "F.Cu") (net 9))
   (segment (start 99.06 88.9) (end 96.52 88.9) (width 0.4064) (layer "F.Cu") (net 9))
   (segment (start 96.52 88.9) (end 88.9 88.9) (width 0.4064) (layer "F.Cu") (net 9))
-  (segment (start 96.52 86.36) (end 88.9 86.36) (width 0.4064) (layer "F.Cu") (net 9))
-  (via (at 96.52 88.9) (size 0.8) (drill 0.4) (layers "F.Cu" "B.Cu") (net 9))
-  (via (at 96.52 86.36) (size 0.8) (drill 0.4) (layers "F.Cu" "B.Cu") (net 9))
-  (segment (start 96.52 88.9) (end 96.52 86.36) (width 0.4064) (layer "In1.Cu") (net 9))
   (segment (start 99.06 27.94) (end 88.9 27.94) (width 0.4064) (layer "F.Cu") (net 13))
   (segment (start 99.06 76.2) (end 88.9 76.2) (width 0.4064) (layer "F.Cu") (net 16))

Commit message: Switches module - prototype wip
Parts:
- Q1, Q2: value J109/112 -> J109/J112
- R4: value 100k -> 240K
- moved R5 7.62 mm to (106.7, 30.5), turned to 180 degrees
Connections:
- R5 pad 1: Net-(R4-Pad1) -> +5V
- R5 pad 2: GND -> Net-(R4-Pad1)
Routing:
- net +5V: track 0.00 -> 106.2 mm, vias 0 -> 1
- net GND: track 213.5 -> 200.8 mm, vias 8 -> 6
- net Net-(Q2-D): track 23.9 -> 22.9 mm, vias 1 -> 2
Changed lines of the file:
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@@
         (effects (font (size 1 1) (thickness 0.15)))
     )
-    (fp_text value "J109/112" (at 2.54 2.79 90) (layer "F.Fab")
+    (fp_text value "J109/J112" (at 2.54 2.79 90) (layer "F.Fab")
         (effects (font (size 1 1) (thickness 0.15)))
     )
@@
         (effects (font (size 1 1) (thickness 0.15)))
     )
-    (fp_text value "J109/112" (at 2.54 2.79 90) (layer "F.Fab")
+    (fp_text value "J109/J112" (at 2.54 2.79 90) (layer "F.Fab")
         (effects (font (size 1 1) (thickness 0.15)))
     )
@@
         (effects (font (size 1 1) (thickness 0.15)))
     )
-    (fp_text value "100k" (at 2.54 2.37 -90) (layer "F.Fab")
+    (fp_text value "240K" (at 2.54 2.37 -90) (layer "F.Fab")
         (effects (font (size 1 1) (thickness 0.15)))
     )
@@
   )
   (footprint "-lmp-misc:R_Axial_DIN0207_L6.3mm_D2.5mm_P7.62mm_Horizontal" (layer "F.Cu")
-    (at 99.06 30.48)
+    (at 106.68 30.48 180)
     (descr "Resistor, Axial_DIN0207 series, Axial, Horizontal, pin pitch=7.62mm, 0.25W = 1/4W, length*diameter=6.3*2.5mm^2, http://cdn-reichelt.de/documents/datenblatt/B400/1_4W%23YAG.pdf")
     (tags "Resistor Axial_DIN0207 series Axial Horizontal pin pitch 7.62mm 0.25W = 1/4W length 6.3mm diameter 2.5mm")
@@
     (fp_line (start 7.62 0) (end 6.96 0)
       (stroke (width 0.1) (type solid)) (layer "F.Fab"))
-    (pad "1" thru_hole circle (at 0 0) (size 1.6 1.6) (drill 0.8) (layers "*.Cu" "*.Mask")
+    (pad "1" thru_hole circle (at 0 0 180) (size 1.6 1.6) (drill 0.8) (layers "*.Cu" "*.Mask")
+      (net 4 "+5V") (pintype "passive"))
+    (pad "2" thru_hole oval (at 7.62 0 180) (size 1.6 1.6) (drill 0.8) (layers "*.Cu" "*.Mask")
       (net 19 "Net-(R4-Pad1)") (pintype "passive"))
-    (pad "2" thru_hole oval (at 7.62 0) (size 1.6 1.6) (drill 0.8) (layers "*.Cu" "*.Mask")
-      (net 2 "GND") (pintype "passive"))
     (model "${KISYS3DMOD}/Resistor_THT.3dshapes/R_Axial_DIN0207_L6.3mm_D2.5mm_P7.62mm_Horizontal.wrl"
       (offset (xyz 0 0 0))
@@
   (segment (start 116.84 78.74) (end 106.68 78.74) (width 0.4064) (layer "F.Cu") (net 2))
   (segment (start 119.38 25.36) (end 119.38 30.48) (width 0.4064) (layer "F.Cu") (net 2))
-  (segment (start 116.84 30.48) (end 111.76 30.48) (width 0.4064) (layer "F.Cu") (net 2))
   (segment (start 119.38 95.25) (end 119.38 95.25) (width 0.4064) (layer "F.Cu") (net 2))
   (segment (start 86.36 95.25) (end 86.36 95.25) (width 0.4064) (layer "F.Cu") (net 2))
@@
   (segment (start 86.36 78.74) (end 86.36 95.25) (width 0.4064) (layer "F.Cu") (net 2))
   (segment (start 119.38 30.48) (end 119.38 78.74) (width 0.4064) (layer "F.Cu") (net 2))
-  (segment (start 111.76 30.48) (end 106.68 30.48) (width 0.4064) (layer "F.Cu") (net 2))
   (via (at 119.38 95.25) (size 0.8) (drill 0.4) (layers "F.Cu" "B.Cu") (net 2))
-  (via (at 119.38 30.48) (size 0.8) (drill 0.4) (layers "F.Cu" "B.Cu") (net 2))
-  (via (at 116.84 30.48) (size 0.8) (drill 0.4) (layers "F.Cu" "B.Cu") (net 2))
   (via (at 86.36 78.74) (size 0.8) (drill 0.4) (layers "F.Cu" "B.Cu") (net 2))
   (via (at 88.9 78.74) (size 0.8) (drill 0.4) (layers "F.Cu" "B.Cu") (net 2))
@@
   (via (at 86.36 95.25) (size 0.8) (drill 0.4) (layers "F.Cu" "B.Cu") (net 2))
   (via (at 116.84 78.74) (size 0.8) (drill 0.4) (layers "F.Cu" "B.Cu") (net 2))
-  (segment (start 116.84 30.48) (end 119.38 30.48) (width 0.4064) (layer "In1.Cu") (net 2))
   (segment (start 88.9 78.74) (end 86.36 78.74) (width 0.4064) (layer "In1.Cu") (net 2))
   (segment (start 119.38 78.74) (end 116.84 78.74) (width 0.4064) (layer "In1.Cu") (net 2))
@@
   (segment (start 120.015 98.425) (end 113.03 98.425) (width 0.25) (layer "B.Cu") (net 3))
   (segment (start 121.92 96.52) (end 120.015 98.425) (width 0.25) (layer "B.Cu") (net 3))
-  (segment (start 116.84 86.36) (end 111.76 86.36) (width 0.4064) (layer "F.Cu") (net 6))
-  (segment (start 111.76 86.36) (end 109.22 86.36) (width 0.4064) (layer "F.Cu") (net 6))
+  (segment (start 116.84 30.48) (end 111.76 30.48) (width 0.4064) (layer "F.Cu") (net 4))
+  (segment (start 111.76 30.48) (end 106.68 30.48) (width 0.4064) (layer "F.Cu") (net 4))
+  (via (at 116.84 30.48) (size 0.8) (drill 0.4) (layers "F.Cu" "B.Cu") (net 4))
+  (segment (start 99.06 100.965) (end 98.688026 100.593025) (width 0.25) (layer "In4.Cu") (net 4))
+  (segment (start 122.645 94.615) (end 122.645 96.039696) (width 0.25) (layer "In4.Cu") (net 4))
+  (segment (start 121.92 97.79) (end 120.804077 98.905923) (width 0.25) (layer "In4.Cu") (net 4))
+  (segment (start 122.645 86.36) (end 122.645 94.615) (width 0.25) (layer "In4.Cu") (net 4))
+  (segment (start 114.3 101.6) (end 100.593025 101.6) (width 0.25) (layer "In4.Cu") (net 4))
+  (segment (start 122.645 86.36) (end 122.645 44.494509) (width 0.25) (layer "In4.Cu") (net 4))
+  (arc (start 98.688026 100.593025) (mid 98.023389 99.598327) (end 97.79 98.425) (width 0.25) (layer "In4.Cu") (net 4))
+  (arc (start 120.804077 98.905923) (mid 117.819982 100.899832) (end 114.3 101.6) (width 0.25) (layer "In4.Cu") (net 4))
+  (arc (start 100.593025 101.6) (mid 99.763358 101.434969) (end 99.06 100.965) (width 0.25) (layer "In4.Cu") (net 4))
+  (arc (start 122.645 44.494509) (mid 121.13633 36.909912) (end 116.84 30.48) (width 0.25) (layer "In4.Cu") (net 4))
+  (arc (start 122.645 96.039696) (mid 122.456578 96.986953) (end 121.92 97.79) (width 0.25) (layer "In4.Cu") (net 4))
+  (segment (start 116.84 86.36) (end 109.22 86.36) (width 0.4064) (layer "F.Cu") (net 6))
   (segment (start 109.22 86.36) (end 106.68 86.36) (width 0.4064) (layer "F.Cu") (net 6))
-  (via (at 111.76 86.36) (size 0.8) (drill 0.4) (layers "F.Cu" "B.Cu") (net 6))
-  (segment (start 110.49 89.426051) (end 110.49 91.548949) (width 0.4064) (layer "In4.Cu") (net 6))
-  (segment (start 109.22 94.615) (end 105.41 98.425) (width 0.4064) (layer "In4.Cu") (net 6))
-  (arc (start 110.49 91.548949) (mid 110.159938 93.208283) (end 109.22 94.615) (width 0.4064) (layer "In4.Cu") (net 6))
-  (arc (start 111.76 86.36) (mid 110.820062 87.766715) (end 110.49 89.426051) (width 0.4064) (layer "In4.Cu") (net 6))
+  (via (at 109.22 86.36) (size 0.8) (drill 0.4) (layers "F.Cu" "B.Cu") (net 6))
+  (segment (start 105.41 98.425) (end 109.22 94.615) (width 0.4064) (layer "In4.Cu") (net 6))
+  (segment (start 110.49 91.548949) (end 110.49 89.426051) (width 0.4064) (layer "In4.Cu") (net 6))
+  (arc (start 109.22 86.36) (mid 110.159937 87.766715) (end 110.49 89.426051) (width 0.4064) (layer "In4.Cu") (net 6))
+  (arc (start 109.22 94.615) (mid 110.159938 93.208283) (end 110.49 91.548949) (width 0.4064) (layer "In4.Cu") (net 6))
   (segment (start 99.06 86.36) (end 96.52 86.36) (width 0.4064) (layer "F.Cu") (net 7))
   (segment (start 99.06 93.98) (end 93.98 93.98) (width 0.4064) (layer "F.Cu") (net 7))
@@
   (segment (start 116.84 91.44) (end 111.76 91.44) (width 0.4064) (layer "F.Cu") (net 8))
   (segment (start 111.76 88.9) (end 109.22 88.9) (width 0.4064) (layer "F.Cu") (net 8))
-  (via (at 111.76 91.44) (size 0.8) (drill 0.4) (layers "F.Cu" "B.Cu") (net 8))
-  (via (at 111.76 88.9) (size 0.8) (drill 0.4) (layers "F.Cu" "B.Cu") (net 8))
-  (segment (start 111.76 91.44) (end 111.76 88.9) (width 0.4064) (layer "In1.Cu") (net 8))
+  (via (at 109.22 91.44) (size 0.8) (drill 0.4) (layers "F.Cu" "B.Cu") (net 8))
+  (via (at 109.22 88.9) (size 0.8) (drill 0.4) (layers "F.Cu" "B.Cu") (net 8))
+  (segment (start 109.22 91.44) (end 109.22 88.9) (width 0.4064) (layer "In1.Cu") (net 8))
   (segment (start 99.06 88.9) (end 96.52 88.9) (width 0.4064) (layer "F.Cu") (net 9))
   (segment (start 96.52 88.9) (end 88.9 88.9) (width 0.4064) (layer "F.Cu") (net 9))
@@
   (segment (start 99.06 83.82) (end 96.52 83.82) (width 0.4064) (layer "F.Cu") (net 18))
   (segment (start 93.98 83.82) (end 88.9 83.82) (width 0.4064) (layer "F.Cu") (net 18))
+  (via (at 96.52 81.28) (size 0.8) (drill 0.4) (layers "F.Cu" "B.Cu") (net 18))
   (via (at 96.52 83.82) (size 0.8) (drill 0.4) (layers "F.Cu" "B.Cu") (net 18))
-  (segment (start 96.52 83.82) (end 99.06 81.28) (width 0.4064) (layer "In3.Cu") (net 18))
+  (segment (start 96.52 83.82) (end 96.52 81.28) (width 0.4064) (layer "In1.Cu") (net 18))
   (segment (start 99.06 30.48) (end 88.9 30.48) (width 0.4064) (layer "F.Cu") (net 19))
 )

Commit message: Switches module - prototype wip
Parts:
- added Q3: 2N3906, -lmp-misc:TO-92_Inline_Wide, F.Cu at (109.2, 25.4)
- added R7: 10K, -lmp-stripboard:SB_Gen_2, F.Cu at (100.6, 29.2)
- added R8: 10K, -lmp-stripboard:SB_Gen_2, F.Cu at (96.5, 30.7)
- R5: footprint -lmp-misc:R_Axial_DIN0207_L6.3mm_D2.5mm_P7.62mm_Horizontal -> -lmp-stripboard:SB_Gen_2
- moved C1 28.0 mm to (116.9, 35.6), turned to 0 degrees
- moved R4 17.8 mm to (114.3, 30.7)
- moved R5 10.2 mm to (116.8, 30.5), turned to 0 degrees
Connections:
- R4 pad 1: Net-(R4-Pad1) -> Net-(Q3-C)
- R5 pad 1: +5V -> Net-(Q3-C)
- R5 pad 2: Net-(R4-Pad1) -> -12V
- SW1 pad 2: -12V -> +5V
- SW1 pad 4: Net-(R4-Pad1) -> Net-(R7-Pad1)
Routing:
- net -12V: track 129.7 -> 96.0 mm, vias 5 -> 3
- net (no net): track 365.8 -> 335.3 mm
- net +5V: track 106.2 -> 129.0 mm, vias 1 -> 3
- net GND: track 200.8 -> 213.5 mm, vias 6 -> 8
- net Net-(R7-Pad1): track 0.00 -> 12.2 mm, vias 0 -> 1
- net Net-(Q3-B): track 0.00 -> 11.8 mm, vias 0 -> 1
- net Net-(R4-Pad1): track 10.2 -> 0.00 mm
- net Net-(Q3-C): track 0.00 -> 10.2 mm

Commit message: Switches module - prototype wip
Changed lines of the file:
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@@
   (segment (start 119.38 95.25) (end 119.38 95.25) (width 0.4064) (layer "F.Cu") (net 2))
   (segment (start 86.36 95.25) (end 86.36 95.25) (width 0.4064) (layer "F.Cu") (net 2))
-  (segment (start 86.36 35.56) (end 86.36 78.74) (width 0.4064) (layer "F.Cu") (net 2))
+  (segment (start 86.36 35.56) (end 86.36 38.1) (width 0.4064) (layer "F.Cu") (net 2))
   (segment (start 119.38 78.74) (end 119.38 95.25) (width 0.4064) (layer "F.Cu") (net 2))
   (segment (start 86.36 78.74) (end 86.36 95.25) (width 0.4064) (layer "F.Cu") (net 2))
   (segment (start 99.06 35.56) (end 91.44 35.56) (width 0.4064) (layer "F.Cu") (net 2))
+  (segment (start 86.36 38.1) (end 86.36 78.74) (width 0.4064) (layer "F.Cu") (net 2))
   (segment (start 119.38 30.48) (end 119.38 78.74) (width 0.4064) (layer "F.Cu") (net 2))
   (segment (start 91.44 35.56) (end 88.9 35.56) (width 0.4064) (layer "F.Cu") (net 2))
   (via (at 119.38 95.25) (size 0.8) (drill 0.4) (layers "F.Cu" "B.Cu") (net 2))
   (via (at 86.36 78.74) (size 0.8) (drill 0.4) (layers "F.Cu" "B.Cu") (net 2))
-  (via (at 86.36 35.56) (size 0.8) (drill 0.4) (layers "F.Cu" "B.Cu") (net 2))
   (via (at 88.9 78.74) (size 0.8) (drill 0.4) (layers "F.Cu" "B.Cu") (net 2))
   (via (at 119.38 78.74) (size 0.8) (drill 0.4) (layers "F.Cu" "B.Cu") (net 2))
@@
   (via (at 86.36 95.25) (size 0.8) (drill 0.4) (layers "F.Cu" "B.Cu") (net 2))
   (via (at 116.84 78.74) (size 0.8) (drill 0.4) (layers "F.Cu" "B.Cu") (net 2))
+  (via (at 86.36 35.56) (size 0.8) (drill 0.4) (layers "F.Cu" "B.Cu") (net 2))
   (segment (start 88.9 35.56) (end 86.36 35.56) (width 0.4064) (layer "In1.Cu") (net 2))
   (segment (start 88.9 78.74) (end 86.36 78.74) (width 0.4064) (layer "In1.Cu") (net 2))

Commit message: Switches module - prototype - wip
Parts:
- SW1: footprint -lmp-synth:SW_Push_LED_C&K_D6R -> -lmp-misc:SW_PUSH_6mm_2
- moved SW1 5.63 mm to (88.9, 28.0)
Connections:
- SW1 pad 1: unconnected-(SW1-Pad1) -> +5V
- SW1 pad 2: +5V -> Net-(R7-Pad1)
Routing:
- net unconnected-(SW1-K-Pad6): track 10.2 -> 0.00 mm
- net (no net): track 335.3 -> 345.4 mm
