File: modules/Switches/prototype/switch/prototype.kicad_sch (KiCad schematic)
At the start: 22 parts, among them J1 Conn_01x09, Q1 J109/J112, Q2 J109/J112, Q3 2N3906, SW2 SW_Push_LED, U1 TL072, U2 SN74HCS74

Commit message: Switches module - prototype - wip
Parts:
- R4: Note (none) -> value as req'd
Changed lines of the file:
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@@
   (symbol (lib_id "-lmp:R_1%_0W166") (at 80.01 90.17 90) (unit 1)
     (in_bom yes) (on_board yes) (dnp no) (fields_autoplaced)
-    (property "Reference" "R4" (at 80.01 85.0097 90)
+    (property "Reference" "R4" (at 80.01 82.5855 90)
       (effects (font (size 1.27 1.27)))
     )
-    (property "Value" "240K" (at 80.01 87.4339 90)
+    (property "Value" "240K" (at 80.01 85.0097 90)
       (effects (font (size 1.27 1.27)))
     )
@@
       (effects (font (size 1.27 1.27)) hide)
     )
+    (property "Note" "value as req'd" (at 80.01 87.4339 90)
+      (effects (font (size 1.27 1.27)))
+    )
     (pin "1")

Commit message: Switches - module design - wip
Parts:
- R12: value 1K -> 330R; Note Output limiting -> as req'd
- R4: Note value as req'd -> as req'd
Connections:
- net IN-OUT-1 renamed IN-1
- net IN-OUT-2 renamed OUT-1
Other:
- moved on the sheet: C1, C2, C3, C4, J1, Q1, Q2, Q3, R1, R10, R11, R12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
