File: modules/Switches/temp/PanelPower.kicad_sch (KiCad schematic)
At the start: 29 parts, among them J10 Conn_Front_Top, J11 Conn_Front_Bottom, J12 Conn_Back_Top, J13 Conn_Back_Bottom, J9 Conn_Eurorack_16, SW1 D6RLxxF1, SW2 D6RLxxF1, SW3 D6RLxxF1, SW4 D6RLxxF1, U2 SN74HCS74

Commit message: Switches - temp partial PCB layout
Parts:
- removed C12, C19, C20: 1N, -lmp-misc:C_Disc_D5.0mm_W2.5mm_P2.50mm, symbol -lmp:CC
- removed C21: 100N, -lmp-misc:C_Disc_D5.0mm_W2.5mm_P2.50mm, symbol -lmp:CC_100N
- removed SW2, SW3, SW4: D6RLxxF1, -lmp-synth:SW_Push_LED_C&K_D6R, symbol -lmp-synth:SW_Push_LED_C&K_D6R
- removed U2: SN74HCS74, Package_SO:SOIC-14_3.9x8.7mm_P1.27mm, symbol -lmp-IC-misc:SN74HCS74
