File: modules/Filter2/Filter2.kicad_pcb (KiCad board)
At the start: 2 copper layers, 111.5 x 108.2 mm, 52 parts, among them J1 WQP-PJ398, J10 Conn_Back_Left, J2 WQP-PJ398, J3 WQP-PJ398, J4 WQP-PJ398, J5 WQP-PJ398, J6 Conn_Eurorack_16, J7 Conn_Front_Left_Top, J8 Conn_Front_Right, J9 Conn_Back_Right_Top, SW1 SW_SP3T, SW2 SW_SP3T, U1 TL074, U2 TL074

Commit message: Filter2 - wip
Parts:
- removed J3: WQP-PJ398, -lmp-synth:Jack_3.5mm_QingPu_WQP-PJ398SM_Vertical
- moved R6 98.0 mm to (112.8, 90.2), turned to 180 degrees
- moved R9 74.7 mm to (166.2, 113.9)
- moved R5 74.5 mm to (166.4, 109.7)
- moved R7 54.3 mm to (177.2, 118.9)
- moved R3 45.6 mm to (166.4, 102.1)
- moved C10 44.2 mm to (174.0, 105.9), turned to 180 degrees
- moved R8 40.6 mm to (177.2, 94.8)
- moved R4 36.6 mm to (174.0, 98.2), turned to 180 degrees
- moved R11 32.1 mm to (203.3, 71.2), turned to 180 degrees
- moved C11 32.0 mm to (190.6, 106.6), turned to 180 degrees
- moved R14 8.53 mm to (101.5, 108.8)
- moved R13 7.89 mm to (203.3, 67.3), turned to 180 degrees
- moved C2 5.57 mm to (188.1, 113.3), turned to 0 degrees
- moved C3 5.08 mm to (193.6, 101.5), turned to 180 degrees
- moved R10 1.27 mm to (105.0, 52.8)
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Connections:
- J7 pad 2: Net-(J7-Pin_2) -> LP-1
- J7 pad 3: Net-(J7-Pin_3) -> BP-1
- J7 pad 4: Net-(J7-Pin_4) -> F-CTRL-1-2
- J7 pad 5: Net-(J7-Pin_5) -> F-CTRL-1-1
- J7 pad 6: Net-(J7-Pin_6) -> HP-1
- J7 pad 7: Net-(J7-Pin_7) -> FILTER-IN-1
- J7 pad 8: Net-(J7-Pin_8) -> Q-CTRL-1
- J9 pad 2: Net-(J7-Pin_2) -> LP-1
- J9 pad 3: Net-(J7-Pin_3) -> BP-1
- J9 pad 4: Net-(J7-Pin_4) -> F-CTRL-1-2
- J9 pad 5: Net-(J7-Pin_5) -> F-CTRL-1-1
- J9 pad 6: Net-(J7-Pin_6) -> HP-1
- J9 pad 7: Net-(J7-Pin_7) -> FILTER-IN-1
- J9 pad 8: Net-(J7-Pin_8) -> Q-CTRL-1
- R11 pad 1: Net-(R11-Pad1) -> F-CTRL-1-1
- R13 pad 1: Net-(R13-Pad1) -> F-CTRL-1-2
- R5 pad 2: Net-(U2B-+) -> Q-CTRL-1
- R6 pad 2: Net-(U2B-+) -> Q-CTRL-1
- R7 pad 1: Net-(U2B-+) -> Q-CTRL-1
- RV3 pad 2: Net-(R13-Pad1) -> F-CTRL-1-2
- RV3 pad 5: Net-(R11-Pad1) -> F-CTRL-1-1
- U2 pad 5: Net-(U2B-+) -> Q-CTRL-1
Routing:
- net Q-CTRL-1: track 0.00 -> 97.7 mm
- net LP-1: track 0.00 -> 88.4 mm
- net BP-1: track 44.0 -> 116.5 mm
- net HP-1: track 46.9 -> 111.9 mm, vias 0 -> 1
- net FILTER-IN-1: track 31.7 -> 92.4 mm, vias 0 -> 1
- net Net-(U2C--): track 0.00 -> 54.6 mm
- net Net-(U2D--): track 0.00 -> 54.1 mm
- net -12V: track 146.1 -> 186.0 mm, vias 2 -> 3
- net +12V: track 129.5 -> 163.9 mm, vias 0 -> 1
- net Net-(U2B--): track 0.00 -> 30.4 mm
- net Net-(R4-Pad2): track 0.00 -> 26.0 mm
- net F-CTRL-1-1: track 0.00 -> 17.9 mm
- net F-CTRL-1-2: track 0.00 -> 17.7 mm
- net Net-(R6-Pad1): track 19.0 -> 3.83 mm
- net Net-(R13-Pad1): track 12.5 -> 0.00 mm
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Other:
- board text removed: "TODO: connect headers"

Commit message: Filter2 - wip
Parts:
- moved C3 21.3 mm to (187.5, 121.9)
- moved R3 21.3 mm to (160.3, 122.5)
- moved R5 21.3 mm to (160.3, 130.0)
- moved R8 21.3 mm to (171.0, 115.2)
- moved C11 21.3 mm to (184.4, 127.0)
- moved R4 21.3 mm to (167.9, 118.6)
- moved R9 21.3 mm to (160.1, 134.3)
- moved C10 21.3 mm to (167.9, 126.3)
- moved C2 21.3 mm to (182.0, 133.7)
- moved U2 21.3 mm to (171.1, 119.4)
- moved R7 21.0 mm to (171.0, 138.9)
Routing:
- net -12V: track 186.0 -> 149.4 mm, vias 3 -> 2
- net FILTER-IN-1: track 92.4 -> 125.8 mm
- net HP-1: track 111.9 -> 145.3 mm
- net Net-(U2D--): track 54.1 -> 87.4 mm
- net Net-(U2C--): track 54.6 -> 87.8 mm
- net LP-1: track 88.4 -> 121.5 mm
- net BP-1: track 116.5 -> 142.9 mm
- net Q-CTRL-1: track 97.7 -> 122.6 mm
- net +12V: track 163.9 -> 185.5 mm

Commit message: fix REFDES
Parts:
- renumbered C6 to C101, C7 to C102, C8 to C103, C9 to C104, C10 to C105, C11 to C106, H2 to H102, H4 to H104, H7 to H107, H9 to H109, J1 to J101, J2 to J102, J4 to J103, J5 to J104, J7 to J105, J9 to J106, J8 to J107, J10 to J108, J6 to J109

Commit message: Filter2 - second channel - wip
Parts:
- added C10: 22P, -lmp-misc:C_Disc_D5.0mm_W2.5mm_P2.50mm, F.Cu at (223.5, 113.1)
- added C107: 100N, -lmp-misc:C_Disc_D5.0mm_W2.5mm_P2.50mm, F.Cu at (225.4, 121.5)
- added C108: 100N, -lmp-misc:C_Disc_D5.0mm_W2.5mm_P2.50mm, F.Cu at (225.4, 125.5)
- added C6: 1U, -lmp-misc:C_Rect_Kemet_L7.2mm_W2.5mm_P5mm, F.Cu at (213.7, 122.3)
- added C7: 6N8, -lmp-misc:C_Rect_Kemet_L7.2mm_W2.5mm_P5mm, F.Cu at (213.7, 127.9)
- added C8: 6N8, -lmp-misc:C_Rect_Kemet_L7.2mm_W2.5mm_P5mm, F.Cu at (213.7, 133.5)
- added C9: 1U, -lmp-misc:C_Rect_Kemet_L7.2mm_W2.5mm_P5mm, F.Cu at (213.7, 139.1)
- added R17: 1M, -lmp-misc:R_Axial_DIN0207_L6.3mm_D2.5mm_P7.62mm_Horizontal, F.Cu at (212.7, 58.2)
- added R18: 100K, -lmp-misc:R_Axial_DIN0207_L6.3mm_D2.5mm_P7.62mm_Horizontal, F.Cu at (212.7, 62.2)
- added R19: 10K, -lmp-misc:R_Axial_DIN0207_L6.3mm_D2.5mm_P7.62mm_Horizontal, F.Cu at (212.7, 66.3)
- added R20: 22K, -lmp-misc:R_Axial_DIN0207_L6.3mm_D2.5mm_P7.62mm_Horizontal, F.Cu at (212.7, 70.3)
- added R21: 22K, -lmp-misc:R_Axial_DIN0207_L6.3mm_D2.5mm_P7.62mm_Horizontal, F.Cu at (212.7, 74.4)
- added R22: 1K, -lmp-misc:R_Axial_DIN0207_L6.3mm_D2.5mm_P7.62mm_Horizontal, F.Cu at (212.7, 78.4)
- added R23: 10K, -lmp-misc:R_Axial_DIN0207_L6.3mm_D2.5mm_P7.62mm_Horizontal, F.Cu at (212.7, 82.5)
- added R24: 15K, -lmp-misc:R_Axial_DIN0207_L6.3mm_D2.5mm_P7.62mm_Horizontal, F.Cu at (212.7, 86.5)
- added R25: 15K, -lmp-misc:R_Axial_DIN0207_L6.3mm_D2.5mm_P7.62mm_Horizontal, F.Cu at (212.7, 90.6)
- added R26: 220R, -lmp-misc:R_Axial_DIN0207_L6.3mm_D2.5mm_P7.62mm_Horizontal, F.Cu at (212.7, 94.6)
- added R27: 10K, -lmp-misc:R_Axial_DIN0207_L6.3mm_D2.5mm_P7.62mm_Horizontal, F.Cu at (212.7, 98.7)
- added R28: 220R, -lmp-misc:R_Axial_DIN0207_L6.3mm_D2.5mm_P7.62mm_Horizontal, F.Cu at (212.7, 102.7)
- added R29: 10K, -lmp-misc:R_Axial_DIN0207_L6.3mm_D2.5mm_P7.62mm_Horizontal, F.Cu at (212.7, 106.8)
- added R30: 1M, -lmp-misc:R_Axial_DIN0207_L6.3mm_D2.5mm_P7.62mm_Horizontal, F.Cu at (212.7, 110.8)
- added R31: 100K, -lmp-misc:R_Axial_DIN0207_L6.3mm_D2.5mm_P7.62mm_Horizontal, F.Cu at (125.9, 132.0)
- added R32: 51R, -lmp-misc:R_Axial_DIN0207_L6.3mm_D2.5mm_P10.16mm_Horizontal, F.Cu at (223.0, 109.1)
- added RV4: 50K, -lmp-synth:Potentiometer_Alpha_RD902F-40-00D_Dual_Vertical, F.Cu at (123.2, 65.6)
- added RV5: 50K, -lmp-synth:Potentiometer_Alpha_RD901F-40-00D_Single_Vertical, F.Cu at (131.8, 93.4)
- added RV6: 10K, -lmp-synth:Potentiometer_Alpha_RD902F-40-00D_Dual_Vertical, F.Cu at (123.2, 79.5)
- added U3: TL074, Package_DIP:DIP-14_W7.62mm, F.Cu at (223.5, 86.0)
Connections:
- J103 pad T: unconnected-(J103-PadT) -> IN-2
- J104 pad T: unconnected-(J104-PadT) -> OUT-2
- SW2 pad 1: unconnected-(SW2-Pad1) -> LP-2
- SW2 pad 2: unconnected-(SW2-Pad2) -> Net-(RV4-Pad6)
- SW2 pad 4: unconnected-(SW2-Pad4) -> BP-2
- SW2 pad 6: unconnected-(SW2-Pad6) -> HP-2
- U1 pad 10: unconnected-(U1C-+-Pad10) -> Net-(U1C-+)
- U1 pad 5: unconnected-(U1B-+-Pad5) -> Net-(U1B-+)
- U1 pad 6: unconnected-(U1B---Pad6) -> Net-(U1B--)
- U1 pad 7: unconnected-(U1-Pad7) -> Net-(C10-Pad2)
- U1 pad 8: unconnected-(U1-Pad8) -> Net-(U1C--)
- U1 pad 9: unconnected-(U1C---Pad9) -> Net-(U1C--)

Commit message: Filter2 - second channel - wip
Parts:
- moved R17 101.0 mm to (133.7, 121.1), turned to -90 degrees
- moved R28 100.6 mm to (127.6, 49.0)
- moved R18 100.2 mm to (125.9, 112.3)
- moved C10 95.9 mm to (129.9, 134.5), turned to 90 degrees
- moved R26 94.8 mm to (127.6, 52.7)
- moved R32 92.2 mm to (133.7, 132.0), turned to -90 degrees
- moved R22 82.9 mm to (130.7, 90.2)
- moved C6 81.5 mm to (132.4, 117.2), turned to 180 degrees
- moved C9 80.4 mm to (137.6, 113.1)
- moved R30 69.5 mm to (143.3, 108.8), turned to 90 degrees
- moved R29 65.8 mm to (162.1, 64.8)
- moved C108 65.4 mm to (176.1, 82.4), turned to -90 degrees
- moved C8 64.7 mm to (171.1, 84.8), turned to 90 degrees
- moved R27 58.3 mm to (162.1, 69.8)
- moved R19 57.3 mm to (172.0, 106.6), turned to 90 degrees
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Connections:
- J107 pad 2: Net-(J107-Pin_2) -> LP-2
- J107 pad 3: Net-(J107-Pin_3) -> F-CTRL-2-2
- J107 pad 4: Net-(J107-Pin_4) -> BP-2
- J107 pad 5: Net-(J107-Pin_5) -> F-CTRL-2-1
- J107 pad 6: Net-(J107-Pin_6) -> HP-2
- J107 pad 7: Net-(J107-Pin_7) -> FILTER-IN-2
- J107 pad 8: Net-(J107-Pin_8) -> Q-CTRL-2
- J108 pad 2: Net-(J107-Pin_2) -> LP-2
- J108 pad 3: Net-(J107-Pin_3) -> F-CTRL-2-2
- J108 pad 4: Net-(J107-Pin_4) -> BP-2
- J108 pad 5: Net-(J107-Pin_5) -> F-CTRL-2-1
- J108 pad 6: Net-(J107-Pin_6) -> HP-2
- J108 pad 7: Net-(J107-Pin_7) -> FILTER-IN-2
- J108 pad 8: Net-(J107-Pin_8) -> Q-CTRL-2
Routing:
- net Q-CTRL-2: track 0.00 -> 95.0 mm
- net Net-(RV4-Pad6): track 0.00 -> 92.6 mm
- net HP-2: track 0.00 -> 87.7 mm
- net BP-2: track 0.00 -> 84.7 mm, vias 0 -> 1
- net FILTER-IN-2: track 0.00 -> 79.2 mm
- net LP-2: track 0.00 -> 68.2 mm
- net -12V: track 149.4 -> 199.9 mm, vias 2 -> 4
- net +12V: track 185.5 -> 218.2 mm, vias 1 -> 2
- net Net-(U1B-+): track 0.00 -> 31.8 mm
- net Net-(U3B--): track 0.00 -> 30.5 mm
- net Net-(R20-Pad2): track 0.00 -> 27.4 mm
- net Net-(U1C--): track 0.00 -> 27.2 mm
- net Net-(U3D--): track 0.00 -> 27.2 mm
- net Net-(U3C--): track 0.00 -> 23.1 mm
- net Net-(R26-Pad1): track 0.00 -> 20.6 mm
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
Commit message: Filter2 - second channel - wip
Parts:
- moved C101 14.4 mm to (204.7, 118.4), turned to 180 degrees
- moved J105 11.4 mm to (97.8, 71.1)
- moved J106 11.4 mm to (206.7, 71.1)
- moved J107 11.4 mm to (145.8, 71.1)
- moved J108 11.4 mm to (158.8, 71.1)
- moved R29 11.4 mm to (162.1, 76.2)
- moved R27 10.3 mm to (162.1, 80.1)
- moved R11 10.2 mm to (203.3, 81.4)
- moved R13 10.2 mm to (203.3, 77.5)
- moved C8 0.38 mm to (171.1, 84.5), turned to 180 degrees
Routing:
- net +12V: track 218.2 -> 189.5 mm, vias 2 -> 1
- net -12V: track 199.9 -> 177.1 mm, vias 4 -> 5
- net FILTER-IN-1: track 125.8 -> 103.0 mm
- net Q-CTRL-2: track 95.0 -> 74.5 mm
- net FILTER-IN-2: track 79.2 -> 59.2 mm
- net Q-CTRL-1: track 122.4 -> 103.0 mm
- net Net-(U2C--): track 87.8 -> 69.1 mm
- net Net-(U2D--): track 87.4 -> 69.4 mm
- net Net-(U3D--): track 27.2 -> 14.3 mm
- net F-CTRL-1-2: track 17.7 -> 25.5 mm
- net HP-1: track 145.3 -> 137.7 mm
- net Net-(U3C--): track 23.1 -> 16.8 mm
- net LP-1: track 121.5 -> 115.8 mm
- net BP-1: track 142.9 -> 137.6 mm
- net F-CTRL-2-2: track 17.1 -> 21.9 mm
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
Commit message: Filter2 - wip
Parts:
- removed H107, H109: MountingHole_M3, -lmp-holes:MountingHole_PCB_3.2mm_M3
- J105: footprint Connector_PinSocket_2.54mm:PinSocket_1x11_P2.54mm_Vertical -> Connector_PinSocket_2.54mm:PinSocket_1x10_P2.54mm_Vertical
- J106: footprint Connector_PinHeader_2.54mm:PinHeader_1x11_P2.54mm_Vertical -> Connector_PinHeader_2.54mm:PinHeader_1x10_P2.54mm_Vertical
- J107: footprint Connector_PinSocket_2.54mm:PinSocket_1x08_P2.54mm_Vertical -> Connector_PinSocket_2.54mm:PinSocket_1x07_P2.54mm_Vertical
- J108: footprint Connector_PinHeader_2.54mm:PinHeader_1x08_P2.54mm_Vertical -> Connector_PinHeader_2.54mm:PinHeader_1x07_P2.54mm_Vertical
- moved G1 72.4 mm to (191.6, 112.3)
- moved G3 66.8 mm to (200.0, 112.1)
- moved H102 34.9 mm to (121.8, 78.7)
- moved H104 34.9 mm to (182.7, 78.7)
- moved G4 20.2 mm to (121.9, 85.0)
- moved G2 17.9 mm to (121.9, 90.1)
- moved J105 2.54 mm to (97.8, 73.7)
- moved J106 2.54 mm to (206.7, 73.7)
- moved J107 2.54 mm to (145.8, 73.7)
- moved J108 2.54 mm to (158.8, 73.7)
- moved C7 0.46 mm to (181.2, 84.5), turned to 0 degrees
Connections:
- J105 pad 1: Net-(J105-Pin_1) -> LP-1
- J105 pad 10: +12V -> GND
- J105 pad 2: LP-1 -> BP-1
- J105 pad 3: BP-1 -> F-CTRL-1-2
- J105 pad 4: F-CTRL-1-2 -> F-CTRL-1-1
- J105 pad 5: F-CTRL-1-1 -> HP-1
- J105 pad 6: HP-1 -> FILTER-IN-1
- J105 pad 7: FILTER-IN-1 -> Q-CTRL-1
- J105 pad 8: Q-CTRL-1 -> -12V
- J105 pad 9: -12V -> +12V
- J106 pad 1: Net-(J105-Pin_1) -> LP-1
- J106 pad 10: +12V -> GND
- J106 pad 2: LP-1 -> BP-1
- J106 pad 3: BP-1 -> F-CTRL-1-2
- J106 pad 4: F-CTRL-1-2 -> F-CTRL-1-1
- J106 pad 5: F-CTRL-1-1 -> HP-1
- J106 pad 6: HP-1 -> FILTER-IN-1
- J106 pad 7: FILTER-IN-1 -> Q-CTRL-1
- J106 pad 8: Q-CTRL-1 -> -12V
- J106 pad 9: -12V -> +12V
- J107 pad 1: Net-(J107-Pin_1) -> LP-2
- J107 pad 2: LP-2 -> F-CTRL-2-2
- J107 pad 3: F-CTRL-2-2 -> BP-2
- J107 pad 4: BP-2 -> F-CTRL-2-1
- J107 pad 5: F-CTRL-2-1 -> HP-2
- J107 pad 6: HP-2 -> FILTER-IN-2
- J107 pad 7: FILTER-IN-2 -> Q-CTRL-2
- J108 pad 1: Net-(J107-Pin_1) -> LP-2
- J108 pad 2: LP-2 -> F-CTRL-2-2
- J108 pad 3: F-CTRL-2-2 -> BP-2
- J108 pad 4: BP-2 -> F-CTRL-2-1
- J108 pad 5: F-CTRL-2-1 -> HP-2
- J108 pad 6: HP-2 -> FILTER-IN-2
- J108 pad 7: FILTER-IN-2 -> Q-CTRL-2
Routing:
- net BP-2: track 85.1 -> 86.4 mm
Other:
- outline, holes or cut-outs redrawn
