File: modules/Filter2/panel/panel.kicad_pcb (KiCad board)
At the start: 2 copper layers, 50.5 x 128.5 mm, 18 parts

Commit message: Filter2: verify front panel positions
Other:
- board text removed: "TODO: verify switch positions"
Changed lines of the file:
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@@
     )
-  )
-  (gr_text "TODO: verify switch positions" (at 121.32 22.712) (layer "Cmts.User")
-    (effects (font (size 2 2) (thickness 0.3)))
   )
   (zone (net 0) (net_name "") (layers "F&B.Cu") (hatch edge 0.508)
